File: Electronics/BPS/Master/USB.sch (KiCad schematic (older format))
At the start: 9 parts

Commit message: Finalized schematics for BPS master.
Parts:
- gave numbers to parts that had none: 9
Changed lines of the file:
@@
 $EndDescr
 $Comp
-L Interface_USB:CP2102N-A01-GQFN24 U?
+L Interface_USB:CP2102N-A01-GQFN24 U17
 U 1 1 5C4963B2
 P 5500 3800
-F 0 "U?" H 5500 5200 50  0000 C CNN
+F 0 "U17" H 5500 5200 50  0000 C CNN
 F 1 "CP2102N-A01-GQFN24" H 5500 5100 50  0000 C CNN
 F 2 "Package_DFN_QFN:QFN-24-1EP_4x4mm_P0.5mm_EP2.6x2.6mm" H 5950 3000 50  0001 L CNN
@@
 $EndComp
 $Comp
-L Connector:USB_B_Micro J?
+L Connector:USB_B_Micro J21
 U 1 1 5C4964BB
 P 3000 4300
-F 0 "J?" H 3000 4750 50  0000 C CNN
+F 0 "J21" H 3000 4750 50  0000 C CNN
 F 1 "USB_B_Micro" H 3000 4650 50  0000 C CNN
 F 2 "" H 3150 4250 50  0001 C CNN
@@
 	3400 4200 3600 4200
 $Comp
-L power:GND #PWR?
+L power:GND #PWR0129
 U 1 1 5C4965DF
 P 3000 4800
-F 0 "#PWR?" H 3000 4550 50  0001 C CNN
+F 0 "#PWR0129" H 3000 4550 50  0001 C CNN
 F 1 "GND" H 3005 4627 50  0000 C CNN
 F 2 "" H 3000 4800 50  0001 C CNN
@@
 Connection ~ 3000 4750
 $Comp
-L power:GND #PWR?
+L power:GND #PWR0130
 U 1 1 5C4966CF
 P 5500 4800
-F 0 "#PWR?" H 5500 4550 50  0001 C CNN
+F 0 "#PWR0130" H 5500 4550 50  0001 C CNN
 F 1 "GND" H 5505 4627 50  0000 C CNN
 F 2 "" H 5500 4800 50  0001 C CNN
@@
 	5400 4750 5500 4750
 $Comp
-L Power_Protection:SP0503BAHT D?
+L Power_Protection:SP0503BAHT D13
 U 1 1 5C496C9B
 P 3950 4800
-F 0 "D?" H 4155 4846 50  0000 L CNN
+F 0 "D13" H 4155 4846 50  0000 L CNN
 F 1 "SP0503BAHT" H 4000 4650 50  0000 L CNN
 F 2 "Package_TO_SOT_SMD:SOT-143" H 4175 4750 50  0001 L CNN
@@
 $EndComp
 $Comp
-L power:GND #PWR?
+L power:GND #PWR0131
 U 1 1 5C497074
 P 3950 5050
-F 0 "#PWR?" H 3950 4800 50  0001 C CNN
+F 0 "#PWR0131" H 3950 4800 50  0001 C CNN
 F 1 "GND" H 3955 4877 50  0000 C CNN
 F 2 "" H 3950 5050 50  0001 C CNN
@@
 Connection ~ 3950 4200
 $Comp
-L Device:R R?
+L Device:R R52
 U 1 1 5C497DB9
 P 4700 4500
-F 0 "R?" H 4770 4546 50  0000 L CNN
+F 0 "R52" H 4770 4546 50  0000 L CNN
 F 1 "47.5k" H 4770 4455 50  0000 L CNN
 F 2 "" V 4630 4500 50  0001 C CNN
@@
 $EndComp
 $Comp
-L Device:R R?
+L Device:R R51
 U 1 1 5C497DDB
 P 4350 4100
-F 0 "R?" V 4143 4100 50  0000 C CNN
+F 0 "R51" V 4143 4100 50  0000 C CNN
 F 1 "22.1k" V 4234 4100 50  0000 C CNN
 F 2 "" V 4280 4100 50  0001 C CNN
@@
 Connection ~ 4050 4300
 $Comp
-L power:GND #PWR?
+L power:GND #PWR0128
 U 1 1 5C498DBE
 P 4700 4700
-F 0 "#PWR?" H 4700 4450 50  0001 C CNN
+F 0 "#PWR0128" H 4700 4450 50  0001 C CNN
 F 1 "GND" H 4705 4527 50  0000 C CNN
 F 2 "" H 4700 4700 50  0001 C CNN
@@
 	4700 4700 4700 4650
 $Comp
-L power:+3.3V #PWR?
+L power:+3.3V #PWR0124
 U 1 1 5C499E7D
 P 5400 2750
-F 0 "#PWR?" H 5400 2600 50  0001 C CNN
+F 0 "#PWR0124" H 5400 2600 50  0001 C CNN
 F 1 "+3.3V" H 5415 2923 50  0000 C CNN
 F 2 "" H 5400 2750 50  0001 C CNN
@@
 	4700 2800 4800 2800
 $Comp
-L Device:R R?
+L Device:R R50
 U 1 1 5C49B01B
 P 4800 3000
-F 0 "R?" H 4870 3046 50  0000 L CNN
+F 0 "R50" H 4870 3046 50  0000 L CNN
 F 1 "1k" H 4870 2955 50  0000 L CNN
 F 2 "" V 4730 3000 50  0001 C CNN
@@
 	4800 2800 5400 2800
 $Comp
-L Device:C C?
+L Device:C C55
 U 1 1 5C49CC52
 P 5900 2800
-F 0 "C?" H 6015 2846 50  0000 L CNN
+F 0 "C55" H 6015 2846 50  0000 L CNN
 F 1 "4.7uF" H 6015 2755 50  0000 L CNN
 F 2 "" H 5938 2650 50  0001 C CNN
@@
 NoConn ~ 6100 4400
 $Comp
-L power:+3.3V #PWR?
+L power:+3.3V #PWR0127
 U 1 1 5C4A2CBF
 P 4700 3700
-F 0 "#PWR?" H 4700 3550 50  0001 C CNN
+F 0 "#PWR0127" H 4700 3550 50  0001 C CNN
 F 1 "+3.3V" H 4715 3873 50  0000 C CNN
 F 2 "" H 4700 3700 50  0001 C CNN
@@
 	4700 3800 4900 3800
 $Comp
-L Device:C C?
+L Device:C C56
 U 1 1 5C4A4791
 P 6400 2800
-F 0 "C?" H 6515 2846 50  0000 L CNN
+F 0 "C56" H 6515 2846 50  0000 L CNN
 F 1 "0.1uF" H 6515 2755 50  0000 L CNN
 F 2 "" H 6438 2650 50  0001 C CNN
@@
 $EndComp
 $Comp
-L power:GND #PWR?
+L power:GND #PWR0125
 U 1 1 5C4A4BE4
 P 6400 3050
-F 0 "#PWR?" H 6400 2800 50  0001 C CNN
+F 0 "#PWR0125" H 6400 2800 50  0001 C CNN
 F 1 "GND" H 6405 2877 50  0000 C CNN
 F 2 "" H 6400 3050 50  0001 C CNN
@@
 	5900 2600 5600 2600
 $Comp
-L Connector_Generic:Conn_01x04 J?
+L Connector_Generic:Conn_01x04 J20
 U 1 1 5C4A7247
 P 3050 3550
-F 0 "J?" H 2970 3125 50  0000 C CNN
+F 0 "J20" H 2970 3125 50  0000 C CNN
 F 1 "USBConnector" H 2970 3216 50  0000 C CNN
 F 2 "" H 3050 3550 50  0001 C CNN
@@
 $EndComp
 $Comp
-L power:GND #PWR?
+L power:GND #PWR0126
 U 1 1 5C4A76D2
 P 3350 3700
-F 0 "#PWR?" H 3350 3450 50  0001 C CNN
+F 0 "#PWR0126" H 3350 3450 50  0001 C CNN
 F 1 "GND" H 3355 3527 50  0000 C CNN
 F 2 "" H 3350 3700 50  0001 C CNN

Commit message: Added SoC skeleton code.
Parts:
- renumbered R50 to R54, R51 to R55, R52 to R56
Changed lines of the file:
@@
 Connection ~ 3950 4200
 $Comp
-L Device:R R52
+L Device:R R56
 U 1 1 5C497DB9
 P 4700 4500
-F 0 "R52" H 4770 4546 50  0000 L CNN
+F 0 "R56" H 4770 4546 50  0000 L CNN
 F 1 "47.5k" H 4770 4455 50  0000 L CNN
 F 2 "" V 4630 4500 50  0001 C CNN
@@
 $EndComp
 $Comp
-L Device:R R51
+L Device:R R55
 U 1 1 5C497DDB
 P 4350 4100
-F 0 "R51" V 4143 4100 50  0000 C CNN
+F 0 "R55" V 4143 4100 50  0000 C CNN
 F 1 "22.1k" V 4234 4100 50  0000 C CNN
 F 2 "" V 4280 4100 50  0001 C CNN
@@
 	4700 2800 4800 2800
 $Comp
-L Device:R R50
+L Device:R R54
 U 1 1 5C49B01B
 P 4800 3000
-F 0 "R50" H 4870 3046 50  0000 L CNN
+F 0 "R54" H 4870 3046 50  0000 L CNN
 F 1 "1k" H 4870 2955 50  0000 L CNN
 F 2 "" V 4730 3000 50  0001 C CNN

Commit message: Assigned footprints to each symbol in BPS schematics.
Parts:
- C51: renamed from C55; footprint (none) -> Capacitor_SMD:C_0805_2012Metric
- C52: renamed from C56; footprint (none) -> Capacitor_SMD:C_0805_2012Metric
- J20: footprint (none) -> UTSVT_Connectors:Molex_MicroFit3.0_1x4xP3.00mm_PolarizingPeg_Vertical
- J21: footprint (none) -> Connector_USB:USB_Micro-B_Molex-105017-0001; P/N (none) -> 105017-1001
- R54, R55, R56: footprint (none) -> Resistor_SMD:R_0805_2012Metric
Changed lines of the file:
@@
 F 0 "J21" H 3000 4750 50  0000 C CNN
 F 1 "USB_B_Micro" H 3000 4650 50  0000 C CNN
-F 2 "" H 3150 4250 50  0001 C CNN
+F 2 "Connector_USB:USB_Micro-B_Molex-105017-0001" H 3150 4250 50  0001 C CNN
 F 3 "~" H 3150 4250 50  0001 C CNN
+F 4 "105017-1001" H 3000 4300 50  0001 C CNN "P/N"
 	1    3000 4300
 	1    0    0    -1
@@
 F 0 "R56" H 4770 4546 50  0000 L CNN
 F 1 "47.5k" H 4770 4455 50  0000 L CNN
-F 2 "" V 4630 4500 50  0001 C CNN
+F 2 "Resistor_SMD:R_0805_2012Metric" V 4630 4500 50  0001 C CNN
 F 3 "~" H 4700 4500 50  0001 C CNN
 	1    4700 4500
@@
 F 0 "R55" V 4143 4100 50  0000 C CNN
 F 1 "22.1k" V 4234 4100 50  0000 C CNN
-F 2 "" V 4280 4100 50  0001 C CNN
+F 2 "Resistor_SMD:R_0805_2012Metric" V 4280 4100 50  0001 C CNN
 F 3 "~" H 4350 4100 50  0001 C CNN
 	1    4350 4100
@@
 F 0 "R54" H 4870 3046 50  0000 L CNN
 F 1 "1k" H 4870 2955 50  0000 L CNN
-F 2 "" V 4730 3000 50  0001 C CNN
+F 2 "Resistor_SMD:R_0805_2012Metric" V 4730 3000 50  0001 C CNN
 F 3 "~" H 4800 3000 50  0001 C CNN
 	1    4800 3000
@@
 	4800 2800 5400 2800
 $Comp
-L Device:C C55
+L Device:C C51
 U 1 1 5C49CC52
 P 5900 2800
-F 0 "C55" H 6015 2846 50  0000 L CNN
+F 0 "C51" H 6015 2846 50  0000 L CNN
 F 1 "4.7uF" H 6015 2755 50  0000 L CNN
-F 2 "" H 5938 2650 50  0001 C CNN
+F 2 "Capacitor_SMD:C_0805_2012Metric" H 5938 2650 50  0001 C CNN
 F 3 "~" H 5900 2800 50  0001 C CNN
 	1    5900 2800
@@
 	4700 3800 4900 3800
 $Comp
-L Device:C C56
+L Device:C C52
 U 1 1 5C4A4791
 P 6400 2800
-F 0 "C56" H 6515 2846 50  0000 L CNN
+F 0 "C52" H 6515 2846 50  0000 L CNN
 F 1 "0.1uF" H 6515 2755 50  0000 L CNN
-F 2 "" H 6438 2650 50  0001 C CNN
+F 2 "Capacitor_SMD:C_0805_2012Metric" H 6438 2650 50  0001 C CNN
 F 3 "~" H 6400 2800 50  0001 C CNN
 	1    6400 2800
@@
 F 0 "J20" H 2970 3125 50  0000 C CNN
 F 1 "USBConnector" H 2970 3216 50  0000 C CNN
-F 2 "" H 3050 3550 50  0001 C CNN
+F 2 "UTSVT_Connectors:Molex_MicroFit3.0_1x4xP3.00mm_PolarizingPeg_Vertical" H 3050 3550 50  0001 C CNN
 F 3 "~" H 3050 3550 50  0001 C CNN
 	1    3050 3550

Commit message: Organized all components in BPS master to where they should be.
Parts:
- renumbered D13 to D14, R54 to R59
Changed lines of the file:
@@
 	5400 4750 5500 4750
 $Comp
-L Power_Protection:SP0503BAHT D13
+L Power_Protection:SP0503BAHT D14
 U 1 1 5C496C9B
 P 3950 4800
-F 0 "D13" H 4155 4846 50  0000 L CNN
+F 0 "D14" H 4155 4846 50  0000 L CNN
 F 1 "SP0503BAHT" H 4000 4650 50  0000 L CNN
 F 2 "Package_TO_SOT_SMD:SOT-143" H 4175 4750 50  0001 L CNN
@@
 	4700 2800 4800 2800
 $Comp
-L Device:R R54
+L Device:R R59
 U 1 1 5C49B01B
 P 4800 3000
-F 0 "R54" H 4870 3046 50  0000 L CNN
+F 0 "R59" H 4870 3046 50  0000 L CNN
 F 1 "1k" H 4870 2955 50  0000 L CNN
 F 2 "Resistor_SMD:R_0805_2012Metric" V 4730 3000 50  0001 C CNN
