File: Electronics/BPS/Master/SPI.sch (KiCad schematic (older format))
At the start: 29 parts

Commit message: Finalized schematics for BPS master.
Parts:
- removed C?: 4.7uF, symbol Device:C
- removed C?: 10uF, symbol Device:C
- removed U?: PDS2-S5-S5-M, UTSVT_ICs:PDSx-M, symbol utsvt-power-regulators:PDM2-S12-S12-S
- added C46, C47: 0.1uF, symbol Device:C
- added C48: 10uF, symbol Device:C
- added C49: CP, symbol Device:C
- added C50: 100uF, symbol Device:C
- added C51: 47uF, symbol Device:C
- added L4: 4.7uH, symbol Device:L
- added R21, R22, R23, R24, R25, R26, R27, R28, R29, R30, R31, R32, R33, R34, R35, R36, R37, R38: 50, symbol Device:R
- added TP14: +5Viso_TP, symbol Connector:TestPoint
- added TP15: GND_TP, symbol Connector:TestPoint
- added U14: SI8660EC-B-IS1, UTSVT_ICs:SOIC-16_9.9x6.0mm_P1.27mm, symbol utsvt-bps:SI8660EC-B-IS1
- added U15: PQMC3-D12-S5-S, symbol utsvt-power-regulators:PQMC3-Dx-Sx-S
- J9: renamed from J?; symbol Connector_Generic:Conn_01x06 -> Connector_Generic:Conn_02x06_Counter_Clockwise
- gave numbers to parts that had none: 25
Connections:
- net labels added: CONN10, CONN11, CONN12, CONN7, CONN8, CONN9, TEMPCS1, TEMPCS2, TEMPCS3, TEMPCS4, TEMPCS5, TEMPCS6, TEMPCS[1..6]
- net labels removed: TEMPCS, TEMP_CS, TEMP_MISO
- wire segments 170 -> 231
- no-connect marks 0 -> 6
Other:
- note added: "MISO"
- note removed: "Isolation Circuitry"
- note removed: "TODO: Make sure isolator is can correctly handle temperature boards"
- moved on the sheet: U13

Commit message: Added SoC skeleton code.
Parts:
- C36, C37, C38, C39, C40, C41, C42, C43, C44, C45, C46, C47, C48, C50: footprint (none) -> Capacitor_SMD:C_0805_2012Metric
- C49: value CP -> 100uF; footprint (none) -> Capacitor_SMD:C_0805_2012Metric
- TP14, TP15: footprint (none) -> TestPoint:TestPoint_Keystone_5005-5009_Compact
- U15: footprint (none) -> UTSVT_ICs:CUI_PQMC3-S
- renumbered R13 to R15, R14 to R16, R15 to R17, R16 to R18, R17 to R19, R18 to R20, R19 to R21, R20 to R22, R21 to R23, R22 to R24, R23 to R25, R24 to R26, R25 to R27, R26 to R28, R27 to R29, R28 to R30, R29 to R31, R30 to R32, R31 to R33, R32 to R34, R33 to R35, R34 to R36, R35 to R37, R36 to R38, R37 to R39, R38 to R40

Commit message: Assigned footprints to each symbol in BPS schematics.
Parts:
- removed C48: 10uF, Capacitor_SMD:C_0805_2012Metric, symbol Device:C
- removed C49, C50: 100uF, Capacitor_SMD:C_0805_2012Metric, symbol Device:C
- removed C51: 47uF, symbol Device:C
- removed TP14: +5Viso_TP, TestPoint:TestPoint_Keystone_5005-5009_Compact, symbol Connector:TestPoint
- removed TP15: GND_TP, TestPoint:TestPoint_Keystone_5005-5009_Compact, symbol Connector:TestPoint
- removed U15: PQMC3-D12-S5-S, UTSVT_ICs:CUI_PQMC3-S, symbol utsvt-power-regulators:PQMC3-Dx-Sx-S
- added C46: 470pF, Capacitor_SMD:C_2220_5650Metric, symbol Device:C
- added C47: 4.7uF, Capacitor_SMD:C_0805_2012Metric, symbol Device:C
- added U15: RI3-1205S, UTSVT_ICs:RI3_DC_Converter, symbol utsvt-power-regulators:RI3-1205S
- J10: footprint (none) -> Connector_PinHeader_2.54mm:PinHeader_2x03_P2.54mm_Vertical
- J7: footprint (none) -> UTSVT_Connectors:Molex_MicroFit3.0_1x2xP3.00mm_PolarizingPeg_Vertical
- J8: footprint (none) -> UTSVT_Connectors:Molex_MicroFit3.0_1x4xP3.00mm_PolarizingPeg_Vertical
- J9: footprint (none) -> UTSVT_Connectors:Molex_MicroFit3.0_2x6xP3.00mm_PolarizingPeg_Vertical
- L4: value 4.7uH -> 10uH; footprint (none) -> Inductor_SMD:L_0805_2012Metric
- R15, R16, R17, R18, R19, R20, R21, R22, R23, R24, R25, R26, R27, R28, R29, R30, R31, R32, R33, R34, R35, R36, R37, R38, R39, R40: footprint (none) -> Resistor_SMD:R_0805_2012Metric
- U10, U12: footprint (none) -> Package_SO:MSOP-16_3x4mm_P0.5mm
- U11: footprint (none) -> UTSVT_BPS:HXXXX
- U14: footprint UTSVT_ICs:SOIC-16_9.9x6.0mm_P1.27mm -> Package_SO:SOIC-16_3.9x9.9mm_P1.27mm
- renumbered C36 to C34, C37 to C35, C38 to C36, C39 to C37, C40 to C38, C41 to C39, C42 to C40, C43 to C41, C44 to C42, C45 to C43, C46 to C44, C47 to C45
Connections:
- wire segments 231 -> 223
- no-connect marks 6 -> 5
Other:
- note added: "This regulator is to power the Temperature slave boards."

Commit message: Organized all components in BPS master to where they should be.
Parts:
- J10: symbol Connector_Generic:Conn_02x03_Top_Bottom -> Connector_Generic:Conn_02x03_Odd_Even
Connections:
- wire segments 223 -> 225
- no-connect marks 5 -> 4
Changed lines of the file:
@@
 L Connector_Generic:Conn_01x04 J8
 U 1 1 5C5232C7
-P 10450 2350
-F 0 "J8" H 10530 2342 50  0000 L CNN
-F 1 "DisplayConnector" H 10530 2251 50  0000 L CNN
-F 2 "UTSVT_Connectors:Molex_MicroFit3.0_1x4xP3.00mm_PolarizingPeg_Vertical" H 10450 2350 50  0001 C CNN
-F 3 "~" H 10450 2350 50  0001 C CNN
-	1    10450 2350
+P 10450 2550
+F 0 "J8" H 10530 2542 50  0000 L CNN
+F 1 "DisplayConnector" H 10530 2451 50  0000 L CNN
+F 2 "UTSVT_Connectors:Molex_MicroFit3.0_1x4xP3.00mm_PolarizingPeg_Vertical" H 10450 2550 50  0001 C CNN
+F 3 "~" H 10450 2550 50  0001 C CNN
+	1    10450 2550
 	1    0    0    -1
 $EndComp
@@
 L power:+12V #PWR076
 U 1 1 5C635F56
-P 10150 2150
-F 0 "#PWR076" H 10150 2000 50  0001 C CNN
-F 1 "+12V" H 10165 2323 50  0000 C CNN
-F 2 "" H 10150 2150 50  0001 C CNN
-F 3 "" H 10150 2150 50  0001 C CNN
-	1    10150 2150
-	1    0    0    -1
-$EndComp
-Wire Wire Line
-	10150 2150 10150 2250
-Wire Wire Line
-	10150 2250 10250 2250
-Wire Wire Line
-	10250 2350 10150 2350
-Wire Wire Line
-	10150 2350 10150 2650
-$Comp
-L Connector_Generic:Conn_02x03_Top_Bottom J10
+P 10150 2350
+F 0 "#PWR076" H 10150 2200 50  0001 C CNN
+F 1 "+12V" H 10165 2523 50  0000 C CNN
+F 2 "" H 10150 2350 50  0001 C CNN
+F 3 "" H 10150 2350 50  0001 C CNN
+	1    10150 2350
+	1    0    0    -1
+$EndComp
+Wire Wire Line
+	10250 2750 10150 2750
+Wire Wire Line
+	10150 2750 10150 2850
+$Comp
+L Connector_Generic:Conn_02x03_Odd_Even J10
 U 1 1 5C31CB2C
 P 3650 5700
@@
 L power:GNDPWR #PWR080
 U 1 1 5C3FDE53
-P 10150 2650
-F 0 "#PWR080" H 10150 2450 50  0001 C CNN
-F 1 "GNDPWR" H 10154 2496 50  0000 C CNN
-F 2 "" H 10150 2600 50  0001 C CNN
-F 3 "" H 10150 2600 50  0001 C CNN
-	1    10150 2650
+P 10150 2850
+F 0 "#PWR080" H 10150 2650 50  0001 C CNN
+F 1 "GNDPWR" H 10154 2696 50  0000 C CNN
+F 2 "" H 10150 2800 50  0001 C CNN
+F 3 "" H 10150 2800 50  0001 C CNN
+	1    10150 2850
 	1    0    0    -1
 $EndComp
@@
 NoConn ~ 9400 1900
 NoConn ~ 9400 2300
-NoConn ~ 9600 4250
 NoConn ~ 8400 4150
 NoConn ~ 7600 4150
@@
 Wire Wire Line
 	9500 2550 10250 2550
+Wire Wire Line
+	10150 2650 10250 2650
+Wire Wire Line
+	10150 2350 10150 2650
+Wire Wire Line
+	9500 4350 9500 4250
+Wire Wire Line
+	9500 4250 9600 4250
+Connection ~ 9500 4350
 Wire Bus Line
 	6350 5400 6350 6000

Commit message: Added more traces to master BPS.
Connections:
- net labels added: CS1, CS2, CS3, CS4, CS5, CS6
- net labels removed: CONN10, CONN11, CONN12, CONN7, CONN8, CONN9
Changed lines of the file:
@@
 	8600 5300 8500 5300
 Wire Wire Line
-	9550 5400 9100 5400
+	9550 5900 9100 5900
 $Comp
 L utsvt-bps:GND_A #PWR088
@@
 $EndComp
 Wire Wire Line
-	9550 5700 9100 5700
-Wire Wire Line
-	9550 5800 9100 5800
-Wire Wire Line
-	9550 5900 9100 5900
+	9550 5600 9100 5600
+Wire Wire Line
+	9550 5500 9100 5500
+Wire Wire Line
+	9550 5400 9100 5400
+Text Label 9550 5900 2    50   ~ 0
+CS6
+Text Label 9550 5800 2    50   ~ 0
+CS5
+Text Label 9550 5700 2    50   ~ 0
+CS4
+Text Label 9550 5600 2    50   ~ 0
+CS3
+Text Label 9550 5500 2    50   ~ 0
+CS2
 Text Label 9550 5400 2    50   ~ 0
-CONN7
-Text Label 9550 5500 2    50   ~ 0
-CONN8
-Text Label 9550 5600 2    50   ~ 0
-CONN9
-Text Label 9550 5700 2    50   ~ 0
-CONN10
-Text Label 9550 5800 2    50   ~ 0
-CONN11
-Text Label 9550 5900 2    50   ~ 0
-CONN12
-Wire Wire Line
-	10550 4350 10100 4350
-Wire Wire Line
-	10550 4250 10100 4250
-Wire Wire Line
-	10550 4150 10100 4150
-Wire Wire Line
-	10550 4050 10100 4050
-Wire Wire Line
-	10550 3950 10100 3950
-Wire Wire Line
-	10550 3850 10100 3850
-Text Label 10550 4350 2    50   ~ 0
-CONN7
-Text Label 10550 4250 2    50   ~ 0
-CONN8
-Text Label 10550 4150 2    50   ~ 0
-CONN9
-Text Label 10550 4050 2    50   ~ 0
-CONN10
-Text Label 10550 3950 2    50   ~ 0
-CONN11
-Text Label 10550 3850 2    50   ~ 0
-CONN12
+CS1
 Text Notes 9600 4150 2    50   ~ 0
 MISO
@@
 $EndComp
 Wire Wire Line
-	9550 5600 9100 5600
-Wire Wire Line
-	9550 5500 9100 5500
+	9550 5700 9100 5700
+Wire Wire Line
+	9550 5800 9100 5800
 Wire Wire Line
 	8500 5400 8800 5400
@@
 	9500 4250 9600 4250
 Connection ~ 9500 4350
+Wire Wire Line
+	10550 4350 10100 4350
+Wire Wire Line
+	10550 4050 10100 4050
+Wire Wire Line
+	10550 3950 10100 3950
+Wire Wire Line
+	10550 3850 10100 3850
+Text Label 10550 4350 2    50   ~ 0
+CS6
+Text Label 10550 4250 2    50   ~ 0
+CS5
+Text Label 10550 4150 2    50   ~ 0
+CS4
+Text Label 10550 4050 2    50   ~ 0
+CS3
+Text Label 10550 3950 2    50   ~ 0
+CS2
+Text Label 10550 3850 2    50   ~ 0
+CS1
+Wire Wire Line
+	10550 4150 10100 4150
+Wire Wire Line
+	10550 4250 10100 4250
 Wire Bus Line
 	6350 5400 6350 6000
