File: Electronics/BPS/Master/BPSMaster.sch (KiCad schematic (older format))
At the start: 32 parts

Commit message: Finalized schematics for BPS master.
Parts:
- removed D?: Heartbeat, symbol Device:LED_ALT
- removed D?: Fault, symbol Device:LED_ALT
- removed D?: OVolt, symbol Device:LED_ALT
- removed D?: UVolt, symbol Device:LED_ALT
- removed D?: OTemp, symbol Device:LED_ALT
- removed D?: OCurr, symbol Device:LED_ALT
- removed D?: WDError, symbol Device:LED_ALT
- removed R?: 680, symbol Device:R
- removed R? (x6): 750, symbol Device:R
- added C12: 0.1uF, symbol Device:C
- added J3: CurrentSlaveConnector, symbol Connector_Generic:Conn_01x04
- added MH1, MH2, MH3, MH4: MountingHole, symbol Mechanical:MountingHole
- gave numbers to parts that had none: 18
Connections:
- net labels added: PA5, PA6, PA[5..6], PC[0..5], TEMP_CS1, TEMP_CS2, TEMP_CS3, TEMP_CS4, TEMP_CS5, TEMP_CS6, TEMP_CS[1..6]
- net labels removed: LTC2983_CS, OSC32_IN, OSC32_OUT, VCAP_1
- wire segments 194 -> 187
- no-connect marks 0 -> 18
Other:
- note added: "- Display\n- Volt Slave\n- Temp Slave"
- note added: "- EEPROM\n- IMU"
- note added: "Bypass Capacitors"
- note added: "Current Board"
- note added: "Debug"
- note removed: "Green LEDs good"
- note removed: "Red LEDs fault"
- moved on the sheet: U1

Commit message: Added SoC skeleton code.
Parts:
- C1, C10, C11, C12, C13, C14, C2, C3, C4, C5, C6, C7, C8, C9: footprint (none) -> Capacitor_SMD:C_0805_2012Metric
Changed lines of the file:
@@
 F 0 "C1" H 8065 1796 50  0000 L CNN
 F 1 "0.1uF" H 8065 1705 50  0000 L CNN
-F 2 "" H 7988 1600 50  0001 C CNN
+F 2 "Capacitor_SMD:C_0805_2012Metric" H 7988 1600 50  0001 C CNN
 F 3 "~" H 7950 1750 50  0001 C CNN
 	1    7950 1750
@@
 F 0 "C2" H 8515 1796 50  0000 L CNN
 F 1 "0.1uF" H 8515 1705 50  0000 L CNN
-F 2 "" H 8438 1600 50  0001 C CNN
+F 2 "Capacitor_SMD:C_0805_2012Metric" H 8438 1600 50  0001 C CNN
 F 3 "~" H 8400 1750 50  0001 C CNN
 	1    8400 1750
@@
 F 0 "C3" H 8965 1796 50  0000 L CNN
 F 1 "0.1uF" H 8965 1705 50  0000 L CNN
-F 2 "" H 8888 1600 50  0001 C CNN
+F 2 "Capacitor_SMD:C_0805_2012Metric" H 8888 1600 50  0001 C CNN
 F 3 "~" H 8850 1750 50  0001 C CNN
 	1    8850 1750
@@
 F 0 "C4" H 9415 1796 50  0000 L CNN
 F 1 "0.1uF" H 9415 1705 50  0000 L CNN
-F 2 "" H 9338 1600 50  0001 C CNN
+F 2 "Capacitor_SMD:C_0805_2012Metric" H 9338 1600 50  0001 C CNN
 F 3 "~" H 9300 1750 50  0001 C CNN
 	1    9300 1750
@@
 F 0 "C5" H 9865 1796 50  0000 L CNN
 F 1 "0.1uF" H 9865 1705 50  0000 L CNN
-F 2 "" H 9788 1600 50  0001 C CNN
+F 2 "Capacitor_SMD:C_0805_2012Metric" H 9788 1600 50  0001 C CNN
 F 3 "~" H 9750 1750 50  0001 C CNN
 	1    9750 1750
@@
 F 0 "C6" H 10315 1796 50  0000 L CNN
 F 1 "0.1uF" H 10315 1705 50  0000 L CNN
-F 2 "" H 10238 1600 50  0001 C CNN
+F 2 "Capacitor_SMD:C_0805_2012Metric" H 10238 1600 50  0001 C CNN
 F 3 "~" H 10200 1750 50  0001 C CNN
 	1    10200 1750
@@
 F 0 "C7" H 10768 1796 50  0000 L CNN
 F 1 "4.7uF" H 10768 1705 50  0000 L CNN
-F 2 "" H 10688 1600 50  0001 C CNN
+F 2 "Capacitor_SMD:C_0805_2012Metric" H 10688 1600 50  0001 C CNN
 F 3 "~" H 10650 1750 50  0001 C CNN
 	1    10650 1750
@@
 F 0 "C9" H 8065 2946 50  0000 L CNN
 F 1 "0.1uF" H 8065 2855 50  0000 L CNN
-F 2 "" H 7988 2750 50  0001 C CNN
+F 2 "Capacitor_SMD:C_0805_2012Metric" H 7988 2750 50  0001 C CNN
 F 3 "~" H 7950 2900 50  0001 C CNN
 	1    7950 2900
@@
 F 0 "C10" H 8518 2946 50  0000 L CNN
 F 1 "1uF" H 8518 2855 50  0000 L CNN
-F 2 "" H 8438 2750 50  0001 C CNN
+F 2 "Capacitor_SMD:C_0805_2012Metric" H 8438 2750 50  0001 C CNN
 F 3 "~" H 8400 2900 50  0001 C CNN
 	1    8400 2900
@@
 F 0 "C8" H 4868 2596 50  0000 L CNN
 F 1 "2.2uF" H 4868 2505 50  0000 L CNN
-F 2 "" H 4788 2400 50  0001 C CNN
+F 2 "Capacitor_SMD:C_0805_2012Metric" H 4788 2400 50  0001 C CNN
 F 3 "~" H 4750 2550 50  0001 C CNN
 F 4 "Low ESR <1Ohm" H 4750 2550 50  0001 C CNN "Note"
@@
 F3 "CONTACTOR_EN" I R 2000 2950 50
 F4 "GND" I R 2000 3150 50
-F5 "+3.3V" I R 2000 2850 50
+F5 "+5V" I R 2000 2850 50
 $EndSheet
 $Comp
@@
 Wire Wire Line
 	2400 1900 2400 1950
-$Comp
-L power:+5V #PWR06
-U 1 1 5C2FEA74
-P 2200 1800
-F 0 "#PWR06" H 2200 1650 50  0001 C CNN
-F 1 "+5V" H 2215 1973 50  0000 C CNN
-F 2 "" H 2200 1800 50  0001 C CNN
-F 3 "" H 2200 1800 50  0001 C CNN
-	1    2200 1800
-	1    0    0    -1
-$EndComp
-Wire Wire Line
-	2000 1850 2200 1850
-Wire Wire Line
-	2200 1850 2200 1800
 Wire Wire Line
 	2000 1950 2400 1950
@@
 F 0 "C11" H 9215 2946 50  0000 L CNN
 F 1 "0.1uF" H 9215 2855 50  0000 L CNN
-F 2 "" H 9138 2750 50  0001 C CNN
+F 2 "Capacitor_SMD:C_0805_2012Metric" H 9138 2750 50  0001 C CNN
 F 3 "~" H 9100 2900 50  0001 C CNN
 	1    9100 2900
@@
 F 0 "C14" H 4465 5746 50  0000 L CNN
 F 1 "6pF" H 4465 5655 50  0000 L CNN
-F 2 "" H 4388 5550 50  0001 C CNN
+F 2 "Capacitor_SMD:C_0805_2012Metric" H 4388 5550 50  0001 C CNN
 F 3 "~" H 4350 5700 50  0001 C CNN
 	1    4350 5700
@@
 F 0 "C13" H 4065 5746 50  0000 L CNN
 F 1 "6pF" H 4065 5655 50  0000 L CNN
-F 2 "" H 3988 5550 50  0001 C CNN
+F 2 "Capacitor_SMD:C_0805_2012Metric" H 3988 5550 50  0001 C CNN
 F 3 "~" H 3950 5700 50  0001 C CNN
 	1    3950 5700
@@
 Connection ~ 4350 5350
 $Comp
-L power:GND #PWR029
+L power:GND #PWR028
 U 1 1 5C3D1383
 P 3950 5950
-F 0 "#PWR029" H 3950 5700 50  0001 C CNN
+F 0 "#PWR028" H 3950 5700 50  0001 C CNN
 F 1 "GND" H 3955 5777 50  0000 C CNN
 F 2 "" H 3950 5950 50  0001 C CNN
@@
 F3 "PC[0..5]" I R 2000 7150 50
 F4 "PA[5..6]" I R 2000 7250 50
-F5 "+3.3V" I R 2000 7050 50
+F5 "+5V" I R 2000 7050 50
 $EndSheet
 $Comp
@@
 	2200 6350 2000 6350
 $Comp
-L power:+3.3V #PWR028
+L power:+3.3V #PWR029
 U 1 1 5C4686E9
 P 2200 6000
-F 0 "#PWR028" H 2200 5850 50  0001 C CNN
+F 0 "#PWR029" H 2200 5850 50  0001 C CNN
 F 1 "+3.3V" H 2215 6173 50  0000 C CNN
 F 2 "" H 2200 6000 50  0001 C CNN
@@
 PA[5..6]
 $Comp
-L power:+3.3V #PWR013
-U 1 1 5C9589A8
-P 2200 2800
-F 0 "#PWR013" H 2200 2650 50  0001 C CNN
-F 1 "+3.3V" H 2215 2973 50  0000 C CNN
-F 2 "" H 2200 2800 50  0001 C CNN
-F 3 "" H 2200 2800 50  0001 C CNN
-	1    2200 2800
-	1    0    0    -1
-$EndComp
-Wire Wire Line
-	2200 2800 2200 2850
-Wire Wire Line
-	2200 2850 2000 2850
-$Comp
-L power:+3.3V #PWR031
-U 1 1 5C9F1E26
-P 2200 7000
-F 0 "#PWR031" H 2200 6850 50  0001 C CNN
-F 1 "+3.3V" H 2215 7173 50  0000 C CNN
-F 2 "" H 2200 7000 50  0001 C CNN
-F 3 "" H 2200 7000 50  0001 C CNN
-	1    2200 7000
-	1    0    0    -1
-$EndComp
-Wire Wire Line
-	2200 7000 2200 7050
-Wire Wire Line
-	2200 7050 2000 7050
-$Comp
 L Mechanical:MountingHole MH1
 U 1 1 5C9FCF93
@@
 F 0 "C12" V 8600 5550 50  0000 L CNN
 F 1 "0.1uF" V 8700 5400 50  0000 L CNN
-F 2 "" H 8538 5300 50  0001 C CNN
+F 2 "Capacitor_SMD:C_0805_2012Metric" H 8538 5300 50  0001 C CNN
 F 3 "~" H 8500 5450 50  0001 C CNN
 	1    8500 5450
@@
 NoConn ~ 8400 4600
 $Comp
-L power:PWR_FLAG #FLG0102
+L power:PWR_FLAG #FLG01
 U 1 1 5CC7D7CD
 P 4700 2350
-F 0 "#FLG0102" H 4700 2425 50  0001 C CNN
+F 0 "#FLG01" H 4700 2425 50  0001 C CNN
 F 1 "PWR_FLAG" V 4700 2478 50  0000 L CNN
 F 2 "" H 4700 2350 50  0001 C CNN
@@
 Wire Wire Line
 	4700 2350 4750 2350
+Connection ~ 4750 2350
+Wire Wire Line
+	2200 1850 2200 1800
+Wire Wire Line
+	2000 1850 2200 1850
+$Comp
+L power:+5V #PWR06
+U 1 1 5C2FEA74
+P 2200 1800
+F 0 "#PWR06" H 2200 1650 50  0001 C CNN
+F 1 "+5V" H 2215 1973 50  0000 C CNN
+F 2 "" H 2200 1800 50  0001 C CNN
+F 3 "" H 2200 1800 50  0001 C CNN
+	1    2200 1800
+	1    0    0    -1
+$EndComp
+Wire Wire Line
+	2200 2850 2200 2800
+Wire Wire Line
+	2000 2850 2200 2850
+$Comp
+L power:+5V #PWR013
+U 1 1 5C3D9395
+P 2200 2800
+F 0 "#PWR013" H 2200 2650 50  0001 C CNN
+F 1 "+5V" H 2215 2973 50  0000 C CNN
+F 2 "" H 2200 2800 50  0001 C CNN
+F 3 "" H 2200 2800 50  0001 C CNN
+	1    2200 2800
+	1    0    0    -1
+$EndComp
+Wire Wire Line
+	2200 7050 2200 7000
+Wire Wire Line
+	2000 7050 2200 7050
+$Comp
+L power:+5V #PWR031
+U 1 1 5C3EEFA7
+P 2200 7000
+F 0 "#PWR031" H 2200 6850 50  0001 C CNN
+F 1 "+5V" H 2215 7173 50  0000 C CNN
+F 2 "" H 2200 7000 50  0001 C CNN
+F 3 "" H 2200 7000 50  0001 C CNN
+	1    2200 7000
+	1    0    0    -1
+$EndComp
 Wire Bus Line
 	7000 2250 7000 2450
@@
 Wire Bus Line
 	7000 4250 7000 4850
-Connection ~ 4750 2350
 $EndSCHEMATC

Commit message: Assigned footprints to each symbol in BPS schematics.
Parts:
- J1: footprint (none) -> Connector_PinHeader_2.54mm:PinHeader_1x03_P2.54mm_Vertical
- J2: footprint (none) -> Connector_PinHeader_2.54mm:PinHeader_2x07_P2.54mm_Vertical
- J3: footprint (none) -> UTSVT_Connectors:Molex_MicroFit3.0_1x4xP3.00mm_PolarizingPeg_Vertical
- MH1, MH2, MH3, MH4: footprint (none) -> MountingHole:MountingHole_3mm
Changed lines of the file:
@@
 F3 "CAN_RX" O R 2000 2150 50
 F4 "GND" I R 2000 2250 50
-F5 "+5V" I R 2000 1850 50
-F6 "+3.3V" I R 2000 1950 50
+F5 "+3.3V" I R 2000 1950 50
+F6 "+5V" I R 2000 1850 50
 $EndSheet
 $Comp
@@
 F 0 "J2" H 8650 4817 50  0000 C CNN
 F 1 "Logic Analyzer" H 8650 4726 50  0000 C CNN
-F 2 "" H 8600 4300 50  0001 C CNN
+F 2 "Connector_PinHeader_2.54mm:PinHeader_2x07_P2.54mm_Vertical" H 8600 4300 50  0001 C CNN
 F 3 "~" H 8600 4300 50  0001 C CNN
 	1    8600 4300
@@
 F 0 "J1" H 11050 2700 50  0000 R CNN
 F 1 "SWD" H 11100 2800 50  0000 R CNN
-F 2 "" H 10850 2800 50  0001 C CNN
+F 2 "Connector_PinHeader_2.54mm:PinHeader_1x03_P2.54mm_Vertical" H 10850 2800 50  0001 C CNN
 F 3 "~" H 10850 2800 50  0001 C CNN
 	1    10850 2800
@@
 F 0 "MH1" H 10400 3996 50  0000 L CNN
 F 1 "MountingHole" H 10400 3905 50  0000 L CNN
-F 2 "" H 10300 3950 50  0001 C CNN
+F 2 "MountingHole:MountingHole_3mm" H 10300 3950 50  0001 C CNN
 F 3 "~" H 10300 3950 50  0001 C CNN
 	1    10300 3950
@@
 F 0 "MH2" H 10400 4246 50  0000 L CNN
 F 1 "MountingHole" H 10400 4155 50  0000 L CNN
-F 2 "" H 10300 4200 50  0001 C CNN
+F 2 "MountingHole:MountingHole_3mm" H 10300 4200 50  0001 C CNN
 F 3 "~" H 10300 4200 50  0001 C CNN
 	1    10300 4200
@@
 F 0 "MH3" H 10400 4496 50  0000 L CNN
 F 1 "MountingHole" H 10400 4405 50  0000 L CNN
-F 2 "" H 10300 4450 50  0001 C CNN
+F 2 "MountingHole:MountingHole_3mm" H 10300 4450 50  0001 C CNN
 F 3 "~" H 10300 4450 50  0001 C CNN
 	1    10300 4450
@@
 F 0 "MH4" H 10400 4746 50  0000 L CNN
 F 1 "MountingHole" H 10400 4655 50  0000 L CNN
-F 2 "" H 10300 4700 50  0001 C CNN
+F 2 "MountingHole:MountingHole_3mm" H 10300 4700 50  0001 C CNN
 F 3 "~" H 10300 4700 50  0001 C CNN
 	1    10300 4700
@@
 F 0 "J3" H 9029 5542 50  0000 L CNN
 F 1 "CurrentSlaveConnector" H 9029 5451 50  0000 L CNN
-F 2 "" H 8950 5550 50  0001 C CNN
+F 2 "UTSVT_Connectors:Molex_MicroFit3.0_1x4xP3.00mm_PolarizingPeg_Vertical" H 8950 5550 50  0001 C CNN
 F 3 "~" H 8950 5550 50  0001 C CNN
 	1    8950 5550
@@
 Wire Wire Line
 	8750 5550 8300 5550
-$Comp
-L power:+5V #PWR025
-U 1 1 5CA531CB
-P 8700 5350
-F 0 "#PWR025" H 8700 5200 50  0001 C CNN
-F 1 "+5V" H 8715 5523 50  0000 C CNN
-F 2 "" H 8700 5350 50  0001 C CNN
-F 3 "" H 8700 5350 50  0001 C CNN
-	1    8700 5350
-	1    0    0    -1
-$EndComp
 Wire Wire Line
 	8700 5350 8700 5450
@@
 Wire Bus Line
 	7000 4250 7000 4850
+$Comp
+L power:+5V #PWR0134
+U 1 1 5C4C0F65
+P 8700 5350
+F 0 "#PWR0134" H 8700 5200 50  0001 C CNN
+F 1 "+5V" H 8715 5523 50  0000 C CNN
+F 2 "" H 8700 5350 50  0001 C CNN
+F 3 "" H 8700 5350 50  0001 C CNN
+	1    8700 5350
+	1    0    0    -1
+$EndComp
 $EndSCHEMATC

Commit message: Master board PCB layout organized.
Parts:
- added C53, C54: 1uF, Capacitor_SMD:C_0805_2012Metric, symbol Device:C
- added R57, R58: 220k, Resistor_SMD:R_0805_2012Metric, symbol Device:R
Connections:
- wire segments 187 -> 197
Changed lines of the file:
@@
 Text Label 6900 2250 2    50   ~ 0
 ADC1_CH3
-Text Notes 8050 6050 0    50   ~ 0
+Text Notes 8500 6050 0    50   ~ 0
 PA2 high precision hall effect sensor.\nPA3 low precision hall effect sensor.
 $Sheet
@@
 Current Board
 Wire Wire Line
-	8750 5650 8250 5650
-Wire Wire Line
-	8750 5750 8250 5750
-Text Label 8250 5650 0    50   ~ 0
+	8750 5650 8550 5650
+Wire Wire Line
+	8750 5750 8550 5750
+Text Label 7350 5650 0    50   ~ 0
 ADC1_CH2
-Text Label 8250 5750 0    50   ~ 0
+Text Label 7350 5750 0    50   ~ 0
 ADC1_CH3
 Wire Wire Line
@@
 	1    0    0    -1
 $EndComp
-Wire Bus Line
-	7000 2250 7000 2450
-Wire Bus Line
-	4400 3350 4400 3950
-Wire Bus Line
-	7000 4250 7000 4850
 $Comp
 L power:+5V #PWR0134
@@
 	1    0    0    -1
 $EndComp
+$Comp
+L Device:R R58
+U 1 1 5C83A7AA
+P 8400 5750
+F 0 "R58" V 8450 5950 50  0000 C CNN
+F 1 "220k" V 8400 5750 50  0000 C CNN
+F 2 "Resistor_SMD:R_0805_2012Metric" V 8330 5750 50  0001 C CNN
+F 3 "~" H 8400 5750 50  0001 C CNN
+	1    8400 5750
+	0    1    1    0
+$EndComp
+$Comp
+L Device:R R57
+U 1 1 5C845E9E
+P 8400 5650
+F 0 "R57" V 8450 5850 50  0000 C CNN
+F 1 "220k" V 8400 5650 50  0000 C CNN
+F 2 "Resistor_SMD:R_0805_2012Metric" V 8330 5650 50  0001 C CNN
+F 3 "~" H 8400 5650 50  0001 C CNN
+	1    8400 5650
+	0    1    1    0
+$EndComp
+Wire Wire Line
+	8250 5650 7800 5650
+Wire Wire Line
+	7350 5750 8150 5750
+$Comp
+L Device:C C54
+U 1 1 5C868333
+P 8150 6000
+F 0 "C54" H 8265 6046 50  0000 L CNN
+F 1 "1uF" H 8265 5955 50  0000 L CNN
+F 2 "Capacitor_SMD:C_0805_2012Metric" H 8188 5850 50  0001 C CNN
+F 3 "~" H 8150 6000 50  0001 C CNN
+	1    8150 6000
+	1    0    0    -1
+$EndComp
+Wire Wire Line
+	8150 5850 8150 5750
+Connection ~ 8150 5750
+Wire Wire Line
+	8150 5750 8250 5750
+$Comp
+L Device:C C53
+U 1 1 5C873D8D
+P 7800 6000
+F 0 "C53" H 7915 6046 50  0000 L CNN
+F 1 "1uF" H 7915 5955 50  0000 L CNN
+F 2 "Capacitor_SMD:C_0805_2012Metric" H 7838 5850 50  0001 C CNN
+F 3 "~" H 7800 6000 50  0001 C CNN
+	1    7800 6000
+	1    0    0    -1
+$EndComp
+Wire Wire Line
+	7800 5850 7800 5650
+Connection ~ 7800 5650
+Wire Wire Line
+	7800 5650 7350 5650
+$Comp
+L power:GND #PWR0138
+U 1 1 5C896080
+P 8150 6250
+F 0 "#PWR0138" H 8150 6000 50  0001 C CNN
+F 1 "GND" H 8250 6100 50  0000 R CNN
+F 2 "" H 8150 6250 50  0001 C CNN
+F 3 "" H 8150 6250 50  0001 C CNN
+	1    8150 6250
+	1    0    0    -1
+$EndComp
+Wire Wire Line
+	8150 6250 8150 6200
+Wire Wire Line
+	8150 6200 7800 6200
+Wire Wire Line
+	7800 6200 7800 6150
+Connection ~ 8150 6200
+Wire Wire Line
+	8150 6200 8150 6150
+Wire Bus Line
+	7000 2250 7000 2450
+Wire Bus Line
+	4400 3350 4400 3950
+Wire Bus Line
+	7000 4250 7000 4850
 $EndSCHEMATC
