File: Electronics/BPS/Master/BPSMaster.sch (KiCad schematic (older format))
At the start: 28 parts, among them J1 SWD, J2 Logic Analyzer, J3 CurrentSlaveConnector, SW1 B3SL-1002P, U1 STM32F413RHTx, Y1 NX8045GB-8.000M-STD-CSJ-1

Commit message: Organized all components in BPS master to where they should be.
Connections:
- net labels added: FAULT, PA7, PA[5..7], PB0, PB1, RUN
- net labels removed: PA[5..6], PC6, PC7
- wire segments 197 -> 208
- no-connect marks 18 -> 14
Changed lines of the file:
@@
 UART1_RX
 Wire Wire Line
-	6400 3050 6900 3050
-Text Label 6900 3050 2    50   ~ 0
+	6400 4450 6900 4450
+Text Label 6900 4450 2    50   ~ 0
 CAN1_RX
 Wire Wire Line
-	6400 3150 6900 3150
-Text Label 6900 3150 2    50   ~ 0
+	6400 4550 6900 4550
+Text Label 6900 4550 2    50   ~ 0
 CAN1_TX
 Wire Wire Line
@@
 I2C3_SCL
 Wire Wire Line
-	5000 4150 4500 4150
-Wire Wire Line
-	4500 4250 5000 4250
-Text Label 4500 4150 0    50   ~ 0
-PC6
-Text Label 4500 4250 0    50   ~ 0
-PC7
+	6400 3650 6900 3650
+Wire Wire Line
+	6900 3750 6400 3750
+Text Label 6900 3650 2    50   ~ 0
+PB0
+Text Label 6900 3750 2    50   ~ 0
+PB1
 Wire Wire Line
 	2000 2150 2500 2150
@@
 L Device:Crystal Y1
 U 1 1 5C3BE613
-P 4150 5350
-F 0 "Y1" H 4150 5618 50  0000 C CNN
-F 1 "NX8045GB-8.000M-STD-CSJ-1" H 4150 5527 50  0000 C CNN
-F 2 "UTSVT_BPS:NX8045GB-8.000M-STD-CSJ-1" H 4150 5350 50  0001 C CNN
-F 3 "~" H 4150 5350 50  0001 C CNN
-	1    4150 5350
-	1    0    0    -1
-$EndComp
-Wire Wire Line
-	4000 5350 3950 5350
-Wire Wire Line
-	4300 5350 4350 5350
+P 4150 5500
+F 0 "Y1" H 4150 5768 50  0000 C CNN
+F 1 "NX8045GB-8.000M-STD-CSJ-1" H 4150 5677 50  0000 C CNN
+F 2 "UTSVT_BPS:NX8045GB-8.000M-STD-CSJ-1" H 4150 5500 50  0001 C CNN
+F 3 "~" H 4150 5500 50  0001 C CNN
+	1    4150 5500
+	1    0    0    -1
+$EndComp
+Wire Wire Line
+	4000 5500 3950 5500
+Wire Wire Line
+	4300 5500 4350 5500
 $Comp
 L Device:C C14
 U 1 1 5C3C7C2B
-P 4350 5700
-F 0 "C14" H 4465 5746 50  0000 L CNN
-F 1 "6pF" H 4465 5655 50  0000 L CNN
-F 2 "Capacitor_SMD:C_0805_2012Metric" H 4388 5550 50  0001 C CNN
-F 3 "~" H 4350 5700 50  0001 C CNN
-	1    4350 5700
+P 4350 5850
+F 0 "C14" H 4465 5896 50  0000 L CNN
+F 1 "6pF" H 4465 5805 50  0000 L CNN
+F 2 "Capacitor_SMD:C_0805_2012Metric" H 4388 5700 50  0001 C CNN
+F 3 "~" H 4350 5850 50  0001 C CNN
+	1    4350 5850
 	1    0    0    -1
 $EndComp
@@
 L Device:C C13
 U 1 1 5C3C7D18
-P 3950 5700
-F 0 "C13" H 4065 5746 50  0000 L CNN
-F 1 "6pF" H 4065 5655 50  0000 L CNN
-F 2 "Capacitor_SMD:C_0805_2012Metric" H 3988 5550 50  0001 C CNN
-F 3 "~" H 3950 5700 50  0001 C CNN
-	1    3950 5700
-	1    0    0    -1
-$EndComp
-Wire Wire Line
-	4350 5350 4350 5550
-Connection ~ 4350 5350
+P 3950 5850
+F 0 "C13" H 4065 5896 50  0000 L CNN
+F 1 "6pF" H 4065 5805 50  0000 L CNN
+F 2 "Capacitor_SMD:C_0805_2012Metric" H 3988 5700 50  0001 C CNN
+F 3 "~" H 3950 5850 50  0001 C CNN
+	1    3950 5850
+	1    0    0    -1
+$EndComp
+Wire Wire Line
+	4350 5500 4350 5700
+Connection ~ 4350 5500
 $Comp
 L power:GND #PWR028
 U 1 1 5C3D1383
-P 3950 5950
-F 0 "#PWR028" H 3950 5700 50  0001 C CNN
-F 1 "GND" H 3955 5777 50  0000 C CNN
-F 2 "" H 3950 5950 50  0001 C CNN
-F 3 "" H 3950 5950 50  0001 C CNN
-	1    3950 5950
-	1    0    0    -1
-$EndComp
-Wire Wire Line
-	3950 5900 4350 5900
-Wire Wire Line
-	4350 5900 4350 5850
-Text Notes 4100 6000 0    50   ~ 0
+P 3950 6100
+F 0 "#PWR028" H 3950 5850 50  0001 C CNN
+F 1 "GND" H 3955 5927 50  0000 C CNN
+F 2 "" H 3950 6100 50  0001 C CNN
+F 3 "" H 3950 6100 50  0001 C CNN
+	1    3950 6100
+	1    0    0    -1
+$EndComp
+Wire Wire Line
+	3950 6050 4350 6050
+Wire Wire Line
+	4350 6050 4350 6000
+Text Notes 4100 6150 0    50   ~ 0
 The crystal and caps have to be as close to the uC as possible.
 $Comp
@@
 	2500 3050 2000 3050
 Text Label 2500 2950 2    50   ~ 0
-PC6
+PB0
 Text Label 2500 3050 2    50   ~ 0
-PC7
+PB1
 Text Label 4500 3550 0    50   ~ 0
 PC0
@@
 DISPLAY_CS
 $Sheet
-S 1000 6900 1000 600
+S 1000 6800 1000 800
 U 5C392C6A
 F0 "Misc" 50
 F1 "Misc.sch" 50
-F2 "GND" I R 2000 7350 50
-F3 "PC[0..5]" I R 2000 7150 50
-F4 "PA[5..6]" I R 2000 7250 50
-F5 "+5V" I R 2000 7050 50
+F2 "GND" I R 2000 7450 50
+F3 "PC[0..5]" I R 2000 7050 50
+F4 "+5V" I R 2000 6950 50
+F5 "PA[5..7]" I R 2000 7150 50
+F6 "FAULT" I R 2000 7350 50
+F7 "RUN" I R 2000 7250 50
 $EndSheet
 $Comp
@@
 PC[0..5]
 Wire Wire Line
-	6400 4450 6900 4450
-Wire Wire Line
-	6400 4550 6900 4550
-Wire Wire Line
-	6400 4650 6900 4650
-Wire Wire Line
-	6400 4750 6900 4750
-Wire Wire Line
-	6400 4850 6900 4850
-Text Label 6900 4450 2    50   ~ 0
+	4650 6850 4150 6850
+Wire Wire Line
+	4650 6950 4150 6950
+Wire Wire Line
+	4650 7050 4150 7050
+Wire Wire Line
+	4650 7150 4150 7150
+Wire Wire Line
+	4650 7250 4150 7250
+Text Label 4650 6850 2    50   ~ 0
 TEMP_CS1
 Wire Wire Line
-	6900 4950 6400 4950
-Entry Wire Line
-	6900 4950 7000 4850
-Entry Wire Line
-	6900 4850 7000 4750
-Entry Wire Line
-	6900 4750 7000 4650
-Entry Wire Line
-	6900 4650 7000 4550
-Entry Wire Line
-	6900 4550 7000 4450
-Entry Wire Line
-	6900 4450 7000 4350
-Text Label 6900 4550 2    50   ~ 0
+	4150 7350 4650 7350
+Entry Wire Line
+	4150 7350 4050 7250
+Entry Wire Line
+	4150 7250 4050 7150
+Entry Wire Line
+	4150 7150 4050 7050
+Entry Wire Line
+	4150 7050 4050 6950
+Entry Wire Line
+	4150 6950 4050 6850
+Entry Wire Line
+	4150 6850 4050 6750
+Text Label 4650 6950 2    50   ~ 0
 TEMP_CS2
-Text Label 6900 4650 2    50   ~ 0
+Text Label 4650 7050 2    50   ~ 0
 TEMP_CS3
-Text Label 6900 4750 2    50   ~ 0
+Text Label 4650 7150 2    50   ~ 0
 TEMP_CS4
-Text Label 6900 4850 2    50   ~ 0
+Text Label 4650 7250 2    50   ~ 0
 TEMP_CS5
-Text Label 6900 4950 2    50   ~ 0
+Text Label 4650 7350 2    50   ~ 0
 TEMP_CS6
-Text Label 7000 4250 0    50   ~ 0
+Text Label 4050 6650 2    50   ~ 0
 TEMP_CS[1..6]
 Text Label 2600 5350 2    50   ~ 0
@@
 L power:GND #PWR032
 U 1 1 5C4073F6
-P 2200 7400
-F 0 "#PWR032" H 2200 7150 50  0001 C CNN
-F 1 "GND" H 2205 7227 50  0000 C CNN
-F 2 "" H 2200 7400 50  0001 C CNN
-F 3 "" H 2200 7400 50  0001 C CNN
-	1    2200 7400
-	1    0    0    -1
-$EndComp
-Wire Wire Line
-	2200 7400 2200 7350
-Wire Wire Line
-	2200 7350 2000 7350
-Text Label 2500 7150 2    50   ~ 0
+P 2200 7500
+F 0 "#PWR032" H 2200 7250 50  0001 C CNN
+F 1 "GND" H 2205 7327 50  0000 C CNN
+F 2 "" H 2200 7500 50  0001 C CNN
+F 3 "" H 2200 7500 50  0001 C CNN
+	1    2200 7500
+	1    0    0    -1
+$EndComp
+Wire Wire Line
+	2200 7500 2200 7450
+Wire Wire Line
+	2200 7450 2000 7450
+Text Label 2500 7050 2    50   ~ 0
 PC[0..5]
 Wire Wire Line
@@
 	6900 2450 7000 2350
 Text Label 7000 2250 0    50   ~ 0
-PA[5..6]
+PA[5..7]
+Wire Bus Line
+	2000 7050 2500 7050
 Wire Bus Line
 	2000 7150 2500 7150
-Wire Bus Line
-	2000 7250 2500 7250
-Text Label 2500 7250 2    50   ~ 0
-PA[5..6]
+Text Label 2500 7150 2    50   ~ 0
+PA[5..7]
 $Comp
 L Mechanical:MountingHole MH1
@@
 Wire Wire Line
 	8750 5750 8550 5750
+Text Label 7350 5750 0    50   ~ 0
+ADC1_CH2
 Text Label 7350 5650 0    50   ~ 0
-ADC1_CH2
-Text Label 7350 5750 0    50   ~ 0
 ADC1_CH3
 Wire Wire Line
@@
 	8700 5450 8750 5450
 Wire Wire Line
-	3950 5950 3950 5900
-Connection ~ 3950 5900
-Wire Wire Line
-	3950 5900 3950 5850
-Text Label 3950 4800 3    50   ~ 0
+	3950 6100 3950 6050
+Connection ~ 3950 6050
+Wire Wire Line
+	3950 6050 3950 6000
+Text Label 3950 4950 3    50   ~ 0
 OSC_OUT
-Text Label 4350 4800 3    50   ~ 0
+Text Label 4350 4950 3    50   ~ 0
 OSC_IN
 Wire Wire Line
-	4350 4800 4350 5350
-Wire Wire Line
-	3950 4800 3950 5350
-Wire Wire Line
-	3950 5550 3950 5350
-Connection ~ 3950 5350
+	4350 4950 4350 5500
+Wire Wire Line
+	3950 4950 3950 5500
+Wire Wire Line
+	3950 5700 3950 5500
+Connection ~ 3950 5500
 NoConn ~ 5000 5050
 NoConn ~ 5000 4950
@@
 NoConn ~ 5000 4650
 NoConn ~ 5000 4550
-NoConn ~ 5000 4350
-NoConn ~ 6400 5050
 NoConn ~ 6400 3850
-NoConn ~ 6400 3750
-NoConn ~ 6400 3650
 NoConn ~ 6400 3450
 NoConn ~ 5000 3350
-NoConn ~ 6400 2650
 NoConn ~ 6400 2350
 NoConn ~ 6400 2050
-NoConn ~ 6400 1950
 NoConn ~ 8400 4600
 $Comp
@@
 $EndComp
 Wire Wire Line
-	2200 7050 2200 7000
-Wire Wire Line
-	2000 7050 2200 7050
+	2200 6950 2200 6900
+Wire Wire Line
+	2000 6950 2200 6950
 $Comp
 L power:+5V #PWR031
 U 1 1 5C3EEFA7
-P 2200 7000
-F 0 "#PWR031" H 2200 6850 50  0001 C CNN
-F 1 "+5V" H 2215 7173 50  0000 C CNN
-F 2 "" H 2200 7000 50  0001 C CNN
-F 3 "" H 2200 7000 50  0001 C CNN
-	1    2200 7000
+P 2200 6900
+F 0 "#PWR031" H 2200 6750 50  0001 C CNN
+F 1 "+5V" H 2215 7073 50  0000 C CNN
+F 2 "" H 2200 6900 50  0001 C CNN
+F 3 "" H 2200 6900 50  0001 C CNN
+	1    2200 6900
 	1    0    0    -1
 $EndComp
@@
 Wire Wire Line
 	8150 6200 8150 6150
+Wire Wire Line
+	6400 4850 6900 4850
+Wire Wire Line
+	6400 4950 6900 4950
+Wire Wire Line
+	6400 5050 6900 5050
+Text Label 6900 4850 2    50   ~ 0
+TEMP_CS1
+Text Label 6900 4950 2    50   ~ 0
+TEMP_CS2
+Text Label 6900 5050 2    50   ~ 0
+TEMP_CS3
+Wire Wire Line
+	4500 4150 5000 4150
+Text Label 4500 4150 0    50   ~ 0
+TEMP_CS4
+Wire Wire Line
+	4500 4250 5000 4250
+Wire Wire Line
+	5000 4350 4500 4350
+Text Label 4500 4250 0    50   ~ 0
+TEMP_CS5
+Text Label 4500 4350 0    50   ~ 0
+TEMP_CS6
+NoConn ~ 6400 3050
+NoConn ~ 6400 3150
+Wire Wire Line
+	6400 2650 6900 2650
+Text Label 6900 2650 2    50   ~ 0
+PA7
+Entry Wire Line
+	6900 2650 7000 2550
+Wire Wire Line
+	6400 4750 6900 4750
+Text Label 6900 4750 2    50   ~ 0
+FAULT
+Wire Wire Line
+	2000 7350 2500 7350
+Text Label 2500 7350 2    50   ~ 0
+FAULT
+Wire Wire Line
+	6400 1950 6900 1950
+Text Label 6900 1950 2    50   ~ 0
+RUN
+Wire Wire Line
+	2000 7250 2500 7250
+Text Label 2500 7250 2    50   ~ 0
+RUN
 Wire Bus Line
-	7000 2250 7000 2450
+	7000 2250 7000 2550
 Wire Bus Line
 	4400 3350 4400 3950
 Wire Bus Line
-	7000 4250 7000 4850
+	4050 6650 4050 7250
 $EndSCHEMATC

Commit message: Traced regular GPIO pins on master board.
Parts:
- added L5, L6: 600, Inductor_SMD:L_0805_2012Metric, symbol Device:Ferrite_Bead_Small
Connections:
- wire segments 208 -> 210
Changed lines of the file:
@@
 L Connector_Generic:Conn_01x04 J3
 U 1 1 5CA1D80F
-P 8950 5550
-F 0 "J3" H 9029 5542 50  0000 L CNN
-F 1 "CurrentSlaveConnector" H 9029 5451 50  0000 L CNN
-F 2 "UTSVT_Connectors:Molex_MicroFit3.0_1x4xP3.00mm_PolarizingPeg_Vertical" H 8950 5550 50  0001 C CNN
-F 3 "~" H 8950 5550 50  0001 C CNN
-	1    8950 5550
+P 9450 5550
+F 0 "J3" H 9529 5542 50  0000 L CNN
+F 1 "CurrentSlaveConnector" H 9529 5451 50  0000 L CNN
+F 2 "UTSVT_Connectors:Molex_MicroFit3.0_1x4xP3.00mm_PolarizingPeg_Vertical" H 9450 5550 50  0001 C CNN
+F 3 "~" H 9450 5550 50  0001 C CNN
+	1    9450 5550
 	1    0    0    -1
 $EndComp
@@
 Wire Wire Line
 	8750 5650 8550 5650
-Wire Wire Line
-	8750 5750 8550 5750
 Text Label 7350 5750 0    50   ~ 0
 ADC1_CH2
 Text Label 7350 5650 0    50   ~ 0
 ADC1_CH3
-Wire Wire Line
-	8750 5550 8300 5550
 Wire Wire Line
 	8700 5350 8700 5450
@@
 	8300 5550 8250 5550
 Connection ~ 8700 5450
-Wire Wire Line
-	8700 5450 8750 5450
 Wire Wire Line
 	3950 6100 3950 6050
@@
 Text Label 2500 7250 2    50   ~ 0
 RUN
+$Comp
+L Device:Ferrite_Bead_Small L5
+U 1 1 5C515416
+P 8850 5650
+F 0 "L5" V 8800 5550 50  0000 C CNN
+F 1 "600" V 8800 5800 50  0000 C CNN
+F 2 "Inductor_SMD:L_0805_2012Metric" V 8780 5650 50  0001 C CNN
+F 3 "~" H 8850 5650 50  0001 C CNN
+	1    8850 5650
+	0    1    1    0
+$EndComp
+Wire Wire Line
+	8950 5650 9250 5650
+Wire Wire Line
+	8300 5550 9250 5550
+Wire Wire Line
+	8700 5450 9250 5450
+$Comp
+L Device:Ferrite_Bead_Small L6
+U 1 1 5C53EB53
+P 9050 5750
+F 0 "L6" V 9000 5650 50  0000 C CNN
+F 1 "600" V 9000 5900 50  0000 C CNN
+F 2 "Inductor_SMD:L_0805_2012Metric" V 8980 5750 50  0001 C CNN
+F 3 "~" H 9050 5750 50  0001 C CNN
+	1    9050 5750
+	0    1    1    0
+$EndComp
+Wire Wire Line
+	9150 5750 9250 5750
+Wire Wire Line
+	8550 5750 8950 5750
 Wire Bus Line
 	7000 2250 7000 2550

Commit message: Completed master board PCB
Parts:
- J2: footprint Connector_PinHeader_2.54mm:PinHeader_2x07_P2.54mm_Vertical -> Connector_PinHeader_2.54mm:PinHeader_2x05_P2.54mm_Vertical; symbol Connector_Generic:Conn_02x07_Counter_Clockwise -> Connector_Generic:Conn_02x05_Odd_Even
Connections:
- wire segments 210 -> 199
- no-connect marks 14 -> 13
Changed lines of the file:
@@
 $Descr A4 11693 8268
 encoding utf-8
-Sheet 1 8
+Sheet 1 7
 Title ""
 Date ""
@@
 The crystal and caps have to be as close to the uC as possible.
 $Comp
-L Connector_Generic:Conn_02x07_Counter_Clockwise J2
+L Connector_Generic:Conn_02x05_Odd_Even J2
 U 1 1 5C3000B6
-P 8600 4300
-F 0 "J2" H 8650 4817 50  0000 C CNN
-F 1 "Logic Analyzer" H 8650 4726 50  0000 C CNN
-F 2 "Connector_PinHeader_2.54mm:PinHeader_2x07_P2.54mm_Vertical" H 8600 4300 50  0001 C CNN
-F 3 "~" H 8600 4300 50  0001 C CNN
-	1    8600 4300
+P 8600 4200
+F 0 "J2" H 8650 4600 50  0000 C CNN
+F 1 "Logic Analyzer" H 8650 4500 50  0000 C CNN
+F 2 "Connector_PinHeader_2.54mm:PinHeader_2x05_P2.54mm_Vertical" H 8600 4200 50  0001 C CNN
+F 3 "~" H 8600 4200 50  0001 C CNN
+	1    8600 4200
 	1    0    0    -1
 $EndComp
@@
 	7900 4000 8400 4000
 Wire Wire Line
-	8400 4100 7900 4100
-Wire Wire Line
-	8400 4200 7900 4200
-Wire Wire Line
-	8400 4300 7900 4300
-Wire Wire Line
-	8400 4400 7900 4400
-Text Label 7900 4100 0    50   ~ 0
+	8900 4200 9400 4200
+Wire Wire Line
+	8900 4300 9400 4300
+Wire Wire Line
+	8900 4400 9400 4400
+Text Label 9400 4200 2    50   ~ 0
 SPI1_CLK
-Text Label 7900 4200 0    50   ~ 0
+Text Label 9400 4300 2    50   ~ 0
 SPI1_MISO
-Text Label 7900 4300 0    50   ~ 0
+Text Label 9400 4400 2    50   ~ 0
 SPI1_MOSI
-Text Label 7900 4400 0    50   ~ 0
-LTC6811_CS
-Wire Wire Line
-	8400 4500 7900 4500
-Text Label 7900 4500 0    50   ~ 0
-DISPLAY_CS
 Wire Wire Line
 	6400 4350 6900 4350
@@
 DISPLAY_CS
 Wire Wire Line
+	8400 4100 7900 4100
+Wire Wire Line
+	8400 4200 7900 4200
+Text Label 7900 4100 0    50   ~ 0
+UART1_TX
+Text Label 7900 4200 0    50   ~ 0
+UART1_RX
+Wire Wire Line
 	8900 4100 9400 4100
-Wire Wire Line
-	8900 4200 9400 4200
 Text Label 9400 4100 2    50   ~ 0
-UART1_TX
-Text Label 9400 4200 2    50   ~ 0
-UART1_RX
-Wire Wire Line
-	8900 4400 9400 4400
-Text Label 9400 4400 2    50   ~ 0
 CAN1_RX
 Wire Wire Line
-	8900 4300 9400 4300
-Text Label 9400 4300 2    50   ~ 0
+	8900 4000 9400 4000
+Text Label 9400 4000 2    50   ~ 0
 CAN1_TX
-Wire Wire Line
-	8900 4600 9400 4600
-Text Label 9400 4600 2    50   ~ 0
-I2C3_SDA
-Wire Wire Line
-	8900 4500 9400 4500
-Text Label 9400 4500 2    50   ~ 0
-I2C3_SCL
-$Comp
-L power:GND #PWR020
-U 1 1 5C369850
-P 9400 4000
-F 0 "#PWR020" H 9400 3750 50  0001 C CNN
-F 1 "GND" H 9405 3827 50  0000 C CNN
-F 2 "" H 9400 4000 50  0001 C CNN
-F 3 "" H 9400 4000 50  0001 C CNN
-	1    9400 4000
-	0    -1   1    0
-$EndComp
-Wire Wire Line
-	9400 4000 8900 4000
 Wire Wire Line
 	5000 4050 4500 4050
@@
 Wire Wire Line
 	2000 4750 2400 4750
-$Sheet
-S 1000 5900 1000 600
-U 5C3A2E97
-F0 "USB" 50
-F1 "USB.sch" 50
-F2 "GND" I R 2000 6350 50
-F3 "+3.3V" I R 2000 6050 50
-F4 "UART_RX" I R 2000 6150 50
-F5 "UART_TX" O R 2000 6250 50
-$EndSheet
-Wire Wire Line
-	2000 6150 2500 6150
-Wire Wire Line
-	2000 6250 2500 6250
-Text Label 2500 6150 2    50   ~ 0
-UART1_TX
-Text Label 2500 6250 2    50   ~ 0
-UART1_RX
-$Comp
-L power:GND #PWR030
-U 1 1 5C45DAE4
-P 2200 6400
-F 0 "#PWR030" H 2200 6150 50  0001 C CNN
-F 1 "GND" H 2205 6227 50  0000 C CNN
-F 2 "" H 2200 6400 50  0001 C CNN
-F 3 "" H 2200 6400 50  0001 C CNN
-	1    2200 6400
-	1    0    0    -1
-$EndComp
-Wire Wire Line
-	2200 6400 2200 6350
-Wire Wire Line
-	2200 6350 2000 6350
-$Comp
-L power:+3.3V #PWR029
-U 1 1 5C4686E9
-P 2200 6000
-F 0 "#PWR029" H 2200 5850 50  0001 C CNN
-F 1 "+3.3V" H 2215 6173 50  0000 C CNN
-F 2 "" H 2200 6000 50  0001 C CNN
-F 3 "" H 2200 6000 50  0001 C CNN
-	1    2200 6000
-	1    0    0    -1
-$EndComp
-Wire Wire Line
-	2200 6000 2200 6050
-Wire Wire Line
-	2200 6050 2000 6050
 Wire Bus Line
 	2000 5350 2600 5350
@@
 NoConn ~ 6400 2350
 NoConn ~ 6400 2050
-NoConn ~ 8400 4600
 $Comp
 L power:PWR_FLAG #FLG01
