File: Electronics/BPS/Master/CAN.sch (KiCad schematic (older format))
At the start: 25 parts

Commit message: Finalized schematics for BPS master.
Parts:
- gave numbers to parts that had none: 25
Changed lines of the file:
@@
 $EndDescr
 $Comp
-L utsvt-connectors:CANConnector J?
+L utsvt-connectors:CANConnector J5
 U 1 1 5C2B42F3
 P 9250 3800
-F 0 "J?" H 9250 3550 60  0000 C CNN
+F 0 "J5" H 9250 3550 60  0000 C CNN
 F 1 "CAN_Out" H 9250 4050 60  0000 C CNN
 F 2 "UTSVT_Connectors:Molex_MicroFit3.0_1x4xP3.00mm_PolarizingPeg_Vertical" H 9400 4100 60  0001 C CNN
@@
 $EndComp
 $Comp
-L Device:R R?
+L Device:R R3
 U 1 1 5C2B42FA
 P 8200 3550
-F 0 "R?" V 8280 3550 50  0000 C CNN
+F 0 "R3" V 8280 3550 50  0000 C CNN
 F 1 "60" V 8200 3550 50  0000 C CNN
 F 2 "Resistors_SMD:R_0805_HandSoldering" V 8130 3550 50  0001 C CNN
@@
 $EndComp
 $Comp
-L Device:R R?
+L Device:R R2
 U 1 1 5C2B4301
 P 8000 3550
-F 0 "R?" V 8080 3550 50  0000 C CNN
+F 0 "R2" V 8080 3550 50  0000 C CNN
 F 1 "60" V 8000 3550 50  0000 C CNN
 F 2 "Resistors_SMD:R_0805_HandSoldering" V 7930 3550 50  0001 C CNN
@@
 $EndComp
 $Comp
-L Device:Jumper_NO_Small JP?
+L Device:Jumper_NO_Small JP1
 U 1 1 5C2B4308
 P 8100 3250
-F 0 "JP?" H 8100 3330 50  0000 C CNN
+F 0 "JP1" H 8100 3330 50  0000 C CNN
 F 1 "Termination Resistors" H 8100 3200 50  0000 C CNN
 F 2 "Pin_Headers:Pin_Header_Straight_1x02_Pitch2.54mm" H 8100 3250 50  0001 C CNN
@@
 $EndComp
 $Comp
-L Device:C_Small C?
+L Device:C_Small C25
 U 1 1 5C2B4310
 P 2150 3350
-F 0 "C?" H 2160 3420 50  0000 L CNN
+F 0 "C25" H 2160 3420 50  0000 L CNN
 F 1 "10uF" H 2160 3270 50  0000 L CNN
 F 2 "Capacitors_SMD:C_0805" H 2150 3350 50  0001 C CNN
@@
 $EndComp
 $Comp
-L Device:C_Small C?
+L Device:C_Small C26
 U 1 1 5C2B4317
 P 2500 3350
-F 0 "C?" H 2510 3420 50  0000 L CNN
+F 0 "C26" H 2510 3420 50  0000 L CNN
 F 1 "0.1uF" H 2510 3270 50  0000 L CNN
 F 2 "Capacitors_SMD:C_0805" H 2500 3350 50  0001 C CNN
@@
 $EndComp
 $Comp
-L Device:C_Small C?
+L Device:C_Small C27
 U 1 1 5C2B431E
 P 2950 3350
-F 0 "C?" H 2960 3420 50  0000 L CNN
+F 0 "C27" H 2960 3420 50  0000 L CNN
 F 1 "0.1uF" H 2960 3270 50  0000 L CNN
 F 2 "Capacitors_SMD:C_0805" H 2950 3350 50  0001 C CNN
@@
 $EndComp
 $Comp
-L Device:C_Small C?
+L Device:C_Small C28
 U 1 1 5C2B4325
 P 3300 3350
-F 0 "C?" H 3310 3420 50  0000 L CNN
+F 0 "C28" H 3310 3420 50  0000 L CNN
 F 1 "0.01uF" H 3310 3270 50  0000 L CNN
 F 2 "Capacitors_SMD:C_0805" H 3300 3350 50  0001 C CNN
@@
 $EndComp
 $Comp
-L Device:C_Small C?
+L Device:C_Small C22
 U 1 1 5C2B432E
 P 6150 3200
-F 0 "C?" H 6160 3270 50  0000 L CNN
+F 0 "C22" H 6160 3270 50  0000 L CNN
 F 1 "0.22uF" H 6160 3120 50  0000 L CNN
 F 2 "Capacitors_SMD:C_0805_HandSoldering" H 6150 3200 50  0001 C CNN
@@
 $EndComp
 $Comp
-L Device:C_Small C?
+L Device:C_Small C21
 U 1 1 5C2B4335
 P 5750 3200
-F 0 "C?" H 5760 3270 50  0000 L CNN
+F 0 "C21" H 5760 3270 50  0000 L CNN
 F 1 "10uF" H 5760 3120 50  0000 L CNN
 F 2 "Capacitors_SMD:C_0805_HandSoldering" H 5750 3200 50  0001 C CNN
@@
 $EndComp
 $Comp
-L Device:Ferrite_Bead_Small L?
+L Device:Ferrite_Bead_Small L2
 U 1 1 5C2B433C
 P 5950 3050
-F 0 "L?" V 5850 3100 50  0000 L CNN
+F 0 "L2" V 5850 3100 50  0000 L CNN
 F 1 "2kH" V 5850 2900 50  0000 L CNN
 F 2 "Inductors_SMD:L_0805_HandSoldering" V 5880 3050 50  0001 C CNN
@@
 $EndComp
 $Comp
-L Device:Ferrite_Bead_Small L?
+L Device:Ferrite_Bead_Small L3
 U 1 1 5C2B4343
 P 5950 3350
-F 0 "L?" V 6050 3400 50  0000 L CNN
+F 0 "L3" V 6050 3400 50  0000 L CNN
 F 1 "2kH" V 6050 3200 50  0000 L CNN
 F 2 "Inductors_SMD:L_0805_HandSoldering" V 5880 3350 50  0001 C CNN
@@
 $EndComp
 $Comp
-L Device:C_Small C?
+L Device:C_Small C23
 U 1 1 5C2B434A
 P 6550 3200
-F 0 "C?" H 6560 3270 50  0000 L CNN
+F 0 "C23" H 6560 3270 50  0000 L CNN
 F 1 "0.1uF" H 6560 3120 50  0000 L CNN
 F 2 "Capacitors_SMD:C_0805_HandSoldering" H 6550 3200 50  0001 C CNN
@@
 $EndComp
 $Comp
-L Device:C_Small C?
+L Device:C_Small C24
 U 1 1 5C2B4351
 P 6850 3200
-F 0 "C?" H 6860 3270 50  0000 L CNN
+F 0 "C24" H 6860 3270 50  0000 L CNN
 F 1 "0.01uF" H 6860 3120 50  0000 L CNN
 F 2 "Capacitors_SMD:C_0805_HandSoldering" H 6850 3200 50  0001 C CNN
@@
 $EndComp
 $Comp
-L utsvt-chips:ADM3055E U?
+L utsvt-chips:ADM3055E U5
 U 1 1 5C2B4359
 P 4350 3600
-F 0 "U?" H 4100 4250 60  0000 C CNN
+F 0 "U5" H 4100 4250 60  0000 C CNN
 F 1 "ADM3055E" H 4550 3500 60  0000 C CNN
 F 2 "UTSVT_ICs:SOIC-20W_7.5x15.4mm_Pitch1.27mm" H 4350 3700 60  0001 C CNN
@@
 Must be close\nto V_ISO_In
 $Comp
-L Connector:TestPoint TP?
+L Connector:TestPoint TP6
 U 1 1 5C2B4371
 P 5100 2900
-F 0 "TP?" V 5200 3100 50  0000 L BNN
+F 0 "TP6" V 5200 3100 50  0000 L BNN
 F 1 "CAN_ISO_Vin" V 5100 3100 50  0000 L CNN
 F 2 "Measurement_Points:Test_Point_Keystone_5005-5009_Compact" H 5100 2900 50  0001 C CNN
@@
 $EndComp
 $Comp
-L Connector:TestPoint TP?
+L Connector:TestPoint TP8
 U 1 1 5C2B4378
 P 6200 3700
-F 0 "TP?" V 6300 3900 50  0000 L BNN
+F 0 "TP8" V 6300 3900 50  0000 L BNN
 F 1 "CAN_ISO_GndOut" V 6200 3900 50  0000 L CNN
 F 2 "Measurement_Points:Test_Point_Keystone_5005-5009_Compact" H 6200 3700 50  0001 C CNN
@@
 $EndComp
 $Comp
-L Connector:TestPoint TP?
+L Connector:TestPoint TP7
 U 1 1 5C2B437F
 P 6200 3550
-F 0 "TP?" V 6300 3750 50  0000 L BNN
+F 0 "TP7" V 6300 3750 50  0000 L BNN
 F 1 "CAN_ISO_GndIn" V 6200 3750 50  0000 L CNN
 F 2 "Measurement_Points:Test_Point_Keystone_5005-5009_Compact" H 6200 3550 50  0001 C CNN
@@
 $EndComp
 $Comp
-L Connector:TestPoint TP?
+L Connector:TestPoint TP5
 U 1 1 5C2B4386
 P 5100 2750
-F 0 "TP?" V 5200 2950 50  0000 L BNN
+F 0 "TP5" V 5200 2950 50  0000 L BNN
 F 1 "CAN_ISO_Vout" V 5100 2950 50  0000 L CNN
 F 2 "Measurement_Points:Test_Point_Keystone_5005-5009_Compact" H 5100 2750 50  0001 C CNN
@@
 NoConn ~ 3650 4100
 $Comp
-L power:PWR_FLAG #FLG?
+L power:PWR_FLAG #FLG01
 U 1 1 5C2B4394
 P 7300 3000
-F 0 "#FLG?" H 7300 3075 50  0001 C CNN
+F 0 "#FLG01" H 7300 3075 50  0001 C CNN
 F 1 "PWR_FLAG" H 7300 2900 30  0000 C CNN
 F 2 "" H 7300 3000 50  0001 C CNN
@@
 $EndComp
 $Comp
-L power:PWR_FLAG #FLG?
+L power:PWR_FLAG #FLG02
 U 1 1 5C2B439A
 P 7300 3200
-F 0 "#FLG?" H 7300 3275 50  0001 C CNN
+F 0 "#FLG02" H 7300 3275 50  0001 C CNN
 F 1 "PWR_FLAG" H 7200 3150 50  0001 L CNN
 F 2 "" H 7300 3200 50  0001 C CNN
@@
 $EndComp
 $Comp
-L utsvt-chips:CDSOT23-T24CAN U?
+L utsvt-chips:CDSOT23-T24CAN U4
 U 1 1 5C2B43A0
 P 8100 2850
-F 0 "U?" H 8100 2700 60  0000 C CNN
+F 0 "U4" H 8100 2700 60  0000 C CNN
 F 1 "CDSOT23-T24CAN" H 8100 3000 60  0000 C CNN
 F 2 "TO_SOT_Packages_SMD:SOT-23W_Handsoldering" H 8100 2850 60  0001 C CNN
@@
 CAN Bus\nProtection
 $Comp
-L Connector:TestPoint TP?
+L Connector:TestPoint TP9
 U 1 1 5C2B43B6
 P 7300 3800
-F 0 "TP?" H 7300 4100 50  0000 C BNN
+F 0 "TP9" H 7300 4100 50  0000 C BNN
 F 1 "CAN_H" H 7300 4050 50  0000 C CNN
 F 2 "Measurement_Points:Test_Point_Keystone_5005-5009_Compact" H 7300 3800 50  0001 C CNN
@@
 $EndComp
 $Comp
-L Connector:TestPoint TP?
+L Connector:TestPoint TP12
 U 1 1 5C2B43BD
 P 7300 4000
-F 0 "TP?" H 7250 4200 50  0000 L BNN
+F 0 "TP12" H 7250 4200 50  0000 L BNN
 F 1 "CAN_L" H 7200 4300 50  0000 L CNN
 F 2 "Measurement_Points:Test_Point_Keystone_5005-5009_Compact" H 7300 4000 50  0001 C CNN
@@
 $EndComp
 $Comp
-L Device:R R?
+L Device:R R4
 U 1 1 5C2B43C4
 P 5550 4150
-F 0 "R?" V 5630 4150 50  0000 C CNN
+F 0 "R4" V 5630 4150 50  0000 C CNN
 F 1 "0" V 5550 4150 50  0000 C CNN
 F 2 "Resistors_SMD:R_0805_HandSoldering" V 5480 4150 50  0001 C CNN
@@
 	3400 3800 3650 3800
 $Comp
-L Connector:TestPoint TP?
+L Connector:TestPoint TP10
 U 1 1 5C28B6DC
 P 3100 3850
-F 0 "TP?" H 3350 3950 50  0000 R CNN
+F 0 "TP10" H 3350 3950 50  0000 R CNN
 F 1 "CAN_TX" H 3350 4050 50  0000 R CNN
 F 2 "" H 3300 3850 50  0001 C CNN
@@
 $EndComp
 $Comp
-L Connector:TestPoint TP?
+L Connector:TestPoint TP11
 U 1 1 5C28BA47
 P 3400 3850
-F 0 "TP?" H 3650 3950 50  0000 R CNN
+F 0 "TP11" H 3650 3950 50  0000 R CNN
 F 1 "CAN_RX" H 3650 4050 50  0000 R CNN
 F 2 "" H 3600 3850 50  0001 C CNN
@@
 $EndComp
 $Comp
-L power:GND #PWR?
+L power:GND #PWR042
 U 1 1 5C28BDDE
 P 2150 3550
-F 0 "#PWR?" H 2150 3300 50  0001 C CNN
+F 0 "#PWR042" H 2150 3300 50  0001 C CNN
 F 1 "GND" H 2300 3500 50  0000 C CNN
 F 2 "" H 2150 3550 50  0001 C CNN

Commit message: Added SoC skeleton code.
Parts:
- C21, C22, C23, C24: footprint Capacitors_SMD:C_0805_HandSoldering -> Capacitor_SMD:C_0805_2012Metric
- C25, C26, C27, C28: footprint Capacitors_SMD:C_0805 -> Capacitor_SMD:C_0805_2012Metric
- TP10, TP11: footprint (none) -> TestPoint:TestPoint_Keystone_5005-5009_Compact
- TP12, TP5, TP6, TP7, TP8, TP9: footprint Measurement_Points:Test_Point_Keystone_5005-5009_Compact -> TestPoint:TestPoint_Keystone_5005-5009_Compact
Changed lines of the file:
@@
 F 0 "C25" H 2160 3420 50  0000 L CNN
 F 1 "10uF" H 2160 3270 50  0000 L CNN
-F 2 "Capacitors_SMD:C_0805" H 2150 3350 50  0001 C CNN
+F 2 "Capacitor_SMD:C_0805_2012Metric" H 2150 3350 50  0001 C CNN
 F 3 "" H 2150 3350 50  0001 C CNN
 	1    2150 3350
@@
 F 0 "C26" H 2510 3420 50  0000 L CNN
 F 1 "0.1uF" H 2510 3270 50  0000 L CNN
-F 2 "Capacitors_SMD:C_0805" H 2500 3350 50  0001 C CNN
+F 2 "Capacitor_SMD:C_0805_2012Metric" H 2500 3350 50  0001 C CNN
 F 3 "" H 2500 3350 50  0001 C CNN
 	1    2500 3350
@@
 F 0 "C27" H 2960 3420 50  0000 L CNN
 F 1 "0.1uF" H 2960 3270 50  0000 L CNN
-F 2 "Capacitors_SMD:C_0805" H 2950 3350 50  0001 C CNN
+F 2 "Capacitor_SMD:C_0805_2012Metric" H 2950 3350 50  0001 C CNN
 F 3 "" H 2950 3350 50  0001 C CNN
 	1    2950 3350
@@
 F 0 "C28" H 3310 3420 50  0000 L CNN
 F 1 "0.01uF" H 3310 3270 50  0000 L CNN
-F 2 "Capacitors_SMD:C_0805" H 3300 3350 50  0001 C CNN
+F 2 "Capacitor_SMD:C_0805_2012Metric" H 3300 3350 50  0001 C CNN
 F 3 "" H 3300 3350 50  0001 C CNN
 	1    3300 3350
@@
 F 0 "C22" H 6160 3270 50  0000 L CNN
 F 1 "0.22uF" H 6160 3120 50  0000 L CNN
-F 2 "Capacitors_SMD:C_0805_HandSoldering" H 6150 3200 50  0001 C CNN
+F 2 "Capacitor_SMD:C_0805_2012Metric" H 6150 3200 50  0001 C CNN
 F 3 "" H 6150 3200 50  0001 C CNN
 	1    6150 3200
@@
 F 0 "C21" H 5760 3270 50  0000 L CNN
 F 1 "10uF" H 5760 3120 50  0000 L CNN
-F 2 "Capacitors_SMD:C_0805_HandSoldering" H 5750 3200 50  0001 C CNN
+F 2 "Capacitor_SMD:C_0805_2012Metric" H 5750 3200 50  0001 C CNN
 F 3 "" H 5750 3200 50  0001 C CNN
 	1    5750 3200
@@
 F 0 "C23" H 6560 3270 50  0000 L CNN
 F 1 "0.1uF" H 6560 3120 50  0000 L CNN
-F 2 "Capacitors_SMD:C_0805_HandSoldering" H 6550 3200 50  0001 C CNN
+F 2 "Capacitor_SMD:C_0805_2012Metric" H 6550 3200 50  0001 C CNN
 F 3 "" H 6550 3200 50  0001 C CNN
 	1    6550 3200
@@
 F 0 "C24" H 6860 3270 50  0000 L CNN
 F 1 "0.01uF" H 6860 3120 50  0000 L CNN
-F 2 "Capacitors_SMD:C_0805_HandSoldering" H 6850 3200 50  0001 C CNN
+F 2 "Capacitor_SMD:C_0805_2012Metric" H 6850 3200 50  0001 C CNN
 F 3 "" H 6850 3200 50  0001 C CNN
 	1    6850 3200
@@
 F 0 "TP6" V 5200 3100 50  0000 L BNN
 F 1 "CAN_ISO_Vin" V 5100 3100 50  0000 L CNN
-F 2 "Measurement_Points:Test_Point_Keystone_5005-5009_Compact" H 5100 2900 50  0001 C CNN
+F 2 "TestPoint:TestPoint_Keystone_5005-5009_Compact" H 5100 2900 50  0001 C CNN
 F 3 "" H 5100 2900 50  0001 C CNN
 	1    5100 2900
@@
 F 0 "TP8" V 6300 3900 50  0000 L BNN
 F 1 "CAN_ISO_GndOut" V 6200 3900 50  0000 L CNN
-F 2 "Measurement_Points:Test_Point_Keystone_5005-5009_Compact" H 6200 3700 50  0001 C CNN
+F 2 "TestPoint:TestPoint_Keystone_5005-5009_Compact" H 6200 3700 50  0001 C CNN
 F 3 "" H 6200 3700 50  0001 C CNN
 	1    6200 3700
@@
 F 0 "TP7" V 6300 3750 50  0000 L BNN
 F 1 "CAN_ISO_GndIn" V 6200 3750 50  0000 L CNN
-F 2 "Measurement_Points:Test_Point_Keystone_5005-5009_Compact" H 6200 3550 50  0001 C CNN
+F 2 "TestPoint:TestPoint_Keystone_5005-5009_Compact" H 6200 3550 50  0001 C CNN
 F 3 "" H 6200 3550 50  0001 C CNN
 	1    6200 3550
@@
 F 0 "TP5" V 5200 2950 50  0000 L BNN
 F 1 "CAN_ISO_Vout" V 5100 2950 50  0000 L CNN
-F 2 "Measurement_Points:Test_Point_Keystone_5005-5009_Compact" H 5100 2750 50  0001 C CNN
+F 2 "TestPoint:TestPoint_Keystone_5005-5009_Compact" H 5100 2750 50  0001 C CNN
 F 3 "" H 5100 2750 50  0001 C CNN
 	1    5100 2750
@@
 NoConn ~ 3650 4100
 $Comp
-L power:PWR_FLAG #FLG01
+L power:PWR_FLAG #FLG03
 U 1 1 5C2B4394
 P 7300 3000
-F 0 "#FLG01" H 7300 3075 50  0001 C CNN
+F 0 "#FLG03" H 7300 3075 50  0001 C CNN
 F 1 "PWR_FLAG" H 7300 2900 30  0000 C CNN
 F 2 "" H 7300 3000 50  0001 C CNN
@@
 $EndComp
 $Comp
-L power:PWR_FLAG #FLG02
+L power:PWR_FLAG #FLG04
 U 1 1 5C2B439A
 P 7300 3200
-F 0 "#FLG02" H 7300 3275 50  0001 C CNN
+F 0 "#FLG04" H 7300 3275 50  0001 C CNN
 F 1 "PWR_FLAG" H 7200 3150 50  0001 L CNN
 F 2 "" H 7300 3200 50  0001 C CNN
@@
 F 0 "TP9" H 7300 4100 50  0000 C BNN
 F 1 "CAN_H" H 7300 4050 50  0000 C CNN
-F 2 "Measurement_Points:Test_Point_Keystone_5005-5009_Compact" H 7300 3800 50  0001 C CNN
+F 2 "TestPoint:TestPoint_Keystone_5005-5009_Compact" H 7300 3800 50  0001 C CNN
 F 3 "" H 7300 3800 50  0001 C CNN
 	1    7300 3800
@@
 F 0 "TP12" H 7250 4200 50  0000 L BNN
 F 1 "CAN_L" H 7200 4300 50  0000 L CNN
-F 2 "Measurement_Points:Test_Point_Keystone_5005-5009_Compact" H 7300 4000 50  0001 C CNN
+F 2 "TestPoint:TestPoint_Keystone_5005-5009_Compact" H 7300 4000 50  0001 C CNN
 F 3 "" H 7300 4000 50  0001 C CNN
 	1    7300 4000
@@
 F 0 "TP10" H 3350 3950 50  0000 R CNN
 F 1 "CAN_TX" H 3350 4050 50  0000 R CNN
-F 2 "" H 3300 3850 50  0001 C CNN
+F 2 "TestPoint:TestPoint_Keystone_5005-5009_Compact" H 3300 3850 50  0001 C CNN
 F 3 "~" H 3300 3850 50  0001 C CNN
 	1    3100 3850
@@
 F 0 "TP11" H 3650 3950 50  0000 R CNN
 F 1 "CAN_RX" H 3650 4050 50  0000 R CNN
-F 2 "" H 3600 3850 50  0001 C CNN
+F 2 "TestPoint:TestPoint_Keystone_5005-5009_Compact" H 3600 3850 50  0001 C CNN
 F 3 "~" H 3600 3850 50  0001 C CNN
 	1    3400 3850

Commit message: Assigned footprints to each symbol in BPS schematics.
Parts:
- L2, L3: footprint Inductors_SMD:L_0805_HandSoldering -> Inductor_SMD:L_0805_2012Metric
- R2, R3, R4: footprint Resistors_SMD:R_0805_HandSoldering -> Resistor_SMD:R_0805_2012Metric
- renumbered C21 to C19, C22 to C20, C23 to C21, C24 to C22, C25 to C23, C26 to C24, C27 to C25, C28 to C26
Connections:
- wire segments 106 -> 108
Changed lines of the file:
@@
 F 0 "R3" V 8280 3550 50  0000 C CNN
 F 1 "60" V 8200 3550 50  0000 C CNN
-F 2 "Resistors_SMD:R_0805_HandSoldering" V 8130 3550 50  0001 C CNN
+F 2 "Resistor_SMD:R_0805_2012Metric" V 8130 3550 50  0001 C CNN
 F 3 "" H 8200 3550 50  0001 C CNN
 	1    8200 3550
@@
 F 0 "R2" V 8080 3550 50  0000 C CNN
 F 1 "60" V 8000 3550 50  0000 C CNN
-F 2 "Resistors_SMD:R_0805_HandSoldering" V 7930 3550 50  0001 C CNN
+F 2 "Resistor_SMD:R_0805_2012Metric" V 7930 3550 50  0001 C CNN
 F 3 "" H 8000 3550 50  0001 C CNN
 	1    8000 3550
@@
 $EndComp
 $Comp
-L Device:C_Small C25
+L Device:C_Small C23
 U 1 1 5C2B4310
 P 2150 3350
-F 0 "C25" H 2160 3420 50  0000 L CNN
+F 0 "C23" H 2160 3420 50  0000 L CNN
 F 1 "10uF" H 2160 3270 50  0000 L CNN
 F 2 "Capacitor_SMD:C_0805_2012Metric" H 2150 3350 50  0001 C CNN
@@
 $EndComp
 $Comp
-L Device:C_Small C26
+L Device:C_Small C24
 U 1 1 5C2B4317
 P 2500 3350
-F 0 "C26" H 2510 3420 50  0000 L CNN
+F 0 "C24" H 2510 3420 50  0000 L CNN
 F 1 "0.1uF" H 2510 3270 50  0000 L CNN
 F 2 "Capacitor_SMD:C_0805_2012Metric" H 2500 3350 50  0001 C CNN
@@
 $EndComp
 $Comp
-L Device:C_Small C27
+L Device:C_Small C25
 U 1 1 5C2B431E
 P 2950 3350
-F 0 "C27" H 2960 3420 50  0000 L CNN
+F 0 "C25" H 2960 3420 50  0000 L CNN
 F 1 "0.1uF" H 2960 3270 50  0000 L CNN
 F 2 "Capacitor_SMD:C_0805_2012Metric" H 2950 3350 50  0001 C CNN
@@
 $EndComp
 $Comp
-L Device:C_Small C28
+L Device:C_Small C26
 U 1 1 5C2B4325
 P 3300 3350
-F 0 "C28" H 3310 3420 50  0000 L CNN
+F 0 "C26" H 3310 3420 50  0000 L CNN
 F 1 "0.01uF" H 3310 3270 50  0000 L CNN
 F 2 "Capacitor_SMD:C_0805_2012Metric" H 3300 3350 50  0001 C CNN
@@
 $EndComp
 $Comp
-L Device:C_Small C22
+L Device:C_Small C20
 U 1 1 5C2B432E
 P 6150 3200
-F 0 "C22" H 6160 3270 50  0000 L CNN
+F 0 "C20" H 6160 3270 50  0000 L CNN
 F 1 "0.22uF" H 6160 3120 50  0000 L CNN
 F 2 "Capacitor_SMD:C_0805_2012Metric" H 6150 3200 50  0001 C CNN
@@
 $EndComp
 $Comp
-L Device:C_Small C21
+L Device:C_Small C19
 U 1 1 5C2B4335
 P 5750 3200
-F 0 "C21" H 5760 3270 50  0000 L CNN
+F 0 "C19" H 5760 3270 50  0000 L CNN
 F 1 "10uF" H 5760 3120 50  0000 L CNN
 F 2 "Capacitor_SMD:C_0805_2012Metric" H 5750 3200 50  0001 C CNN
@@
 F 0 "L2" V 5850 3100 50  0000 L CNN
 F 1 "2kH" V 5850 2900 50  0000 L CNN
-F 2 "Inductors_SMD:L_0805_HandSoldering" V 5880 3050 50  0001 C CNN
+F 2 "Inductor_SMD:L_0805_2012Metric" V 5880 3050 50  0001 C CNN
 F 3 "" H 5950 3050 50  0001 C CNN
 	1    5950 3050
@@
 F 0 "L3" V 6050 3400 50  0000 L CNN
 F 1 "2kH" V 6050 3200 50  0000 L CNN
-F 2 "Inductors_SMD:L_0805_HandSoldering" V 5880 3350 50  0001 C CNN
+F 2 "Inductor_SMD:L_0805_2012Metric" V 5880 3350 50  0001 C CNN
 F 3 "" H 5950 3350 50  0001 C CNN
 	1    5950 3350
@@
 $EndComp
 $Comp
-L Device:C_Small C23
+L Device:C_Small C21
 U 1 1 5C2B434A
 P 6550 3200
-F 0 "C23" H 6560 3270 50  0000 L CNN
+F 0 "C21" H 6560 3270 50  0000 L CNN
 F 1 "0.1uF" H 6560 3120 50  0000 L CNN
 F 2 "Capacitor_SMD:C_0805_2012Metric" H 6550 3200 50  0001 C CNN
@@
 $EndComp
 $Comp
-L Device:C_Small C24
+L Device:C_Small C22
 U 1 1 5C2B4351
 P 6850 3200
-F 0 "C24" H 6860 3270 50  0000 L CNN
+F 0 "C22" H 6860 3270 50  0000 L CNN
 F 1 "0.01uF" H 6860 3120 50  0000 L CNN
 F 2 "Capacitor_SMD:C_0805_2012Metric" H 6850 3200 50  0001 C CNN
@@
 F 0 "R4" V 5630 4150 50  0000 C CNN
 F 1 "0" V 5550 4150 50  0000 C CNN
-F 2 "Resistors_SMD:R_0805_HandSoldering" V 5480 4150 50  0001 C CNN
+F 2 "Resistor_SMD:R_0805_2012Metric" V 5480 4150 50  0001 C CNN
 F 3 "" H 5550 4150 50  0001 C CNN
 	1    5550 4150
@@
 Wire Wire Line
 	2500 3100 3650 3100
+Wire Wire Line
+	2500 3000 2500 3100
+$Comp
+L power:+3.3V #PWR0133
+U 1 1 5C4ABE05
+P 2950 3000
+F 0 "#PWR0133" H 2950 2850 50  0001 C CNN
+F 1 "+3.3V" H 2965 3173 50  0000 C CNN
+F 2 "" H 2950 3000 50  0001 C CNN
+F 3 "" H 2950 3000 50  0001 C CNN
+	1    2950 3000
+	1    0    0    -1
+$EndComp
+Wire Wire Line
+	2950 3000 2950 3200
+$Comp
+L power:+5V #PWR0132
+U 1 1 5C4C2AB0
+P 2500 3000
+F 0 "#PWR0132" H 2500 2850 50  0001 C CNN
+F 1 "+5V" H 2515 3173 50  0000 C CNN
+F 2 "" H 2500 3000 50  0001 C CNN
+F 3 "" H 2500 3000 50  0001 C CNN
+	1    2500 3000
+	1    0    0    -1
+$EndComp
 $EndSCHEMATC

Commit message: Master board PCB layout organized.
Parts:
- removed TP10: CAN_TX, TestPoint:TestPoint_Keystone_5005-5009_Compact, symbol Connector:TestPoint
- removed TP11: CAN_RX, TestPoint:TestPoint_Keystone_5005-5009_Compact, symbol Connector:TestPoint
- JP1: footprint Pin_Headers:Pin_Header_Straight_1x02_Pitch2.54mm -> Connector_PinHeader_2.54mm:PinHeader_1x02_P2.54mm_Vertical; symbol Device:Jumper_NO_Small -> Device:Jumper_NC_Small
- U4: footprint TO_SOT_Packages_SMD:SOT-23W_Handsoldering -> Package_TO_SOT_SMD:SOT-23W
Connections:
- wire segments 108 -> 104
Changed lines of the file:
@@
 $EndComp
 $Comp
-L Device:Jumper_NO_Small JP1
+L Device:Jumper_NC_Small JP1
 U 1 1 5C2B4308
 P 8100 3250
 F 0 "JP1" H 8100 3330 50  0000 C CNN
 F 1 "Termination Resistors" H 8100 3200 50  0000 C CNN
-F 2 "Pin_Headers:Pin_Header_Straight_1x02_Pitch2.54mm" H 8100 3250 50  0001 C CNN
+F 2 "Connector_PinHeader_2.54mm:PinHeader_1x02_P2.54mm_Vertical" H 8100 3250 50  0001 C CNN
 F 3 "" H 8100 3250 50  0001 C CNN
 	1    8100 3250
@@
 F 0 "U4" H 8100 2700 60  0000 C CNN
 F 1 "CDSOT23-T24CAN" H 8100 3000 60  0000 C CNN
-F 2 "TO_SOT_Packages_SMD:SOT-23W_Handsoldering" H 8100 2850 60  0001 C CNN
+F 2 "Package_TO_SOT_SMD:SOT-23W" H 8100 2850 60  0001 C CNN
 F 3 "" H 8100 2850 60  0001 C CNN
 	1    8100 2850
@@
 	6150 2900 6150 3050
 Wire Wire Line
-	5050 3550 5250 3550
-Wire Wire Line
 	6150 3300 6150 3350
 Wire Wire Line
@@
 Connection ~ 6150 3350
 Wire Wire Line
-	2950 3700 3100 3700
-Wire Wire Line
-	2950 3800 3400 3800
-Wire Wire Line
 	5400 4150 5050 4150
 Wire Wire Line
@@
 Wire Wire Line
 	5250 3450 5050 3450
-Connection ~ 5250 3550
 Wire Wire Line
 	5250 3250 5250 3350
@@
 	6050 3050 6150 3050
 Wire Wire Line
-	3100 3850 3100 3700
-Connection ~ 3100 3700
-Wire Wire Line
-	3400 3850 3400 3800
-Connection ~ 3400 3800
-Wire Wire Line
 	7300 3800 7300 3850
 Wire Wire Line
@@
 Wire Wire Line
 	6150 3550 6200 3550
-Wire Wire Line
-	3100 3700 3650 3700
-Wire Wire Line
-	3400 3800 3650 3800
-$Comp
-L Connector:TestPoint TP10
-U 1 1 5C28B6DC
-P 3100 3850
-F 0 "TP10" H 3350 3950 50  0000 R CNN
-F 1 "CAN_TX" H 3350 4050 50  0000 R CNN
-F 2 "TestPoint:TestPoint_Keystone_5005-5009_Compact" H 3300 3850 50  0001 C CNN
-F 3 "~" H 3300 3850 50  0001 C CNN
-	1    3100 3850
-	-1   0    0    1
-$EndComp
-$Comp
-L Connector:TestPoint TP11
-U 1 1 5C28BA47
-P 3400 3850
-F 0 "TP11" H 3650 3950 50  0000 R CNN
-F 1 "CAN_RX" H 3650 4050 50  0000 R CNN
-F 2 "TestPoint:TestPoint_Keystone_5005-5009_Compact" H 3600 3850 50  0001 C CNN
-F 3 "~" H 3600 3850 50  0001 C CNN
-	1    3400 3850
-	-1   0    0    1
-$EndComp
 $Comp
 L power:GND #PWR042
@@
 	1    0    0    -1
 $EndComp
+Connection ~ 5250 3550
+Wire Wire Line
+	5050 3550 5250 3550
+Wire Wire Line
+	2950 3700 3650 3700
+Wire Wire Line
+	2950 3800 3650 3800
 $EndSCHEMATC

Commit message: Organized all components in BPS master to where they should be.
Connections:
- net labels removed: CAN_ISA_VOUT, CAN_ISO_VIN, GND_ISO_IN, GND_ISO_OUT
Changed lines of the file:
@@
 Text Label 8200 3350 0    50   ~ 0
 TERM_L
-Text Label 5250 2900 0    50   ~ 0
-CAN_ISO_VIN
-Text Label 5250 3050 0    50   ~ 0
-CAN_ISA_VOUT
-Text Label 5250 3350 0    50   ~ 0
-GND_ISO_OUT
-Text Label 5250 3550 0    50   ~ 0
-GND_ISO_IN
 Connection ~ 5750 3050
 Wire Wire Line
