File: Electronics/BPS/Master/Contactor.sch (KiCad schematic (older format))
At the start: 17 parts

Commit message: Finalized schematics for BPS master.
Parts:
- added Q2: NVR4003NT3G, Package_TO_SOT_SMD:SOT-23, symbol Device:Q_NMOS_GSD
- R5: renamed from R?; value 5.1k -> 775
- R6: renamed from R?; value 150 -> 220
- gave numbers to parts that had none: 15
Connections:
- net labels added: +3.3V
- wire segments 64 -> 72

Commit message: Added SoC skeleton code.
Parts:
- added R11: 0, symbol Device:R
- added R12: 100k, symbol Device:R
- C29, C30, C31: footprint (none) -> Capacitor_SMD:C_0805_2012Metric
- R5: value 775 -> 1.5k
- R7: renamed from R6; value 220 -> 470
- TP13: value Gate_TP -> ContactorGate_TP; footprint (none) -> TestPoint:TestPoint_Keystone_5005-5009_Compact
- renumbered R7 to R6, R9 to R8, R8 to R9, U7 to U6, U6 to U7
Connections:
- net labels removed: +3.3V
- wire segments 72 -> 77

Commit message: Assigned footprints to each symbol in BPS schematics.
Parts:
- D3: footprint (none) -> LED_SMD:LED_0805_2012Metric
- J6: footprint Connector_PinHeader_2.54mm:PinHeader_1x04_P2.54mm_Vertical -> UTSVT_Connectors:Molex_MicroFit3.0_1x4xP3.00mm_PolarizingPeg_Vertical
- R10, R11, R12, R5, R6, R7, R8, R9: footprint (none) -> Resistor_SMD:R_0805_2012Metric
- renumbered C29 to C27, C30 to C28, C31 to C29, C32 to C30
Changed lines of the file:
@@
 F 0 "J6" H 10200 3500 50  0000 R CNN
 F 1 "ContactorConnector" H 10850 3400 50  0000 R CNN
-F 2 "Connector_PinHeader_2.54mm:PinHeader_1x04_P2.54mm_Vertical" H 10050 3500 50  0001 C CNN
+F 2 "UTSVT_Connectors:Molex_MicroFit3.0_1x4xP3.00mm_PolarizingPeg_Vertical" H 10050 3500 50  0001 C CNN
 F 3 "~" H 10050 3500 50  0001 C CNN
 	1    10050 3500
@@
 F 0 "R8" V 8850 3700 50  0000 C CNN
 F 1 "1k" V 8950 3700 50  0000 C CNN
-F 2 "" V 8880 3700 50  0001 C CNN
+F 2 "Resistor_SMD:R_0805_2012Metric" V 8880 3700 50  0001 C CNN
 F 3 "~" H 8950 3700 50  0001 C CNN
 	1    8950 3700
@@
 	9850 3700 9200 3700
 $Comp
-L Device:C C32
+L Device:C C30
 U 1 1 5C3030F2
 P 8700 3950
-F 0 "C32" H 8815 3996 50  0000 L CNN
+F 0 "C30" H 8815 3996 50  0000 L CNN
 F 1 "1uF" H 8815 3905 50  0000 L CNN
 F 2 "Capacitor_SMD:C_0805_2012Metric" H 8738 3800 50  0001 C CNN
@@
 F 0 "R10" H 5250 4100 50  0000 L CNN
 F 1 "100k" V 5200 4000 50  0000 L CNN
-F 2 "" V 5130 4100 50  0001 C CNN
+F 2 "Resistor_SMD:R_0805_2012Metric" V 5130 4100 50  0001 C CNN
 F 3 "~" H 5200 4100 50  0001 C CNN
 	1    5200 4100
@@
 F 0 "R9" V 4850 3850 50  0000 C CNN
 F 1 "0" V 4950 3850 50  0000 C CNN
-F 2 "" V 4880 3850 50  0001 C CNN
+F 2 "Resistor_SMD:R_0805_2012Metric" V 4880 3850 50  0001 C CNN
 F 3 "~" H 4950 3850 50  0001 C CNN
 	1    4950 3850
@@
 $EndComp
 $Comp
-L Device:C C30
+L Device:C C28
 U 1 1 5C30FCB3
 P 3350 3050
-F 0 "C30" H 3465 3096 50  0000 L CNN
+F 0 "C28" H 3465 3096 50  0000 L CNN
 F 1 "10uF" H 3465 3005 50  0000 L CNN
 F 2 "Capacitor_SMD:C_0805_2012Metric" H 3388 2900 50  0001 C CNN
@@
 $EndComp
 $Comp
-L Device:C C31
+L Device:C C29
 U 1 1 5C310937
 P 3800 3050
-F 0 "C31" H 3915 3096 50  0000 L CNN
+F 0 "C29" H 3915 3096 50  0000 L CNN
 F 1 "0.1uF" H 3915 3005 50  0000 L CNN
 F 2 "Capacitor_SMD:C_0805_2012Metric" H 3838 2900 50  0001 C CNN
@@
 F 0 "R7" V 2600 3500 50  0000 C CNN
 F 1 "470" V 2700 3500 50  0000 C CNN
-F 2 "" V 2630 3500 50  0001 C CNN
+F 2 "Resistor_SMD:R_0805_2012Metric" V 2630 3500 50  0001 C CNN
 F 3 "~" H 2700 3500 50  0001 C CNN
 	1    2700 3500
@@
 F 0 "R5" H 2320 3396 50  0000 L CNN
 F 1 "1.5k" V 2250 3350 50  0000 C CNN
-F 2 "" V 2180 3350 50  0001 C CNN
+F 2 "Resistor_SMD:R_0805_2012Metric" V 2180 3350 50  0001 C CNN
 F 3 "~" H 2250 3350 50  0001 C CNN
 	1    2250 3350
@@
 F 0 "D3" V 2300 4000 50  0000 R CNN
 F 1 "ContactorEn" V 2200 4250 50  0000 R CNN
-F 2 "" H 2250 3700 50  0001 C CNN
+F 2 "LED_SMD:LED_0805_2012Metric" H 2250 3700 50  0001 C CNN
 F 3 "~" H 2250 3700 50  0001 C CNN
 F 4 "Green" V 2250 3700 50  0001 C CNN "Color"
@@
 F 0 "R6" V 8600 3400 50  0000 C CNN
 F 1 "4.7k" V 8700 3400 50  0000 C CNN
-F 2 "" V 8630 3400 50  0001 C CNN
+F 2 "Resistor_SMD:R_0805_2012Metric" V 8630 3400 50  0001 C CNN
 F 3 "~" H 8700 3400 50  0001 C CNN
 	1    8700 3400
@@
 $EndComp
 $Comp
-L Device:C C29
+L Device:C C27
 U 1 1 5C3F87F6
 P 5950 2900
-F 0 "C29" V 5698 2900 50  0000 C CNN
+F 0 "C27" V 5698 2900 50  0000 C CNN
 F 1 "1uF" V 5789 2900 50  0000 C CNN
 F 2 "Capacitor_SMD:C_0805_2012Metric" H 5988 2750 50  0001 C CNN
@@
 F 0 "R11" V 1500 4200 50  0000 C CNN
 F 1 "0" V 1600 4200 50  0000 C CNN
-F 2 "" V 1530 4200 50  0001 C CNN
+F 2 "Resistor_SMD:R_0805_2012Metric" V 1530 4200 50  0001 C CNN
 F 3 "~" H 1600 4200 50  0001 C CNN
 	1    1600 4200
@@
 F 0 "R12" H 1900 4400 50  0000 L CNN
 F 1 "100k" V 1850 4300 50  0000 L CNN
-F 2 "" V 1780 4400 50  0001 C CNN
+F 2 "Resistor_SMD:R_0805_2012Metric" V 1780 4400 50  0001 C CNN
 F 3 "~" H 1850 4400 50  0001 C CNN
 	1    1850 4400
