File: Electronics/BPS/Master/I2C.sch (KiCad schematic (older format))
At the start: 11 parts, among them U8 M24128, U9 LSM6DS3

Commit message: Added SoC skeleton code.
Parts:
- C33, C34, C35: footprint (none) -> Capacitor_SMD:C_0805_2012Metric
- renumbered R11 to R13, R12 to R14
Changed lines of the file:
@@
 F 0 "C33" H 3315 2846 50  0000 L CNN
 F 1 "0.1uF" H 3315 2755 50  0000 L CNN
-F 2 "" H 3238 2650 50  0001 C CNN
+F 2 "Capacitor_SMD:C_0805_2012Metric" H 3238 2650 50  0001 C CNN
 F 3 "~" H 3200 2800 50  0001 C CNN
 	1    3200 2800
@@
 	3650 3000 3750 3000
 $Comp
-L Device:R R12
+L Device:R R14
 U 1 1 5C351986
 P 2800 2850
-F 0 "R12" H 2870 2896 50  0000 L CNN
+F 0 "R14" H 2870 2896 50  0000 L CNN
 F 1 "4.7k" H 2870 2805 50  0000 L CNN
 F 2 "" V 2730 2850 50  0001 C CNN
@@
 $EndComp
 $Comp
-L Device:R R11
+L Device:R R13
 U 1 1 5C3519B6
 P 2400 2850
-F 0 "R11" H 2470 2896 50  0000 L CNN
+F 0 "R13" H 2470 2896 50  0000 L CNN
 F 1 "4.7k" H 2470 2805 50  0000 L CNN
 F 2 "" V 2330 2850 50  0001 C CNN
@@
 F 0 "C34" H 5015 4946 50  0000 L CNN
 F 1 "0.1uF" H 5015 4855 50  0000 L CNN
-F 2 "" H 4938 4750 50  0001 C CNN
+F 2 "Capacitor_SMD:C_0805_2012Metric" H 4938 4750 50  0001 C CNN
 F 3 "~" H 4900 4900 50  0001 C CNN
 	1    4900 4900
@@
 F 0 "C35" H 5465 4946 50  0000 L CNN
 F 1 "0.1uF" H 5465 4855 50  0000 L CNN
-F 2 "" H 5388 4750 50  0001 C CNN
+F 2 "Capacitor_SMD:C_0805_2012Metric" H 5388 4750 50  0001 C CNN
 F 3 "~" H 5350 4900 50  0001 C CNN
 	1    5350 4900
@@
 	3650 5400 3700 5400
 $Comp
-L power:PWR_FLAG #FLG0103
+L power:PWR_FLAG #FLG05
 U 1 1 5CC89108
 P 5200 2900
-F 0 "#FLG0103" H 5200 2975 50  0001 C CNN
+F 0 "#FLG05" H 5200 2975 50  0001 C CNN
 F 1 "PWR_FLAG" V 5200 3028 50  0000 L CNN
 F 2 "" H 5200 2900 50  0001 C CNN
@@
 $EndComp
 $Comp
-L power:PWR_FLAG #FLG0104
+L power:PWR_FLAG #FLG06
 U 1 1 5CC89201
 P 5200 3000
-F 0 "#FLG0104" H 5200 3075 50  0001 C CNN
+F 0 "#FLG06" H 5200 3075 50  0001 C CNN
 F 1 "PWR_FLAG" V 5200 3128 50  0000 L CNN
 F 2 "" H 5200 3000 50  0001 C CNN
@@
 $EndComp
 $Comp
-L power:PWR_FLAG #FLG0105
+L power:PWR_FLAG #FLG07
 U 1 1 5CC89222
 P 5200 3100
-F 0 "#FLG0105" H 5200 3175 50  0001 C CNN
+F 0 "#FLG07" H 5200 3175 50  0001 C CNN
 F 1 "PWR_FLAG" V 5200 3228 50  0000 L CNN
 F 2 "" H 5200 3100 50  0001 C CNN

Commit message: Assigned footprints to each symbol in BPS schematics.
Parts:
- R13, R14: footprint (none) -> Resistor_SMD:R_0805_2012Metric
- renumbered C33 to C31, C34 to C32, C35 to C33
Changed lines of the file:
@@
 +3.3V
 $Comp
-L Device:C C33
+L Device:C C31
 U 1 1 5C35143C
 P 3200 2800
-F 0 "C33" H 3315 2846 50  0000 L CNN
+F 0 "C31" H 3315 2846 50  0000 L CNN
 F 1 "0.1uF" H 3315 2755 50  0000 L CNN
 F 2 "Capacitor_SMD:C_0805_2012Metric" H 3238 2650 50  0001 C CNN
@@
 F 0 "R14" H 2870 2896 50  0000 L CNN
 F 1 "4.7k" H 2870 2805 50  0000 L CNN
-F 2 "" V 2730 2850 50  0001 C CNN
+F 2 "Resistor_SMD:R_0805_2012Metric" V 2730 2850 50  0001 C CNN
 F 3 "~" H 2800 2850 50  0001 C CNN
 	1    2800 2850
@@
 F 0 "R13" H 2470 2896 50  0000 L CNN
 F 1 "4.7k" H 2470 2805 50  0000 L CNN
-F 2 "" V 2330 2850 50  0001 C CNN
+F 2 "Resistor_SMD:R_0805_2012Metric" V 2330 2850 50  0001 C CNN
 F 3 "~" H 2400 2850 50  0001 C CNN
 	1    2400 2850
@@
 SDA
 $Comp
-L Device:C C34
+L Device:C C32
 U 1 1 5CA0C7FA
 P 4900 4900
-F 0 "C34" H 5015 4946 50  0000 L CNN
+F 0 "C32" H 5015 4946 50  0000 L CNN
 F 1 "0.1uF" H 5015 4855 50  0000 L CNN
 F 2 "Capacitor_SMD:C_0805_2012Metric" H 4938 4750 50  0001 C CNN
@@
 $EndComp
 $Comp
-L Device:C C35
+L Device:C C33
 U 1 1 5CA0C84A
 P 5350 4900
-F 0 "C35" H 5465 4946 50  0000 L CNN
+F 0 "C33" H 5465 4946 50  0000 L CNN
 F 1 "0.1uF" H 5465 4855 50  0000 L CNN
 F 2 "Capacitor_SMD:C_0805_2012Metric" H 5388 4750 50  0001 C CNN

Commit message: Master board PCB layout organized.
Parts:
- removed JP2, JP3, JP4, JP5: SolderJumper_3_Open, Jumper:SolderJumper-3_P1.3mm_Bridged12_Pad1.0x1.5mm, symbol Jumper:SolderJumper_3_Bridged12
Connections:
- net labels removed: E0, E1, E2
- wire segments 61 -> 53
Other:
- note added: "Addr: 0x64"
- note removed: "Addr: 0x65"
- note removed: "These caps. have to be placed at each VDD pin. One cap per VDD pin."
- note removed: "These jumpers let's you change the EEPROM address if there is a conflict.\nFor now, the EEPROM address is 0x50."
Changed lines of the file:
@@
 Wire Wire Line
 	2400 2500 2400 2600
-Wire Wire Line
-	4750 3000 5200 3000
-$Comp
-L Jumper:SolderJumper_3_Bridged12 JP2
-U 1 1 5C3552F2
-P 6300 2900
-F 0 "JP2" V 6346 2968 50  0000 L CNN
-F 1 "SolderJumper_3_Open" V 6255 2968 50  0000 L CNN
-F 2 "Jumper:SolderJumper-3_P1.3mm_Bridged12_Pad1.0x1.5mm" H 6300 2900 50  0001 C CNN
-F 3 "~" H 6300 2900 50  0001 C CNN
-	1    6300 2900
-	0    1    -1   0
-$EndComp
-$Comp
-L Jumper:SolderJumper_3_Bridged12 JP3
-U 1 1 5C355357
-P 6850 3450
-F 0 "JP3" V 6896 3518 50  0000 L CNN
-F 1 "SolderJumper_3_Open" V 6805 3518 50  0000 L CNN
-F 2 "Jumper:SolderJumper-3_P1.3mm_Bridged12_Pad1.0x1.5mm" H 6850 3450 50  0001 C CNN
-F 3 "~" H 6850 3450 50  0001 C CNN
-	1    6850 3450
-	0    1    -1   0
-$EndComp
-$Comp
-L Jumper:SolderJumper_3_Bridged12 JP4
-U 1 1 5C355391
-P 7400 4000
-F 0 "JP4" V 7446 4068 50  0000 L CNN
-F 1 "SolderJumper_3_Open" V 7355 4068 50  0000 L CNN
-F 2 "Jumper:SolderJumper-3_P1.3mm_Bridged12_Pad1.0x1.5mm" H 7400 4000 50  0001 C CNN
-F 3 "~" H 7400 4000 50  0001 C CNN
-	1    7400 4000
-	0    1    -1   0
-$EndComp
-Wire Wire Line
-	4750 3100 5200 3100
-Wire Wire Line
-	4750 2900 5200 2900
-Text Label 5200 2900 2    50   ~ 0
-E0
-Text Label 5200 3000 2    50   ~ 0
-E1
-Text Label 5200 3100 2    50   ~ 0
-E2
-Wire Wire Line
-	6150 2900 5950 2900
-Text Label 5950 2900 0    50   ~ 0
-E0
-Text Label 6500 3450 0    50   ~ 0
-E1
-Wire Wire Line
-	7250 4000 7050 4000
-Text Label 7050 4000 0    50   ~ 0
-E2
-$Comp
-L power:GND #PWR057
-U 1 1 5C356B3E
-P 6300 3150
-F 0 "#PWR057" H 6300 2900 50  0001 C CNN
-F 1 "GND" H 6305 2977 50  0000 C CNN
-F 2 "" H 6300 3150 50  0001 C CNN
-F 3 "" H 6300 3150 50  0001 C CNN
-	1    6300 3150
-	1    0    0    -1
-$EndComp
-$Comp
-L power:GND #PWR061
-U 1 1 5C3572BE
-P 6850 3700
-F 0 "#PWR061" H 6850 3450 50  0001 C CNN
-F 1 "GND" H 6855 3527 50  0000 C CNN
-F 2 "" H 6850 3700 50  0001 C CNN
-F 3 "" H 6850 3700 50  0001 C CNN
-	1    6850 3700
-	1    0    0    -1
-$EndComp
-$Comp
-L power:GND #PWR063
-U 1 1 5C3572D7
-P 7400 4250
-F 0 "#PWR063" H 7400 4000 50  0001 C CNN
-F 1 "GND" H 7405 4077 50  0000 C CNN
-F 2 "" H 7400 4250 50  0001 C CNN
-F 3 "" H 7400 4250 50  0001 C CNN
-	1    7400 4250
-	1    0    0    -1
-$EndComp
-Wire Wire Line
-	6300 3150 6300 3100
-Wire Wire Line
-	6850 3650 6850 3700
-Wire Wire Line
-	7400 4200 7400 4250
-$Comp
-L power:+3.3V #PWR056
-U 1 1 5C358A09
-P 6300 2650
-F 0 "#PWR056" H 6300 2500 50  0001 C CNN
-F 1 "+3.3V" H 6315 2823 50  0000 C CNN
-F 2 "" H 6300 2650 50  0001 C CNN
-F 3 "" H 6300 2650 50  0001 C CNN
-	1    6300 2650
-	1    0    0    -1
-$EndComp
-Wire Wire Line
-	6300 2650 6300 2700
-$Comp
-L power:+3.3V #PWR058
-U 1 1 5C358E92
-P 6850 3200
-F 0 "#PWR058" H 6850 3050 50  0001 C CNN
-F 1 "+3.3V" H 6865 3373 50  0000 C CNN
-F 2 "" H 6850 3200 50  0001 C CNN
-F 3 "" H 6850 3200 50  0001 C CNN
-	1    6850 3200
-	1    0    0    -1
-$EndComp
-Wire Wire Line
-	6850 3200 6850 3250
-$Comp
-L power:+3.3V #PWR062
-U 1 1 5C359303
-P 7400 3750
-F 0 "#PWR062" H 7400 3600 50  0001 C CNN
-F 1 "+3.3V" H 7415 3923 50  0000 C CNN
-F 2 "" H 7400 3750 50  0001 C CNN
-F 3 "" H 7400 3750 50  0001 C CNN
-	1    7400 3750
-	1    0    0    -1
-$EndComp
-Wire Wire Line
-	7400 3750 7400 3800
-Wire Wire Line
-	6500 3450 6700 3450
-Text Notes 5950 2350 0    50   ~ 0
-These jumpers let's you change the EEPROM address if there is a conflict.\nFor now, the EEPROM address is 0x50.
 Text Label 3600 3100 2    50   ~ 0
 SCL
@@
 Connection ~ 4300 4700
 Wire Wire Line
-	3700 5600 3250 5600
-Wire Wire Line
 	3700 5700 3250 5700
 Text Label 3250 5700 0    50   ~ 0
 SCL
-Text Label 3250 5600 0    50   ~ 0
-SDA
 $Comp
 L Device:C C32
@@
 Wire Wire Line
 	4900 5100 5350 5100
-Text Notes 5900 4950 0    50   ~ 0
-These caps. have to be placed at each VDD pin. One cap per VDD pin.
 Text Notes 3900 2300 0    100  ~ 20
 EEPROM
@@
 Addr: 0x50
 Text Notes 4500 6050 0    50   ~ 0
-Addr: 0x65
-$Comp
-L Jumper:SolderJumper_3_Bridged12 JP5
-U 1 1 5CA180BC
-P 7400 5500
-F 0 "JP5" V 7446 5568 50  0000 L CNN
-F 1 "SolderJumper_3_Open" V 7355 5568 50  0000 L CNN
-F 2 "Jumper:SolderJumper-3_P1.3mm_Bridged12_Pad1.0x1.5mm" H 7400 5500 50  0001 C CNN
-F 3 "~" H 7400 5500 50  0001 C CNN
-	1    7400 5500
-	0    1    -1   0
-$EndComp
-Wire Wire Line
-	7250 5500 7050 5500
-$Comp
-L power:GND #PWR068
-U 1 1 5CA180C5
-P 7400 5750
-F 0 "#PWR068" H 7400 5500 50  0001 C CNN
-F 1 "GND" H 7405 5577 50  0000 C CNN
-F 2 "" H 7400 5750 50  0001 C CNN
-F 3 "" H 7400 5750 50  0001 C CNN
-	1    7400 5750
-	1    0    0    -1
-$EndComp
-Wire Wire Line
-	7400 5700 7400 5750
-$Comp
-L power:+3.3V #PWR066
-U 1 1 5CA180CC
-P 7400 5250
-F 0 "#PWR066" H 7400 5100 50  0001 C CNN
-F 1 "+3.3V" H 7415 5423 50  0000 C CNN
-F 2 "" H 7400 5250 50  0001 C CNN
-F 3 "" H 7400 5250 50  0001 C CNN
-	1    7400 5250
-	1    0    0    -1
-$EndComp
-Wire Wire Line
-	7400 5250 7400 5300
-Text Label 7050 5500 0    50   ~ 0
-SA0
+Addr: 0x64
 Text Label 3250 5200 0    50   ~ 0
 SA0
@@
 Wire Wire Line
 	3650 5400 3700 5400
-$Comp
-L power:PWR_FLAG #FLG05
-U 1 1 5CC89108
-P 5200 2900
-F 0 "#FLG05" H 5200 2975 50  0001 C CNN
-F 1 "PWR_FLAG" V 5200 3028 50  0000 L CNN
-F 2 "" H 5200 2900 50  0001 C CNN
-F 3 "~" H 5200 2900 50  0001 C CNN
-	1    5200 2900
-	0    1    1    0
-$EndComp
-$Comp
-L power:PWR_FLAG #FLG06
-U 1 1 5CC89201
-P 5200 3000
-F 0 "#FLG06" H 5200 3075 50  0001 C CNN
-F 1 "PWR_FLAG" V 5200 3128 50  0000 L CNN
-F 2 "" H 5200 3000 50  0001 C CNN
-F 3 "~" H 5200 3000 50  0001 C CNN
-	1    5200 3000
-	0    1    1    0
-$EndComp
-$Comp
-L power:PWR_FLAG #FLG07
-U 1 1 5CC89222
-P 5200 3100
-F 0 "#FLG07" H 5200 3175 50  0001 C CNN
-F 1 "PWR_FLAG" V 5200 3228 50  0000 L CNN
-F 2 "" H 5200 3100 50  0001 C CNN
-F 3 "~" H 5200 3100 50  0001 C CNN
-	1    5200 3100
-	0    1    1    0
-$EndComp
+Wire Wire Line
+	3700 5600 3650 5600
+Wire Wire Line
+	3650 5600 3650 5400
+Wire Wire Line
+	4850 3200 4850 3100
+Wire Wire Line
+	4850 2900 4750 2900
+Wire Wire Line
+	4750 3000 4850 3000
+Connection ~ 4850 3000
+Wire Wire Line
+	4850 3000 4850 2900
+Wire Wire Line
+	4750 3100 4850 3100
+Connection ~ 4850 3100
+Wire Wire Line
+	4850 3100 4850 3000
 $EndSCHEMATC

Commit message: Organized all components in BPS master to where they should be.
Parts:
- removed C32, C33: 0.1uF, Capacitor_SMD:C_0805_2012Metric, symbol Device:C
- removed U9: LSM6DS3, Package_LGA:LGA-14_3x2.5mm_P0.5mm_LayoutBorder3x4y, symbol Sensor_Motion:LSM6DS3
Connections:
- net labels removed: SA0
- wire segments 53 -> 29
- no-connect marks 3 -> 0
Other:
- note removed: "Addr: 0x64"
- note removed: "IMU"
Changed lines of the file:
@@
 Text Label 3600 3200 2    50   ~ 0
 SDA
-$Comp
-L Sensor_Motion:LSM6DS3 U9
-U 1 1 5CA092E2
-P 4300 5500
-F 0 "U9" H 4941 5546 50  0000 L CNN
-F 1 "LSM6DS3" H 4941 5455 50  0000 L CNN
-F 2 "Package_LGA:LGA-14_3x2.5mm_P0.5mm_LayoutBorder3x4y" H 3900 4800 50  0001 L CNN
-F 3 "www.st.com/resource/en/datasheet/lsm6ds3.pdf" H 4400 4850 50  0001 C CNN
-	1    4300 5500
-	1    0    0    -1
-$EndComp
-$Comp
-L power:GND #PWR069
-U 1 1 5CA0937C
-P 4400 6200
-F 0 "#PWR069" H 4400 5950 50  0001 C CNN
-F 1 "GND" H 4405 6027 50  0000 C CNN
-F 2 "" H 4400 6200 50  0001 C CNN
-F 3 "" H 4400 6200 50  0001 C CNN
-	1    4400 6200
-	1    0    0    -1
-$EndComp
-Wire Wire Line
-	4400 6200 4400 6150
-Wire Wire Line
-	4400 6150 4300 6150
-Wire Wire Line
-	4300 6150 4300 6100
-Connection ~ 4400 6150
-Wire Wire Line
-	4400 6150 4400 6100
-$Comp
-L power:+3.3V #PWR064
-U 1 1 5CA0A32E
-P 4300 4650
-F 0 "#PWR064" H 4300 4500 50  0001 C CNN
-F 1 "+3.3V" H 4315 4823 50  0000 C CNN
-F 2 "" H 4300 4650 50  0001 C CNN
-F 3 "" H 4300 4650 50  0001 C CNN
-	1    4300 4650
-	1    0    0    -1
-$EndComp
-Wire Wire Line
-	4300 4650 4300 4700
-Wire Wire Line
-	4300 4700 4400 4700
-Connection ~ 4300 4700
-Wire Wire Line
-	3700 5700 3250 5700
-Text Label 3250 5700 0    50   ~ 0
-SCL
-$Comp
-L Device:C C32
-U 1 1 5CA0C7FA
-P 4900 4900
-F 0 "C32" H 5015 4946 50  0000 L CNN
-F 1 "0.1uF" H 5015 4855 50  0000 L CNN
-F 2 "Capacitor_SMD:C_0805_2012Metric" H 4938 4750 50  0001 C CNN
-F 3 "~" H 4900 4900 50  0001 C CNN
-	1    4900 4900
-	1    0    0    -1
-$EndComp
-$Comp
-L Device:C C33
-U 1 1 5CA0C84A
-P 5350 4900
-F 0 "C33" H 5465 4946 50  0000 L CNN
-F 1 "0.1uF" H 5465 4855 50  0000 L CNN
-F 2 "Capacitor_SMD:C_0805_2012Metric" H 5388 4750 50  0001 C CNN
-F 3 "~" H 5350 4900 50  0001 C CNN
-	1    5350 4900
-	1    0    0    -1
-$EndComp
-$Comp
-L power:GND #PWR065
-U 1 1 5CA0C8C8
-P 5350 5150
-F 0 "#PWR065" H 5350 4900 50  0001 C CNN
-F 1 "GND" H 5355 4977 50  0000 C CNN
-F 2 "" H 5350 5150 50  0001 C CNN
-F 3 "" H 5350 5150 50  0001 C CNN
-	1    5350 5150
-	1    0    0    -1
-$EndComp
-Wire Wire Line
-	5350 5150 5350 5100
-Wire Wire Line
-	4900 5100 4900 5050
-Connection ~ 5350 5100
-Wire Wire Line
-	5350 5100 5350 5050
-NoConn ~ 4900 5200
-NoConn ~ 4900 5300
-Wire Wire Line
-	4900 4750 4900 4700
-Wire Wire Line
-	4900 4700 4400 4700
-Connection ~ 4900 4700
-Connection ~ 4400 4700
-Wire Wire Line
-	4400 4700 4400 4900
-Wire Wire Line
-	4300 4700 4300 4900
-Wire Wire Line
-	5350 4750 5350 4700
-Wire Wire Line
-	4900 4700 5350 4700
-Wire Wire Line
-	4900 5100 5350 5100
 Text Notes 3900 2300 0    100  ~ 20
 EEPROM
-Text Notes 4200 4250 0    100  ~ 20
-IMU
-NoConn ~ 3700 5800
 Text Notes 3950 3400 0    50   ~ 0
 Addr: 0x50
-Text Notes 4500 6050 0    50   ~ 0
-Addr: 0x64
-Text Label 3250 5200 0    50   ~ 0
-SA0
-Wire Wire Line
-	3250 5200 3700 5200
-$Comp
-L power:GND #PWR067
-U 1 1 5CA1AF1B
-P 3550 5400
-F 0 "#PWR067" H 3550 5150 50  0001 C CNN
-F 1 "GND" H 3555 5227 50  0000 C CNN
-F 2 "" H 3550 5400 50  0001 C CNN
-F 3 "" H 3550 5400 50  0001 C CNN
-	1    3550 5400
-	0    1    1    0
-$EndComp
-Wire Wire Line
-	3550 5400 3650 5400
-Wire Wire Line
-	3650 5400 3650 5300
-Wire Wire Line
-	3650 5300 3700 5300
-Connection ~ 3650 5400
-Wire Wire Line
-	3650 5400 3700 5400
-Wire Wire Line
-	3700 5600 3650 5600
-Wire Wire Line
-	3650 5600 3650 5400
 Wire Wire Line
 	4850 3200 4850 3100

Commit message: Completed master board PCB
Parts:
- added J14: Conn_01x03, Connector_PinHeader_2.54mm:PinHeader_1x02_P2.54mm_Vertical, symbol Connector_Generic:Conn_01x02
Connections:
- wire segments 29 -> 33
Changed lines of the file:
@@
 $Descr A4 11693 8268
 encoding utf-8
-Sheet 5 8
+Sheet 5 7
 Title ""
 Date ""
@@
 Wire Wire Line
 	2400 3100 2400 3000
-Wire Wire Line
-	2400 3100 3750 3100
 Connection ~ 2400 3100
 Wire Wire Line
@@
 Wire Wire Line
 	2800 3000 2800 3200
-Wire Wire Line
-	2800 3200 2300 3200
-Wire Wire Line
-	2800 3200 3750 3200
 Connection ~ 2800 3200
 Wire Wire Line
@@
 Wire Wire Line
 	4850 3100 4850 3000
+$Comp
+L Connector_Generic:Conn_01x02 J14
+U 1 1 5C646686
+P 2600 3700
+F 0 "J14" V 2473 3780 50  0000 L CNN
+F 1 "Conn_01x03" V 2564 3780 50  0000 L CNN
+F 2 "Connector_PinHeader_2.54mm:PinHeader_1x02_P2.54mm_Vertical" H 2600 3700 50  0001 C CNN
+F 3 "~" H 2600 3700 50  0001 C CNN
+	1    2600 3700
+	0    1    1    0
+$EndComp
+Wire Wire Line
+	2800 3200 3750 3200
+Wire Wire Line
+	2400 3100 2600 3100
+Wire Wire Line
+	2600 3500 2600 3100
+Connection ~ 2600 3100
+Wire Wire Line
+	2600 3100 3750 3100
+Wire Wire Line
+	2500 3500 2500 3200
+Wire Wire Line
+	2300 3200 2500 3200
+Connection ~ 2500 3200
+Wire Wire Line
+	2500 3200 2800 3200
 $EndSCHEMATC
