File: Electronics/BPS/Master/Misc.sch (KiCad schematic (older format))
At the start: 5 parts

Commit message: Added LTC6811 symbol for BPS voltage schematics.
Parts:
- added U?: SI8261ABC-IS, symbol utsvt-bps:SI8261ABC-IS
Changed lines of the file:
@@
 Text Notes 6000 2150 0    100  ~ 20
 Error Light
+$Comp
+L utsvt-bps:SI8261ABC-IS U?
+U 1 1 5C35EBB6
+P 4750 2900
+F 0 "U?" H 4750 3065 50  0000 C CNN
+F 1 "SI8261ABC-IS" H 4750 2974 50  0000 C CNN
+F 2 "" H 4750 2900 50  0001 C CNN
+F 3 "" H 4750 2900 50  0001 C CNN
+	1    4750 2900
+	1    0    0    -1
+$EndComp
 $EndSCHEMATC

Commit message: Finalized schematics for BPS master.
Parts:
- added C52: 1uF, symbol Device:C
- added C53: 10uF, symbol Device:C
- added C54: 0.1uF, symbol Device:C
- added D10: OCurr, symbol Device:LED_ALT
- added D11: WDError, symbol Device:LED_ALT
- added D12: CANError, symbol Device:LED_ALT
- added D4: 1N4148WS, Diode_SMD:D_SOD-323, symbol Device:D_ALT
- added D5: Fault, symbol Device:LED_ALT
- added D6: Heartbeat, symbol Device:LED_ALT
- added D7: OVolt, symbol Device:LED_ALT
- added D8: UVolt, symbol Device:LED_ALT
- added D9: OTemp, symbol Device:LED_ALT
- added J16: Fan5, symbol Connector_Generic:Conn_01x02
- added J17: Fan6, symbol Connector_Generic:Conn_01x02
- added J18: Fan7, symbol Connector_Generic:Conn_01x02
- added J19: Fan8, symbol Connector_Generic:Conn_01x02
- added Q3, Q4: NVR4003NT3G, Package_TO_SOT_SMD:SOT-23, symbol Device:Q_NMOS_GSD
- added R39: 5.1k, symbol Device:R
- added R40: 220, symbol Device:R
- added R41: 0, symbol Device:R
- added R42: 100k, symbol Device:R
- added R43: 680, symbol Device:R
- added R44, R45, R46, R47, R48, R49: 750, symbol Device:R
- added TP16: Gate_TP, symbol Connector:TestPoint
- gave numbers to parts that had none: 6
Connections:
- net labels added: +3.3V, GNDPWR, PA5, PA6, PA[5..6], PC0, PC1, PC2, PC3, PC4, PC5, PC[0..5]
- wire segments 16 -> 114
- no-connect marks 0 -> 3
Other:
- note added: "Green LEDs good"
- note added: "Please check footprint and symbol matches!\n1: G\n2: D\n3: S"
- note added: "Red LEDs fault"
- note added: "Status LEDs"

Commit message: Added SoC skeleton code.
Parts:
- added R45: 0, symbol Device:R
- added R46: 100k, symbol Device:R
- C52: footprint (none) -> Capacitor_SMD:C_0805_2012Metric
- R41: renamed from R39; value 5.1k -> 1.6k
- R42: renamed from R40; value 220 -> 470
- TP16: value Gate_TP -> StrobeLightGate_TP; footprint (none) -> TestPoint:TestPoint_Keystone_5005-5009_Compact
- renumbered R41 to R43, R42 to R44, R43 to R47, R44 to R48, R45 to R49, R46 to R50, R47 to R51, R48 to R52, R49 to R53
Connections:
- net labels added: +5V
- net labels removed: +3.3V
- wire segments 114 -> 119
Changed lines of the file:
@@
 	1    0    0    -1
 $EndComp
-Text HLabel 2000 4150 0    50   Input ~ 0
+Text HLabel 1550 4250 0    50   Input ~ 0
 GND
 $Comp
-L Device:R R40
+L Device:R R42
 U 1 1 5C36C3FE
 P 2500 3150
-F 0 "R40" H 2400 3100 50  0000 C CNN
-F 1 "220" V 2500 3150 50  0000 C CNN
+F 0 "R42" H 2400 3100 50  0000 C CNN
+F 1 "470" V 2500 3150 50  0000 C CNN
 F 2 "" V 2430 3150 50  0001 C CNN
 F 3 "~" H 2500 3150 50  0001 C CNN
@@
 $EndComp
 Wire Wire Line
-	1800 3850 1600 3850
+	1200 3850 1000 3850
 NoConn ~ 2800 3250
 NoConn ~ 2800 3550
@@
 P 4800 3700
 AR Path="/5C38C674/5C372AA5" Ref="R?"  Part="1"
-AR Path="/5C392C6A/5C372AA5" Ref="R42"  Part="1"
-F 0 "R42" H 4850 3700 50  0000 L CNN
+AR Path="/5C392C6A/5C372AA5" Ref="R44"  Part="1"
+F 0 "R44" H 4850 3700 50  0000 L CNN
 F 1 "100k" V 4800 3600 50  0000 L CNN
 F 2 "" V 4730 3700 50  0001 C CNN
@@
 P 4550 3450
 AR Path="/5C38C674/5C372AB3" Ref="R?"  Part="1"
-AR Path="/5C392C6A/5C372AB3" Ref="R41"  Part="1"
-F 0 "R41" V 4450 3450 50  0000 C CNN
+AR Path="/5C392C6A/5C372AB3" Ref="R43"  Part="1"
+F 0 "R43" V 4450 3450 50  0000 C CNN
 F 1 "0" V 4550 3450 50  0000 C CNN
 F 2 "" V 4480 3450 50  0001 C CNN
@@
 AR Path="/5C392C6A/5C372ACD" Ref="TP16"  Part="1"
 F 0 "TP16" H 4258 3420 50  0000 L CNN
-F 1 "Gate_TP" H 4258 3329 50  0000 L CNN
-F 2 "" H 4400 3300 50  0001 C CNN
+F 1 "StrobeLightGate_TP" H 4258 3329 50  0000 L CNN
+F 2 "TestPoint:TestPoint_Keystone_5005-5009_Compact" H 4400 3300 50  0001 C CNN
 F 3 "~" H 4400 3300 50  0001 C CNN
 	1    4200 3300
@@
 P 2100 3000
 AR Path="/5C38C674/5C372AD7" Ref="R?"  Part="1"
-AR Path="/5C392C6A/5C372AD7" Ref="R39"  Part="1"
-F 0 "R39" H 2170 3046 50  0000 L CNN
-F 1 "5.1k" V 2100 2900 50  0000 L CNN
+AR Path="/5C392C6A/5C372AD7" Ref="R41"  Part="1"
+F 0 "R41" H 2170 3046 50  0000 L CNN
+F 1 "1.6k" V 2100 2900 50  0000 L CNN
 F 2 "" V 2030 3000 50  0001 C CNN
 F 3 "~" H 2100 3000 50  0001 C CNN
@@
 F 0 "C52" V 5298 2500 50  0000 C CNN
 F 1 "1uF" V 5389 2500 50  0000 C CNN
-F 2 "" H 5588 2350 50  0001 C CNN
+F 2 "Capacitor_SMD:C_0805_2012Metric" H 5588 2350 50  0001 C CNN
 F 3 "~" H 5550 2500 50  0001 C CNN
 	1    5550 2500
@@
 	3800 6400 4200 6400
 $Comp
-L Device:R R43
+L Device:R R47
 U 1 1 5C3C06D9
 P 2950 5800
-F 0 "R43" H 3020 5846 50  0000 L CNN
+F 0 "R47" H 3020 5846 50  0000 L CNN
 F 1 "680" H 3020 5755 50  0000 L CNN
 F 2 "" V 2880 5800 50  0001 C CNN
@@
 $EndComp
 $Comp
-L Device:R R44
+L Device:R R48
 U 1 1 5C3C06E0
 P 3800 5800
-F 0 "R44" H 3870 5846 50  0000 L CNN
+F 0 "R48" H 3870 5846 50  0000 L CNN
 F 1 "750" H 3870 5755 50  0000 L CNN
 F 2 "" V 3730 5800 50  0001 C CNN
@@
 $EndComp
 $Comp
-L Device:R R45
+L Device:R R49
 U 1 1 5C3C06E7
 P 4200 5800
-F 0 "R45" H 4270 5846 50  0000 L CNN
+F 0 "R49" H 4270 5846 50  0000 L CNN
 F 1 "750" H 4270 5755 50  0000 L CNN
 F 2 "" V 4130 5800 50  0001 C CNN
@@
 $EndComp
 $Comp
-L Device:R R46
+L Device:R R50
 U 1 1 5C3C06EE
 P 4600 5800
-F 0 "R46" H 4670 5846 50  0000 L CNN
+F 0 "R50" H 4670 5846 50  0000 L CNN
 F 1 "750" H 4670 5755 50  0000 L CNN
 F 2 "" V 4530 5800 50  0001 C CNN
@@
 $EndComp
 $Comp
-L Device:R R47
+L Device:R R51
 U 1 1 5C3C06F5
 P 5000 5800
-F 0 "R47" H 5070 5846 50  0000 L CNN
+F 0 "R51" H 5070 5846 50  0000 L CNN
 F 1 "750" H 5070 5755 50  0000 L CNN
 F 2 "" V 4930 5800 50  0001 C CNN
@@
 	5000 6400 5400 6400
 $Comp
-L Device:R R48
+L Device:R R52
 U 1 1 5C3C0718
 P 5400 5800
-F 0 "R48" H 5470 5846 50  0000 L CNN
+F 0 "R52" H 5470 5846 50  0000 L CNN
 F 1 "750" H 5470 5755 50  0000 L CNN
 F 2 "" V 5330 5800 50  0001 C CNN
@@
 Text Label 2650 4700 3    50   ~ 0
 PC1
-Text Label 1600 3850 0    50   ~ 0
+Text Label 1000 3850 0    50   ~ 0
 PC1
 $Comp
@@
 	5900 6400 5900 6300
 $Comp
-L Device:R R49
+L Device:R R53
 U 1 1 5C6CF943
 P 5900 5800
-F 0 "R49" H 5970 5846 50  0000 L CNN
+F 0 "R53" H 5970 5846 50  0000 L CNN
 F 1 "750" H 5970 5755 50  0000 L CNN
 F 2 "" V 5830 5800 50  0001 C CNN
@@
 	1    0    0    -1
 $EndComp
-$Comp
-L power:+3.3V #PWR0116
-U 1 1 5C986786
+Wire Wire Line
+	2500 2650 2500 2750
+Connection ~ 2100 2750
+$Comp
+L power:GND #PWR0120
+U 1 1 5C98DE41
+P 2100 4350
+F 0 "#PWR0120" H 2100 4100 50  0001 C CNN
+F 1 "GND" H 2105 4177 50  0000 C CNN
+F 2 "" H 2100 4350 50  0001 C CNN
+F 3 "" H 2100 4350 50  0001 C CNN
+	1    2100 4350
+	1    0    0    -1
+$EndComp
+Wire Wire Line
+	2100 4350 2100 4250
+Connection ~ 2100 4250
+Wire Wire Line
+	2100 3500 2100 3600
+Wire Wire Line
+	2100 3600 2500 3600
+Wire Wire Line
+	2500 3600 2500 3450
+Connection ~ 2100 3600
+Wire Wire Line
+	2100 3600 2100 3650
+Wire Wire Line
+	2500 3350 2800 3350
+Wire Wire Line
+	2500 3450 2800 3450
+Text HLabel 2000 2750 0    50   Input ~ 0
++5V
+Wire Wire Line
+	2000 2750 2100 2750
+Connection ~ 2500 2750
+NoConn ~ 3900 3350
+$Comp
+L power:+5V #PWR0116
+U 1 1 5C39A4BC
 P 2500 2650
 F 0 "#PWR0116" H 2500 2500 50  0001 C CNN
-F 1 "+3.3V" H 2515 2823 50  0000 C CNN
+F 1 "+5V" H 2515 2823 50  0000 C CNN
 F 2 "" H 2500 2650 50  0001 C CNN
 F 3 "" H 2500 2650 50  0001 C CNN
@@
 	1    0    0    -1
 $EndComp
-Wire Wire Line
-	2500 2650 2500 2750
-Connection ~ 2100 2750
-Wire Wire Line
-	2100 4050 2100 4150
-Wire Wire Line
-	2100 4150 2000 4150
-$Comp
-L power:GND #PWR0120
-U 1 1 5C98DE41
-P 2100 4250
-F 0 "#PWR0120" H 2100 4000 50  0001 C CNN
-F 1 "GND" H 2105 4077 50  0000 C CNN
-F 2 "" H 2100 4250 50  0001 C CNN
-F 3 "" H 2100 4250 50  0001 C CNN
-	1    2100 4250
-	1    0    0    -1
-$EndComp
-Wire Wire Line
-	2100 4250 2100 4150
-Connection ~ 2100 4150
-Wire Wire Line
-	2100 3500 2100 3600
-Wire Wire Line
-	2100 3600 2500 3600
-Wire Wire Line
-	2500 3600 2500 3450
-Connection ~ 2100 3600
-Wire Wire Line
-	2100 3600 2100 3650
-Wire Wire Line
-	2500 3350 2800 3350
-Wire Wire Line
-	2500 3450 2800 3450
-Text HLabel 2000 2750 0    50   Input ~ 0
-+3.3V
-Wire Wire Line
-	2000 2750 2100 2750
-Connection ~ 2500 2750
-NoConn ~ 3900 3350
+$Comp
+L Device:R R?
+U 1 1 5C39AAD5
+P 1350 3850
+AR Path="/5C38C674/5C39AAD5" Ref="R?"  Part="1"
+AR Path="/5C392C6A/5C39AAD5" Ref="R45"  Part="1"
+F 0 "R45" V 1250 3850 50  0000 C CNN
+F 1 "0" V 1350 3850 50  0000 C CNN
+F 2 "" V 1280 3850 50  0001 C CNN
+F 3 "~" H 1350 3850 50  0001 C CNN
+	1    1350 3850
+	0    1    1    0
+$EndComp
+$Comp
+L Device:R R?
+U 1 1 5C39EDC5
+P 1650 4050
+AR Path="/5C38C674/5C39EDC5" Ref="R?"  Part="1"
+AR Path="/5C392C6A/5C39EDC5" Ref="R46"  Part="1"
+F 0 "R46" H 1700 4050 50  0000 L CNN
+F 1 "100k" V 1650 3950 50  0000 L CNN
+F 2 "" V 1580 4050 50  0001 C CNN
+F 3 "~" H 1650 4050 50  0001 C CNN
+	1    1650 4050
+	1    0    0    -1
+$EndComp
+Wire Wire Line
+	1500 3850 1650 3850
+Wire Wire Line
+	1650 3850 1650 3900
+Connection ~ 1650 3850
+Wire Wire Line
+	1650 3850 1800 3850
+Wire Wire Line
+	1550 4250 1650 4250
+Wire Wire Line
+	1650 4250 1650 4200
+Wire Wire Line
+	1650 4250 2100 4250
+Connection ~ 1650 4250
+Wire Wire Line
+	2100 4050 2100 4250
 Wire Bus Line
 	5500 5200 6100 5200

Commit message: Assigned footprints to each symbol in BPS schematics.
Parts:
- C49: renamed from C53; footprint (none) -> Capacitor_SMD:C_0805_2012Metric
- C50: renamed from C54; footprint (none) -> Capacitor_SMD:C_0805_2012Metric
- D10, D11, D12, D5, D6, D7, D8, D9: footprint (none) -> LED_SMD:LED_0805_2012Metric
- J11, J12, J13, J14, J15, J16, J17, J18, J19: footprint (none) -> UTSVT_Connectors:Molex_MicroFit3.0_1x2xP3.00mm_PolarizingPeg_Vertical
- R41, R42, R43, R44, R45, R46, R47, R48, R49, R50, R51, R52, R53: footprint (none) -> Resistor_SMD:R_0805_2012Metric
- U16: footprint (none) -> Package_SO:SOIC-8_3.9x4.9mm_P1.27mm
- renumbered C52 to C48, TP16 to TP14
Changed lines of the file:
@@
 F 0 "J11" H 8430 2442 50  0000 L CNN
 F 1 "Fan1" H 8430 2351 50  0000 L CNN
-F 2 "" H 8350 2450 50  0001 C CNN
+F 2 "UTSVT_Connectors:Molex_MicroFit3.0_1x2xP3.00mm_PolarizingPeg_Vertical" H 8350 2450 50  0001 C CNN
 F 3 "~" H 8350 2450 50  0001 C CNN
 	1    8350 2450
@@
 F 0 "J12" H 8430 2742 50  0000 L CNN
 F 1 "Fan2" H 8430 2651 50  0000 L CNN
-F 2 "" H 8350 2750 50  0001 C CNN
+F 2 "UTSVT_Connectors:Molex_MicroFit3.0_1x2xP3.00mm_PolarizingPeg_Vertical" H 8350 2750 50  0001 C CNN
 F 3 "~" H 8350 2750 50  0001 C CNN
 	1    8350 2750
@@
 F 0 "J14" H 8430 3042 50  0000 L CNN
 F 1 "Fan3" H 8430 2951 50  0000 L CNN
-F 2 "" H 8350 3050 50  0001 C CNN
+F 2 "UTSVT_Connectors:Molex_MicroFit3.0_1x2xP3.00mm_PolarizingPeg_Vertical" H 8350 3050 50  0001 C CNN
 F 3 "~" H 8350 3050 50  0001 C CNN
 	1    8350 3050
@@
 F 0 "J15" H 8430 3342 50  0000 L CNN
 F 1 "Fan4" H 8430 3251 50  0000 L CNN
-F 2 "" H 8350 3350 50  0001 C CNN
+F 2 "UTSVT_Connectors:Molex_MicroFit3.0_1x2xP3.00mm_PolarizingPeg_Vertical" H 8350 3350 50  0001 C CNN
 F 3 "~" H 8350 3350 50  0001 C CNN
 	1    8350 3350
@@
 F 0 "J13" H 5580 2942 50  0000 L CNN
 F 1 "ErrorLightConnector" H 5580 2851 50  0000 L CNN
-F 2 "" H 5500 2950 50  0001 C CNN
+F 2 "UTSVT_Connectors:Molex_MicroFit3.0_1x2xP3.00mm_PolarizingPeg_Vertical" H 5500 2950 50  0001 C CNN
 F 3 "~" H 5500 2950 50  0001 C CNN
 	1    5500 2950
@@
 F 0 "U16" H 3350 2500 50  0000 C CNN
 F 1 "SI8261ABC-IS" H 3350 2600 50  0000 C CNN
-F 2 "" H 3350 3150 50  0001 C CNN
+F 2 "Package_SO:SOIC-8_3.9x4.9mm_P1.27mm" H 3350 3150 50  0001 C CNN
 F 3 "" H 3350 3150 50  0001 C CNN
 	1    3350 3150
@@
 F 0 "R42" H 2400 3100 50  0000 C CNN
 F 1 "470" V 2500 3150 50  0000 C CNN
-F 2 "" V 2430 3150 50  0001 C CNN
+F 2 "Resistor_SMD:R_0805_2012Metric" V 2430 3150 50  0001 C CNN
 F 3 "~" H 2500 3150 50  0001 C CNN
 	1    2500 3150
@@
 $EndComp
 $Comp
-L Device:C C53
+L Device:C C49
 U 1 1 5C36F4C8
 P 3150 2650
-F 0 "C53" H 3265 2696 50  0000 L CNN
+F 0 "C49" H 3265 2696 50  0000 L CNN
 F 1 "10uF" H 3265 2605 50  0000 L CNN
-F 2 "" H 3188 2500 50  0001 C CNN
+F 2 "Capacitor_SMD:C_0805_2012Metric" H 3188 2500 50  0001 C CNN
 F 3 "~" H 3150 2650 50  0001 C CNN
 	1    3150 2650
@@
 	3150 2400 3150 2450
 $Comp
-L Device:C C54
+L Device:C C50
 U 1 1 5C36FD88
 P 3600 2650
-F 0 "C54" H 3715 2696 50  0000 L CNN
+F 0 "C50" H 3715 2696 50  0000 L CNN
 F 1 "0.1uF" H 3715 2605 50  0000 L CNN
-F 2 "" H 3638 2500 50  0001 C CNN
+F 2 "Capacitor_SMD:C_0805_2012Metric" H 3638 2500 50  0001 C CNN
 F 3 "~" H 3600 2650 50  0001 C CNN
 	1    3600 2650
@@
 F 0 "R44" H 4850 3700 50  0000 L CNN
 F 1 "100k" V 4800 3600 50  0000 L CNN
-F 2 "" V 4730 3700 50  0001 C CNN
+F 2 "Resistor_SMD:R_0805_2012Metric" V 4730 3700 50  0001 C CNN
 F 3 "~" H 4800 3700 50  0001 C CNN
 	1    4800 3700
@@
 F 0 "R43" V 4450 3450 50  0000 C CNN
 F 1 "0" V 4550 3450 50  0000 C CNN
-F 2 "" V 4480 3450 50  0001 C CNN
+F 2 "Resistor_SMD:R_0805_2012Metric" V 4480 3450 50  0001 C CNN
 F 3 "~" H 4550 3450 50  0001 C CNN
 	1    4550 3450
@@
 P 4200 3300
 AR Path="/5C38C674/5C372ACD" Ref="TP?"  Part="1"
-AR Path="/5C392C6A/5C372ACD" Ref="TP16"  Part="1"
-F 0 "TP16" H 4258 3420 50  0000 L CNN
+AR Path="/5C392C6A/5C372ACD" Ref="TP14"  Part="1"
+F 0 "TP14" H 4258 3420 50  0000 L CNN
 F 1 "StrobeLightGate_TP" H 4258 3329 50  0000 L CNN
 F 2 "TestPoint:TestPoint_Keystone_5005-5009_Compact" H 4400 3300 50  0001 C CNN
@@
 F 0 "R41" H 2170 3046 50  0000 L CNN
 F 1 "1.6k" V 2100 2900 50  0000 L CNN
-F 2 "" V 2030 3000 50  0001 C CNN
+F 2 "Resistor_SMD:R_0805_2012Metric" V 2030 3000 50  0001 C CNN
 F 3 "~" H 2100 3000 50  0001 C CNN
 	1    2100 3000
@@
 P 5550 2500
 AR Path="/5C38C674/5C372AF8" Ref="C?"  Part="1"
-AR Path="/5C392C6A/5C372AF8" Ref="C52"  Part="1"
-F 0 "C52" V 5298 2500 50  0000 C CNN
+AR Path="/5C392C6A/5C372AF8" Ref="C48"  Part="1"
+F 0 "C48" V 5298 2500 50  0000 C CNN
 F 1 "1uF" V 5389 2500 50  0000 C CNN
 F 2 "Capacitor_SMD:C_0805_2012Metric" H 5588 2350 50  0001 C CNN
@@
 F 0 "D5" V 2138 3233 50  0000 R CNN
 F 1 "Fault" V 2047 3233 50  0000 R CNN
-F 2 "" H 2100 3350 50  0001 C CNN
+F 2 "LED_SMD:LED_0805_2012Metric" H 2100 3350 50  0001 C CNN
 F 3 "~" H 2100 3350 50  0001 C CNN
 F 4 "Red" V 2100 3350 50  0001 C CNN "Color"
@@
 F 0 "D6" V 2988 6033 50  0000 R CNN
 F 1 "Heartbeat" V 2897 6033 50  0000 R CNN
-F 2 "" H 2950 6150 50  0001 C CNN
+F 2 "LED_SMD:LED_0805_2012Metric" H 2950 6150 50  0001 C CNN
 F 3 "~" H 2950 6150 50  0001 C CNN
 F 4 "Green" V 2950 6150 50  0001 C CNN "Color"
@@
 F 0 "D7" V 3838 6032 50  0000 R CNN
 F 1 "OVolt" V 3747 6032 50  0000 R CNN
-F 2 "" H 3800 6150 50  0001 C CNN
+F 2 "LED_SMD:LED_0805_2012Metric" H 3800 6150 50  0001 C CNN
 F 3 "~" H 3800 6150 50  0001 C CNN
 F 4 "Red" V 3800 6150 50  0001 C CNN "Color"
@@
 F 0 "D8" V 4238 6032 50  0000 R CNN
 F 1 "UVolt" V 4147 6032 50  0000 R CNN
-F 2 "" H 4200 6150 50  0001 C CNN
+F 2 "LED_SMD:LED_0805_2012Metric" H 4200 6150 50  0001 C CNN
 F 3 "~" H 4200 6150 50  0001 C CNN
 F 4 "Red" V 4200 6150 50  0001 C CNN "Color"
@@
 F 0 "D9" V 4638 6032 50  0000 R CNN
 F 1 "OTemp" V 4547 6032 50  0000 R CNN
-F 2 "" H 4600 6150 50  0001 C CNN
+F 2 "LED_SMD:LED_0805_2012Metric" H 4600 6150 50  0001 C CNN
 F 3 "~" H 4600 6150 50  0001 C CNN
 F 4 "Red" V 4600 6150 50  0001 C CNN "Color"
@@
 F 0 "D10" V 5038 6033 50  0000 R CNN
 F 1 "OCurr" V 4947 6033 50  0000 R CNN
-F 2 "" H 5000 6150 50  0001 C CNN
+F 2 "LED_SMD:LED_0805_2012Metric" H 5000 6150 50  0001 C CNN
 F 3 "~" H 5000 6150 50  0001 C CNN
 F 4 "Red" V 5000 6150 50  0001 C CNN "Color"
@@
 F 0 "R47" H 3020 5846 50  0000 L CNN
 F 1 "680" H 3020 5755 50  0000 L CNN
-F 2 "" V 2880 5800 50  0001 C CNN
+F 2 "Resistor_SMD:R_0805_2012Metric" V 2880 5800 50  0001 C CNN
 F 3 "~" H 2950 5800 50  0001 C CNN
 	1    2950 5800
@@
 F 0 "R48" H 3870 5846 50  0000 L CNN
 F 1 "750" H 3870 5755 50  0000 L CNN
-F 2 "" V 3730 5800 50  0001 C CNN
+F 2 "Resistor_SMD:R_0805_2012Metric" V 3730 5800 50  0001 C CNN
 F 3 "~" H 3800 5800 50  0001 C CNN
 	1    3800 5800
@@
 F 0 "R49" H 4270 5846 50  0000 L CNN
 F 1 "750" H 4270 5755 50  0000 L CNN
-F 2 "" V 4130 5800 50  0001 C CNN
+F 2 "Resistor_SMD:R_0805_2012Metric" V 4130 5800 50  0001 C CNN
 F 3 "~" H 4200 5800 50  0001 C CNN
 	1    4200 5800
@@
 F 0 "R50" H 4670 5846 50  0000 L CNN
 F 1 "750" H 4670 5755 50  0000 L CNN
-F 2 "" V 4530 5800 50  0001 C CNN
+F 2 "Resistor_SMD:R_0805_2012Metric" V 4530 5800 50  0001 C CNN
 F 3 "~" H 4600 5800 50  0001 C CNN
 	1    4600 5800
@@
 F 0 "R51" H 5070 5846 50  0000 L CNN
 F 1 "750" H 5070 5755 50  0000 L CNN
-F 2 "" V 4930 5800 50  0001 C CNN
+F 2 "Resistor_SMD:R_0805_2012Metric" V 4930 5800 50  0001 C CNN
 F 3 "~" H 5000 5800 50  0001 C CNN
 	1    5000 5800
@@
 F 0 "D11" V 5438 6033 50  0000 R CNN
 F 1 "WDError" V 5347 6033 50  0000 R CNN
-F 2 "" H 5400 6150 50  0001 C CNN
+F 2 "LED_SMD:LED_0805_2012Metric" H 5400 6150 50  0001 C CNN
 F 3 "~" H 5400 6150 50  0001 C CNN
 F 4 "Red" V 5400 6150 50  0001 C CNN "Color"
@@
 F 0 "R52" H 5470 5846 50  0000 L CNN
 F 1 "750" H 5470 5755 50  0000 L CNN
-F 2 "" V 5330 5800 50  0001 C CNN
+F 2 "Resistor_SMD:R_0805_2012Metric" V 5330 5800 50  0001 C CNN
 F 3 "~" H 5400 5800 50  0001 C CNN
 	1    5400 5800
@@
 F 0 "D12" V 5938 6033 50  0000 R CNN
 F 1 "CANError" V 5847 6033 50  0000 R CNN
-F 2 "" H 5900 6150 50  0001 C CNN
+F 2 "LED_SMD:LED_0805_2012Metric" H 5900 6150 50  0001 C CNN
 F 3 "~" H 5900 6150 50  0001 C CNN
 F 4 "Red" V 5900 6150 50  0001 C CNN "Color"
@@
 F 0 "R53" H 5970 5846 50  0000 L CNN
 F 1 "750" H 5970 5755 50  0000 L CNN
-F 2 "" V 5830 5800 50  0001 C CNN
+F 2 "Resistor_SMD:R_0805_2012Metric" V 5830 5800 50  0001 C CNN
 F 3 "~" H 5900 5800 50  0001 C CNN
 	1    5900 5800
@@
 F 0 "J16" H 8430 3642 50  0000 L CNN
 F 1 "Fan5" H 8430 3551 50  0000 L CNN
-F 2 "" H 8350 3650 50  0001 C CNN
+F 2 "UTSVT_Connectors:Molex_MicroFit3.0_1x2xP3.00mm_PolarizingPeg_Vertical" H 8350 3650 50  0001 C CNN
 F 3 "~" H 8350 3650 50  0001 C CNN
 	1    8350 3650
@@
 F 0 "J17" H 8430 3942 50  0000 L CNN
 F 1 "Fan6" H 8430 3851 50  0000 L CNN
-F 2 "" H 8350 3950 50  0001 C CNN
+F 2 "UTSVT_Connectors:Molex_MicroFit3.0_1x2xP3.00mm_PolarizingPeg_Vertical" H 8350 3950 50  0001 C CNN
 F 3 "~" H 8350 3950 50  0001 C CNN
 	1    8350 3950
@@
 F 0 "J18" H 8430 4242 50  0000 L CNN
 F 1 "Fan7" H 8430 4151 50  0000 L CNN
-F 2 "" H 8350 4250 50  0001 C CNN
+F 2 "UTSVT_Connectors:Molex_MicroFit3.0_1x2xP3.00mm_PolarizingPeg_Vertical" H 8350 4250 50  0001 C CNN
 F 3 "~" H 8350 4250 50  0001 C CNN
 	1    8350 4250
@@
 F 0 "J19" H 8430 4542 50  0000 L CNN
 F 1 "Fan8" H 8430 4451 50  0000 L CNN
-F 2 "" H 8350 4550 50  0001 C CNN
+F 2 "UTSVT_Connectors:Molex_MicroFit3.0_1x2xP3.00mm_PolarizingPeg_Vertical" H 8350 4550 50  0001 C CNN
 F 3 "~" H 8350 4550 50  0001 C CNN
 	1    8350 4550
@@
 F 0 "R45" V 1250 3850 50  0000 C CNN
 F 1 "0" V 1350 3850 50  0000 C CNN
-F 2 "" V 1280 3850 50  0001 C CNN
+F 2 "Resistor_SMD:R_0805_2012Metric" V 1280 3850 50  0001 C CNN
 F 3 "~" H 1350 3850 50  0001 C CNN
 	1    1350 3850
@@
 F 0 "R46" H 1700 4050 50  0000 L CNN
 F 1 "100k" V 1650 3950 50  0000 L CNN
-F 2 "" V 1580 4050 50  0001 C CNN
+F 2 "Resistor_SMD:R_0805_2012Metric" V 1580 4050 50  0001 C CNN
 F 3 "~" H 1650 4050 50  0001 C CNN
 	1    1650 4050
