File: Electronics/BPS/Master/PowerDist.sch (KiCad schematic (older format))
At the start: 18 parts

Commit message: Finalized schematics for BPS master.
Parts:
- removed C?: 100uF, symbol Device:CP
- removed C?: 47uF, symbol Device:CP
- removed C?: 10uF, symbol Device:CP
- removed C?: CP, symbol Device:CP
- removed L?: 4.7uH, symbol Device:L
- removed U?: PQMC3-D12-S3-S, symbol utsvt-power-regulators:PQMC3-Dx-Sx-S
- added C19: 0.1uF, symbol Device:C
- added C20: 10uF, symbol Device:C
- added TP4: +3.3V_TP, symbol Connector:TestPoint
- added U3: NCP1117-3.3_SOT223, Package_TO_SOT_SMD:SOT-223-3_TabPin2, symbol Regulator_Linear:LD1117S33TR_SOT223
- gave numbers to parts that had none: 12
Connections:
- wire segments 70 -> 58
- no-connect marks 2 -> 1

Commit message: Added SoC skeleton code.
Parts:
- C15, C17, C18, C19, C20: footprint (none) -> Capacitor_SMD:C_0805_2012Metric
- C16: value CP -> 100uF; footprint (none) -> Capacitor_SMD:C_0805_2012Metric
- TP1, TP2, TP3, TP4: footprint (none) -> TestPoint:TestPoint_Keystone_5005-5009_Compact
- U2: footprint (none) -> UTSVT_ICs:CUI_PQMC3-S
Changed lines of the file:
@@
 F 0 "U2" H 4800 3850 60  0000 C CNN
 F 1 "PQMC3-D12-S5-S" H 4800 3750 60  0000 C CNN
-F 2 "" H 4800 3450 60  0001 C CNN
+F 2 "UTSVT_ICs:CUI_PQMC3-S" H 4800 3450 60  0001 C CNN
 F 3 "" H 4800 3450 60  0001 C CNN
 	1    4800 3400
@@
 F 0 "C17" H 3618 3446 50  0000 L CNN
 F 1 "100uF" H 3618 3355 50  0000 L CNN
-F 2 "" H 3538 3250 50  0001 C CNN
+F 2 "Capacitor_SMD:C_0805_2012Metric" H 3538 3250 50  0001 C CNN
 F 3 "~" H 3500 3400 50  0001 C CNN
 	1    3500 3400
@@
 F 0 "C18" H 4218 3446 50  0000 L CNN
 F 1 "47uF" H 4218 3355 50  0000 L CNN
-F 2 "" H 4138 3250 50  0001 C CNN
+F 2 "Capacitor_SMD:C_0805_2012Metric" H 4138 3250 50  0001 C CNN
 F 3 "~" H 4100 3400 50  0001 C CNN
 	1    4100 3400
@@
 F 0 "C15" V 5200 3450 50  0000 C CNN
 F 1 "10uF" V 5200 3250 50  0000 C CNN
-F 2 "" H 5388 3200 50  0001 C CNN
+F 2 "Capacitor_SMD:C_0805_2012Metric" H 5388 3200 50  0001 C CNN
 F 3 "~" H 5350 3350 50  0001 C CNN
 	1    5350 3350
@@
 P 5900 3350
 F 0 "C16" H 6018 3396 50  0000 L CNN
-F 1 "CP" H 6018 3305 50  0000 L CNN
-F 2 "" H 5938 3200 50  0001 C CNN
+F 1 "100uF" H 6018 3305 50  0000 L CNN
+F 2 "Capacitor_SMD:C_0805_2012Metric" H 5938 3200 50  0001 C CNN
 F 3 "~" H 5900 3350 50  0001 C CNN
 	1    5900 3350
@@
 F 0 "TP2" H 3500 3500 50  0000 L CNN
 F 1 "+12V_TP" H 3500 3400 50  0000 L CNN
-F 2 "" H 3700 3150 50  0001 C CNN
+F 2 "TestPoint:TestPoint_Keystone_5005-5009_Compact" H 3700 3150 50  0001 C CNN
 F 3 "~" H 3700 3150 50  0001 C CNN
 	1    3500 3150
@@
 F 0 "TP1" H 5458 3220 50  0000 L CNN
 F 1 "+5V_TP" H 5458 3129 50  0000 L CNN
-F 2 "" H 5600 3100 50  0001 C CNN
+F 2 "TestPoint:TestPoint_Keystone_5005-5009_Compact" H 5600 3100 50  0001 C CNN
 F 3 "~" H 5600 3100 50  0001 C CNN
 	1    5400 3100
@@
 F 0 "TP3" H 5842 3677 50  0000 R CNN
 F 1 "GND_TP" H 5842 3768 50  0000 R CNN
-F 2 "" H 6100 3650 50  0001 C CNN
+F 2 "TestPoint:TestPoint_Keystone_5005-5009_Compact" H 6100 3650 50  0001 C CNN
 F 3 "~" H 6100 3650 50  0001 C CNN
 	1    5900 3650
@@
 F 0 "C19" H 4415 4746 50  0000 L CNN
 F 1 "0.1uF" H 4415 4655 50  0000 L CNN
-F 2 "" H 4338 4550 50  0001 C CNN
+F 2 "Capacitor_SMD:C_0805_2012Metric" H 4338 4550 50  0001 C CNN
 F 3 "~" H 4300 4700 50  0001 C CNN
 	1    4300 4700
@@
 F 0 "C20" H 5415 4746 50  0000 L CNN
 F 1 "10uF" H 5415 4655 50  0000 L CNN
-F 2 "" H 5338 4550 50  0001 C CNN
+F 2 "Capacitor_SMD:C_0805_2012Metric" H 5338 4550 50  0001 C CNN
 F 3 "~" H 5300 4700 50  0001 C CNN
 	1    5300 4700
@@
 F 0 "TP4" H 5558 4570 50  0000 L CNN
 F 1 "+3.3V_TP" H 5550 4650 50  0000 L CNN
-F 2 "" H 5700 4450 50  0001 C CNN
+F 2 "TestPoint:TestPoint_Keystone_5005-5009_Compact" H 5700 4450 50  0001 C CNN
 F 3 "~" H 5700 4450 50  0001 C CNN
 	1    5500 4450
@@
 	5500 4500 5300 4500
 $Comp
-L power:PWR_FLAG #FLG0101
+L power:PWR_FLAG #FLG02
 U 1 1 5CC7C643
 P 4100 3100
-F 0 "#FLG0101" H 4100 3175 50  0001 C CNN
+F 0 "#FLG02" H 4100 3175 50  0001 C CNN
 F 1 "PWR_FLAG" H 4100 3274 50  0000 C CNN
 F 2 "" H 4100 3100 50  0001 C CNN

Commit message: Assigned footprints to each symbol in BPS schematics.
Parts:
- removed C15: 10uF, Capacitor_SMD:C_0805_2012Metric, symbol Device:C
- removed C18: 47uF, Capacitor_SMD:C_0805_2012Metric, symbol Device:C
- removed U2: PQMC3-D12-S5-S, UTSVT_ICs:CUI_PQMC3-S, symbol utsvt-power-regulators:PQMC3-Dx-Sx-S
- added U2: RI3-1205S, UTSVT_ICs:RI3_DC_Converter, symbol utsvt-power-regulators:RI3-1205S
- C15: renamed from C16; value 100uF -> 470pF; footprint Capacitor_SMD:C_0805_2012Metric -> Capacitor_SMD:C_2220_5650Metric; Rating (none) -> 4kV
- C16: renamed from C17; value 100uF -> 4.7uF
- D1: footprint (none) -> LED_SMD:LED_0805_2012Metric
- J4: footprint (none) -> UTSVT_Connectors:Molex_MicroFit3.0_1x2xP3.00mm_PolarizingPeg_Vertical
- L1: value 4.7uH -> 10uH; footprint (none) -> Inductor_SMD:L_0805_2012Metric
- R1: value R -> 1.5k; footprint (none) -> Resistor_SMD:R_0805_2012Metric
- renumbered C19 to C17, C20 to C18, TP2 to TP1, TP1 to TP2
Connections:
- wire segments 58 -> 55
- no-connect marks 1 -> 0

Commit message: Master board PCB layout organized.
Parts:
- added TP15: GNDPWR_TP, TestPoint:TestPoint_Keystone_5005-5009_Compact, symbol Connector:TestPoint
Connections:
- wire segments 55 -> 56
Changed lines of the file:
@@
 	5100 2850 5100 3200
 Connection ~ 5100 3200
+$Comp
+L Connector:TestPoint TP15
+U 1 1 5C82CEA3
+P 3400 3650
+F 0 "TP15" H 3342 3677 50  0000 R CNN
+F 1 "GNDPWR_TP" H 3342 3768 50  0000 R CNN
+F 2 "TestPoint:TestPoint_Keystone_5005-5009_Compact" H 3600 3650 50  0001 C CNN
+F 3 "~" H 3600 3650 50  0001 C CNN
+	1    3400 3650
+	-1   0    0    1
+$EndComp
+Wire Wire Line
+	3400 3650 3400 3600
 $EndSCHEMATC
