File: Electronics/BPS/Master/BPSMaster.kicad_pcb (KiCad board)
At the start: 2 copper layers, 100 x 75 mm, 178 parts, among them J1 SWD, J10 DisplayJumper, J11 FrontFans, J12 BackFans, J13 ErrorLightConnector, J14 Conn_01x03, J2 Logic Analyzer, J3 CurrentSlaveConnector, J4 CarPowerConnector, J5 CAN_Out, J6 ContactorConnector, J7 VoltageSlaveConnector, J8 DisplayConnector, J9 TempSlaveConnector, Q1 VND5N07-E, Q2 NVR4003NT3G, Q3 NVR4003NT3G, Q4 NVR4003NT3G, SW1 B3SL-1002P, U1 STM32F413RHTx, U10 LTC6820, U11 HX1188FNL, U12 LTC6820, U13 Si8641EC-B-IS1, U14 SI8660EC-B-IS1, U15 RI3-1205S, U16 SI8261ABC-IS, U2 RI3-1205S, U3 NCP1117-3.3_SOT223, U4 CDSOT23-T24CAN, U5 ADM3055E, U6 BAS70-04, U7 SI8261ABC-IS, U8 M24128, Y1 NX8045GB-8.000M-STD-CSJ-1

Commit message: Finalized all boards. Created gerber files.
Parts:
- added G***: LOGO, UTSVT_Special:UTSVT_Logo_Symbol, F.Cu at (195.2, 90.8)
- added G***: LOGO, UTSVT_Special:Hallock_Image_Small, B.Cu at (165.6, 94.6)
Other:
- outline, holes or cut-outs redrawn
- board text added: "Dr. Gary Hallock"
- board text added: "Gate"
- board text added: "RESET"
- board text added: "Spring 2019: Monolo Alvarez Chase Block Corbin Capo Richard Li Austin Tsao Garrett Wong Sihyung Woo Sijin Woo"
- board text removed: "Spring 2019: Monolo Alvarez Chase Block Corbin Capo Richard Li Garrett Wong Sijin Woo"
