File: Electronics/BPS/Tester/BPSTester.sch (KiCad schematic (older format))
At the start: 13 parts

Commit message: changed power from potentiometers, upgraded to KiCad 5.0
Parts:
- J?: symbol Conn_01x13_Male -> conn:Conn_01x13_Male
- RV? (x12): symbol POT -> BPSTester-rescue:POT
Connections:
- net +BATT: now also J?.12 (Pin_12), RV?.2; no longer RV?.1
- net at RV?.3: now also J?.11 (Pin_11), RV?.2; no longer RV?.1
- net at RV?.3: now also J?.10 (Pin_10), RV?.2; no longer RV?.1
- net at RV?.3: now also J?.9 (Pin_9), RV?.2; no longer RV?.1
- net at RV?.3: now also J?.8 (Pin_8), RV?.2; no longer RV?.1
- net at RV?.3: now also J?.7 (Pin_7), RV?.2; no longer RV?.1
- net at RV?.3: now also J?.6 (Pin_6), RV?.2; no longer RV?.1
- net at RV?.3: now also J?.5 (Pin_5), RV?.2; no longer RV?.1
- net at RV?.3: now also J?.4 (Pin_4), RV?.2; no longer RV?.1
- net at RV?.3: now also J?.3 (Pin_3), RV?.2; no longer RV?.1
- net at RV?.3: now also J?.2 (Pin_2), RV?.2; no longer RV?.1
- net at RV?.3: now also J?.1 (Pin_1), RV?.2; no longer RV?.1
Other:
- moved on the sheet: RV?

Commit message: updated footprints, net, and organized footprints on pcb. Have not routed
Parts:
- added TP1, TP10, TP11, TP12, TP13, TP2, TP3, TP4, TP5, TP6, TP7, TP8, TP9: TestPoint, Measurement_Points:Test_Point_Keystone_5005-5009_Compact, symbol Connector:TestPoint
- 1K1, 1K10, 1K11, 1K12, 1K2, 1K3, 1K4, 1K5, 1K6, 1K7, 1K8, 1K9: renamed from RV?; footprint (none) -> Potentiometers:Potentiometer_Trimmer_Bourns_3296W
- J1: renamed from J?; footprint (none) -> Connectors_Molex:Molex_KK-6410-13_13x2.54mm_Straight
Connections:
- wire segments 75 -> 101
- no-connect marks 0 -> 12

Commit message: Placed a ground plane and labeled Testing board
Parts:
- added J2: Conn_01x02_Male, Connectors_Molex:Molex_KK-6410-02_02x2.54mm_Straight, symbol Connector:Conn_01x02_Male
Connections:
- wire segments 101 -> 103
Changed lines of the file:
@@
 Wire Wire Line
 	2250 6300 2250 6350
+$Comp
+L Connector:Conn_01x02_Male J2
+U 1 1 5C561D48
+P 4950 1900
+F 0 "J2" V 5103 1713 50  0000 R CNN
+F 1 "Conn_01x02_Male" V 5012 1713 50  0000 R CNN
+F 2 "Connectors_Molex:Molex_KK-6410-02_02x2.54mm_Straight" H 4950 1900 50  0001 C CNN
+F 3 "~" H 4950 1900 50  0001 C CNN
+	1    4950 1900
+	0    1    1    0
+$EndComp
+Wire Wire Line
+	4850 2100 4850 2300
+$Comp
+L power:+BATT #PWR0104
+U 1 1 5C577058
+P 4850 2300
+F 0 "#PWR0104" H 4850 2150 50  0001 C CNN
+F 1 "+BATT" H 4850 2440 50  0000 C CNN
+F 2 "" H 4850 2300 50  0001 C CNN
+F 3 "" H 4850 2300 50  0001 C CNN
+	1    4850 2300
+	-1   0    0    1
+$EndComp
+$Comp
+L power:GND #PWR0105
+U 1 1 5C58426B
+P 4950 2350
+F 0 "#PWR0105" H 4950 2100 50  0001 C CNN
+F 1 "GND" H 4950 2200 50  0000 C CNN
+F 2 "" H 4950 2350 50  0001 C CNN
+F 3 "" H 4950 2350 50  0001 C CNN
+	1    4950 2350
+	1    0    0    -1
+$EndComp
+Wire Wire Line
+	4950 2100 4950 2350
 $EndSCHEMATC
