File: Electronics/BPS/Voltage/BPSVoltage.sch (KiCad schematic (older format))
At the start: 1 part

Commit message: Finished up the voltage board. Revise later.
Parts:
- added C1, C3: 100nF, Capacitor_SMD:C_0805_2012Metric, symbol Device:C
- added C10, C8, C9: 10u, Capacitor_SMD:C_0805_2012Metric, symbol Device:C
- added C11, C12, C13, C14, C15, C16, C17, C18, C19, C2, C20, C21, C4, C5, C6, C7: 10nF, Capacitor_SMD:C_0805_2012Metric, symbol Device:C
- added J1: Conn1, UTSVT_Connectors:Molex_MicroFit3.0_1x2xP3.00mm_PolarizingPeg_Vertical, symbol utsvt-connectors:CarPowerConnector
- added J2: Conn2, UTSVT_Connectors:Molex_MicroFit3.0_1x2xP3.00mm_PolarizingPeg_Vertical, symbol utsvt-connectors:CarPowerConnector
- added J3: Conn_01x06, Connector_Molex:Molex_Micro-Fit_3.0_43650-0615_1x06_P3.00mm_Vertical, symbol Connector_Generic:Conn_01x06
- added J4: Conn_01x07, Connector_Molex:Molex_Micro-Fit_3.0_43650-0715_1x07_P3.00mm_Vertical, symbol Connector_Generic:Conn_01x07
- added Q1, Q10, Q11, Q12, Q13, Q2, Q3, Q4, Q6, Q7, Q8, Q9: BSS308PE, Package_TO_SOT_SMD:SOT-23, symbol Device:Q_PMOS_GSD
- added Q5: NSV1C201MZ4, Package_TO_SOT_SMD:SOT-223, symbol Device:Q_NPN_BCEC
- added R1, R11, R13, R15, R19, R2, R22, R26, R29, R3, R31, R5, R7, R9: 100R, Resistor_SMD:R_0805_2012Metric, symbol Device:R
- added R10, R12, R14, R18, R21, R25, R28, R30, R32, R4, R6, R8: 33R, Resistor_SMD:R_2512_6332Metric, symbol Device:R
- added R16, R17: 1k, Resistor_SMD:R_0805_2012Metric, symbol Device:R
- added R20, R23, R24, R27: 49R9, Resistor_SMD:R_0805_2012Metric, symbol Device:R
- added U2: HX1188FNL, UTSVT_BPS:HXXXX, symbol utsvt-bps:HX1188FNL
- U1: renamed from U?; footprint (none) -> Package_SO:SSOP-48_7.5x15.9mm_P0.635mm
Connections:
- net labels added: Batt1, Batt10, Batt11, Batt12, Batt2, Batt3, Batt4, Batt5, Batt6, Batt7, Batt8, Batt9, GND, IMA, IMB, IPA, IPB, V12, VREG
- wire segments 0 -> 279
- no-connect marks 0 -> 10

Commit message: Finished up revision 2 of the board.
Parts:
- added D1, D10, D11, D12, D13, D2, D3, D4, D5, D6, D7, D8, D9: LED, LED_SMD:LED_0805_2012Metric, symbol Device:LED
- added J5: Conn_01x03, Connector_PinHeader_2.54mm:PinHeader_1x03_P2.54mm_Vertical, symbol Connector_Generic:Conn_01x03
- added J6: Conn_01x05, Connector_PinHeader_2.54mm:PinHeader_1x05_P2.54mm_Vertical, symbol Connector_Generic:Conn_01x05
- added J7: Conn_02x03_Counter_Clockwise, Connector_PinHeader_2.54mm:PinHeader_2x03_P2.54mm_Vertical, symbol Connector_Generic:Conn_02x03_Odd_Even
- added L1, L10, L11, L12, L13, L14, L2, L3, L4, L5, L6, L7, L8, L9: Ferrite_Bead, Inductor_SMD:L_0805_2012Metric, symbol Device:Ferrite_Bead
- added MH1, MH2, MH3, MH4: MountingHole, MountingHole:MountingHole_3mm, symbol Mechanical:MountingHole
- added R33: 1.5k, Resistor_SMD:R_0805_2012Metric, symbol Device:R
- added R34, R35, R36, R37, R38, R39, R40, R41, R42, R43, R44, R45: 1.2k, Resistor_SMD:R_0805_2012Metric, symbol Device:R
- added TP1: V+, TestPoint:TestPoint_Keystone_5005-5009_Compact, symbol Connector:TestPoint
- added TP2: VREG, TestPoint:TestPoint_Keystone_5005-5009_Compact, symbol Connector:TestPoint
- added TP3: GND, TestPoint:TestPoint_Keystone_5005-5009_Compact, symbol Connector:TestPoint
- R16: value 1k -> 806
- R17: value 1k -> 1.21k
Connections:
- net labels added: Batt0, GPIO1, GPIO2, GPIO3, GPIO4, GPIO5, ISOMD, L0, L1, L10, L11, L2, L3, L4, L5, L6, L7, L8, L9
- wire segments 279 -> 353
- no-connect marks 10 -> 6
Other:
- moved on the sheet: C14, C15, C17, C18, R20, R23, R24, R27, R32

Commit message: Footprints, BOM, and final board edits.
Parts:
- removed J7: Conn_02x03_Counter_Clockwise, Connector_PinHeader_2.54mm:PinHeader_2x03_P2.54mm_Vertical, symbol Connector_Generic:Conn_02x03_Odd_Even
- added J7: Conn_01x05, Connector_PinHeader_2.54mm:PinHeader_1x05_P2.54mm_Vertical, symbol Connector_Generic:Conn_01x05
- J1, J2: symbol utsvt-connectors:CarPowerConnector -> BPSVoltage-rescue:CarPowerConnector-utsvt-connectors
- J3: footprint Connector_Molex:Molex_Micro-Fit_3.0_43650-0615_1x06_P3.00mm_Vertical -> UTSVT_Connectors:Molex_MicroFit_01x06_Horizontal
- J4: footprint Connector_Molex:Molex_Micro-Fit_3.0_43650-0715_1x07_P3.00mm_Vertical -> UTSVT_Connectors:Molex_MicroFit_01x07_Horizontal
- U1: symbol utsvt-bps:LTC6811-1 -> BPSVoltage-rescue:LTC6811-1-utsvt-bps
- U2: symbol utsvt-bps:HX1188FNL -> BPSVoltage-rescue:HX1188FNL-utsvt-bps
Connections:
- net labels added: SDI, SDO
- no-connect marks 6 -> 3
Changed lines of the file:
@@
 $EndDescr
 $Comp
-L utsvt-bps:LTC6811-1 U1
+L BPSVoltage-rescue:LTC6811-1-utsvt-bps U1
 U 1 1 5C356477
 P 6400 2650
@@
 Wire Wire Line
 	7950 4050 8050 4050
-NoConn ~ 7200 4150
-NoConn ~ 7200 4250
 NoConn ~ 7200 4750
 $Comp
@@
 IMA
 $Comp
-L utsvt-bps:HX1188FNL U2
+L BPSVoltage-rescue:HX1188FNL-utsvt-bps U2
 U 1 1 5CAB08B5
 P 9700 5250
@@
 $EndComp
 $Comp
-L utsvt-connectors:CarPowerConnector J1
+L BPSVoltage-rescue:CarPowerConnector-utsvt-connectors J1
 U 1 1 5CAB16B3
 P 10750 5450
@@
 $EndComp
 $Comp
-L utsvt-connectors:CarPowerConnector J2
+L BPSVoltage-rescue:CarPowerConnector-utsvt-connectors J2
 U 1 1 5CADF981
 P 10750 5850
@@
 F 0 "J4" H 750 4850 50  0000 C CNN
 F 1 "Conn_01x07" H 750 4750 50  0000 C CNN
-F 2 "Connector_Molex:Molex_Micro-Fit_3.0_43650-0715_1x07_P3.00mm_Vertical" H 700 4300 50  0001 C CNN
+F 2 "UTSVT_Connectors:Molex_MicroFit_01x07_Horizontal" H 700 4300 50  0001 C CNN
 F 3 "~" H 700 4300 50  0001 C CNN
 	1    700  4300
@@
 F 0 "J3" H 620 3175 50  0000 C CNN
 F 1 "Conn_01x06" H 620 3266 50  0000 C CNN
-F 2 "Connector_Molex:Molex_Micro-Fit_3.0_43650-0615_1x06_P3.00mm_Vertical" H 700 3700 50  0001 C CNN
+F 2 "UTSVT_Connectors:Molex_MicroFit_01x06_Horizontal" H 700 3700 50  0001 C CNN
 F 3 "~" H 700 3700 50  0001 C CNN
 	1    700  3700
@@
 F 3 "~" H 9100 1900 50  0001 C CNN
 	1    9100 1900
-	1    0    0    -1
+	1    0    0    1
 $EndComp
 Text Label 8650 2100 0    50   ~ 0
@@
 Wire Wire Line
 	8650 2100 8900 2100
-$Comp
-L Connector_Generic:Conn_02x03_Odd_Even J7
-U 1 1 5C69EFB9
-P 10250 4550
-F 0 "J7" H 10300 4867 50  0000 C CNN
-F 1 "Conn_02x03_Counter_Clockwise" H 10300 4776 50  0000 C CNN
-F 2 "Connector_PinHeader_2.54mm:PinHeader_2x03_P2.54mm_Vertical" H 10250 4550 50  0001 C CNN
-F 3 "~" H 10250 4550 50  0001 C CNN
-	1    10250 4550
-	1    0    0    -1
-$EndComp
-Text Label 9850 4450 0    50   ~ 0
+Text Label 10000 3550 0    50   ~ 0
 IPA
-Text Label 9850 4550 0    50   ~ 0
+Text Label 10000 3650 0    50   ~ 0
 IMA
 Wire Wire Line
-	9850 4450 10050 4450
-Wire Wire Line
-	9850 4550 10050 4550
+	10000 3550 10200 3550
+Wire Wire Line
+	10000 3650 10200 3650
 $Comp
 L power:GND #PWR0114
 U 1 1 5C6CFA3C
-P 9850 4750
-F 0 "#PWR0114" H 9850 4500 50  0001 C CNN
-F 1 "GND" H 10000 4700 50  0000 C CNN
-F 2 "" H 9850 4750 50  0001 C CNN
-F 3 "" H 9850 4750 50  0001 C CNN
-	1    9850 4750
-	1    0    0    -1
-$EndComp
-Wire Wire Line
-	9850 4750 9850 4650
-Wire Wire Line
-	9850 4650 10050 4650
-Text Label 10700 4450 0    50   ~ 0
-IPB
-Wire Wire Line
-	10550 4450 10700 4450
-Text Label 10700 4550 0    50   ~ 0
-IMB
-Wire Wire Line
-	10550 4550 10700 4550
-NoConn ~ 10550 4650
+P 10000 4050
+F 0 "#PWR0114" H 10000 3800 50  0001 C CNN
+F 1 "GND" H 10150 4000 50  0000 C CNN
+F 2 "" H 10000 4050 50  0001 C CNN
+F 3 "" H 10000 4050 50  0001 C CNN
+	1    10000 4050
+	1    0    0    -1
+$EndComp
+Wire Wire Line
+	10000 4050 10000 3950
+Wire Wire Line
+	10000 3950 10200 3950
 Text Label 2500 1400 0    50   ~ 0
 L11
@@
 	5500 5250 5500 7150
 Connection ~ 3300 7150
+$Comp
+L Connector_Generic:Conn_01x05 J7
+U 1 1 5C56A49F
+P 10400 3750
+F 0 "J7" H 10480 3792 50  0000 L CNN
+F 1 "Conn_01x05" H 10480 3701 50  0000 L CNN
+F 2 "Connector_PinHeader_2.54mm:PinHeader_1x05_P2.54mm_Vertical" H 10400 3750 50  0001 C CNN
+F 3 "~" H 10400 3750 50  0001 C CNN
+	1    10400 3750
+	1    0    0    -1
+$EndComp
+Text Label 7200 4150 0    50   ~ 0
+SDO
+Text Label 7200 4250 0    50   ~ 0
+SDI
+Text Label 10000 3850 0    50   ~ 0
+SDO
+Text Label 10000 3750 0    50   ~ 0
+SDI
+Wire Wire Line
+	10000 3750 10200 3750
+Wire Wire Line
+	10000 3850 10200 3850
+Wire Notes Line
+	5850 6600 6800 6600
+Wire Notes Line
+	6800 6600 6800 7550
+Wire Notes Line
+	7600 5000 7600 6550
+Wire Notes Line
+	7600 6550 11250 6550
+Wire Notes Line
+	11250 6550 11250 5000
+Wire Notes Line
+	11250 5000 7600 5000
+Wire Notes Line
+	9850 3350 9850 4250
+Wire Notes Line
+	9850 4250 11050 4250
+Wire Notes Line
+	11050 4250 11050 3350
+Wire Notes Line
+	11050 3350 9850 3350
+Wire Notes Line
+	9750 550  9750 3050
+Wire Notes Line
+	9750 3050 11150 3050
+Wire Notes Line
+	11150 3050 11150 550
+Wire Notes Line
+	11150 550  9750 550
+Wire Notes Line
+	8550 1550 9750 1550
+Wire Notes Line
+	8550 750  8550 2250
+Wire Notes Line
+	8000 750  8000 2250
+Wire Notes Line
+	8000 750  9750 750
+Wire Notes Line
+	8000 2250 9750 2250
+Wire Notes Line
+	6800 7550 5850 7550
+Wire Notes Line
+	5850 7550 5850 6600
 $EndSCHEMATC
