File: Electronics/BPS/Voltage/BPSVoltage.kicad_pcb (KiCad board)
At the start: 2 copper layers, 75 x 65 mm, 124 parts, among them J1 Conn1, J2 Conn2, J3 Conn_01x06, J4 Conn_01x07, J5 Conn_01x03, J6 Conn_01x05, J7 Conn_01x05, Q1 BSS308PE, Q10 BSS308PE, Q11 BSS308PE, Q12 BSS308PE, Q13 BSS308PE, Q2 BSS308PE, Q3 BSS308PE, Q4 BSS308PE, Q5 NSV1C201MZ4, Q6 BSS308PE, Q7 BSS308PE, Q8 BSS308PE, Q9 BSS308PE, U1 LTC6811-1, U2 HX1188FNL

Commit message: Finalized all boards. Created gerber files.
Other:
- board text added: "Dr. Gary Hallock"
