File: Electronics/BPS/Temperature/BPSTemperature.kicad_pcb (KiCad board)
At the start: 2 copper layers, 82 x 65 mm, 83 parts, among them J1 Conn_02x10_Counter_Clockwise, J2 Logic Analyzer, J3 Conn_02x06_Counter_Clockwise, J4 Conn_02x06_Counter_Clockwise, J5 Conn_01x02, SW1 SW_DIP_x06, U1 LTC2983

Commit message: Finalized all boards. Created gerber files.
Routing:
- net GND: vias 26 -> 29
Other:
- board text added: "Dr. Gary Hallock"
Changed lines of the file:
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@@
   (general
     (thickness 1.6)
-    (drawings 54)
-    (tracks 692)
+    (drawings 55)
+    (tracks 696)
     (zones 0)
     (modules 83)
@@
       (layerselection 0x010fc_ffffffff)
       (usegerberextensions false)
-      (usegerberattributes false)
+      (usegerberattributes true)
       (usegerberadvancedattributes false)
       (creategerberjobfile false)
@@
       (outputformat 1)
       (mirror false)
-      (drillshape 1)
+      (drillshape 0)
       (scaleselection 1)
-      (outputdirectory ""))
+      (outputdirectory "../GerberFiles/Temperature/"))
   )
   (net 0 "")
@@
       (xy -3.770496 -5.687082) (xy -3.551303 -5.609675) (xy -3.473034 -5.588) (xy -3.408236 -5.646283)) (layer B.SilkS) (width 0.01))
   )
+  (gr_text "Dr. Gary Hallock" (at 82.425 118.8) (layer B.SilkS)
+    (effects (font (size 1.5 1.5) (thickness 0.3)) (justify mirror))
+  )
   (gr_text GND (at 115.4 81.775 90) (layer F.SilkS)
     (effects (font (size 1 1) (thickness 0.15)))
@@
     (effects (font (size 1.5 1.5) (thickness 0.3)))
   )
-  (gr_text "Spring 2019:\nMonolo Alvarez\nChase Block\nCorbin Capo\nRichard Li\nAustin Tsao\nGarrett Wong\nSihyung Woo\nSijin Woo" (at 109.38 87.21) (layer B.SilkS)
-    (effects (font (size 0.738 0.738) (thickness 0.1845)) (justify mirror))
+  (gr_text "Spring 2019:\nMonolo Alvarez\nChase Block\nCorbin Capo\nRichard Li\nAustin Tsao\nGarrett Wong\nSihyung Woo\nSijin Woo" (at 121.3 101.175) (layer B.SilkS)
+    (effects (font (size 1.5 1.5) (thickness 0.3)) (justify left mirror))
   )
   (segment (start 95.5675 86.8045) (end 95.5675 95.0595) (width 0.2032) (layer F.Cu) (net 1))
@@
   (segment (start 132.842 86.0425) (end 132.842 78.867) (width 0.3048) (layer B.Cu) (net 2))
   (segment (start 97.819542 98.760871) (end 98.349871 98.230542) (width 0.2032) (layer F.Cu) (net 2))
-  (segment (start 97.112435 99.467978) (end 97.819542 98.760871) (width 0.2032) (layer F.Cu) (net 2))
+  (segment (start 97.112435 99.467978) (end 97.112435 99.467978) (width 0.2032) (layer F.Cu) (net 2))
   (segment (start 95.910351 99.467978) (end 97.112435 99.467978) (width 0.2032) (layer F.Cu) (net 2))
   (segment (start 95.380022 98.937649) (end 95.910351 99.467978) (width 0.2032) (layer F.Cu) (net 2))
@@
   (segment (start 103.7 100.65) (end 103.55 100.5) (width 0.2032) (layer F.Cu) (net 2))
   (via (at 103.7 100.65) (size 0.762) (drill 0.381) (layers F.Cu B.Cu) (net 2))
+  (segment (start 97.112435 99.467978) (end 97.819542 98.760871) (width 0.2032) (layer F.Cu) (net 2))
+  (via (at 97.112435 99.467978) (size 0.762) (drill 0.381) (layers F.Cu B.Cu) (net 2))
+  (via (at 95 103.125) (size 0.762) (drill 0.381) (layers F.Cu B.Cu) (net 2))
+  (via (at 96.9 105.15) (size 0.762) (drill 0.381) (layers F.Cu B.Cu) (net 2))
   (segment (start 94.9325 86.5505) (end 94.9325 94.996) (width 0.2032) (layer F.Cu) (net 3))
   (segment (start 94.9325 94.996) (end 93.6625 96.266) (width 0.2032) (layer F.Cu) (net 3))
