File: Electronics/BPS/Temperature/BPSTemperature.sch (KiCad schematic (older format))
At the start: 53 parts

Commit message: Added labels to temperature board for BPS
Connections:
- wire segments 185 -> 208
Changed lines of the file:
@@
 EESchema Schematic File Version 4
-LIBS:Temper Board-cache
 EELAYER 26 0
 EELAYER END
@@
 Text Notes 9650 650  0    50   ~ 0
 CT2196MST-ND  : 6 position dip switch
+Text Label 1300 700  2    50   ~ 0
+CH1_LPF
+Text Label 1300 1800 2    50   ~ 0
+CH2_LPF
+Text Label 1300 2900 2    50   ~ 0
+CH3_LPF
+Text Label 1300 4000 2    50   ~ 0
+CH4_LPF
+Text Label 1300 5100 2    50   ~ 0
+CH5_LPF
+Text Label 1300 6200 2    50   ~ 0
+CH6_LPF
+Text Label 1900 700  2    50   ~ 0
+CH7_LPF
+Text Label 1900 1800 2    50   ~ 0
+CH8_LPF
+Text Label 1900 2900 2    50   ~ 0
+CH9_LPF
+Text Label 1900 4000 2    50   ~ 0
+CH10_LPF
+Text Label 1900 5100 2    50   ~ 0
+CH11_LPF
+Text Label 1900 6200 2    50   ~ 0
+CH12_LPF
+Text Label 2450 700  2    50   ~ 0
+CH13_LPF
+Text Label 2450 1800 2    50   ~ 0
+CH14_LPF
+Text Label 2450 2900 2    50   ~ 0
+CH15_LPF
+Text Label 2450 4000 2    50   ~ 0
+CH16_LPF
+Text Label 2450 5100 2    50   ~ 0
+CH17_LPF
+Text Label 2450 6200 2    50   ~ 0
+CH18_LPF
+Text Label 3000 700  2    50   ~ 0
+CH19_LPF
+Text Label 3000 1800 2    50   ~ 0
+CH20_LPF
+Text Label 5650 2400 2    50   ~ 0
+CH1
+Text Label 5650 2500 2    50   ~ 0
+CH2
+Text Label 5650 2600 2    50   ~ 0
+CH3
+Text Label 5650 2700 2    50   ~ 0
+CH4
+Text Label 5650 2800 2    50   ~ 0
+CH5
+Text Label 5650 2900 2    50   ~ 0
+CH6
+Text Label 5650 3000 2    50   ~ 0
+CH7
+Text Label 5650 3100 2    50   ~ 0
+CH8
+Text Label 5650 3200 2    50   ~ 0
+CH9
+Text Label 5650 3300 2    50   ~ 0
+CH10
+Text Label 5650 3400 2    50   ~ 0
+CH11
+Text Label 5650 3500 2    50   ~ 0
+CH12
+Text Label 5650 3600 2    50   ~ 0
+CH13
+Text Label 5650 3700 2    50   ~ 0
+CH14
+Text Label 5650 3800 2    50   ~ 0
+CH15
+Text Label 5650 3900 2    50   ~ 0
+CH16
+Text Label 5650 4000 2    50   ~ 0
+CH17
+Text Label 5650 4100 2    50   ~ 0
+CH18
+Text Label 5650 4200 2    50   ~ 0
+CH19
+Text Label 5650 4300 2    50   ~ 0
+CH20
+Wire Wire Line
+	5650 2400 5800 2400
+Wire Wire Line
+	5650 2500 5800 2500
+Wire Wire Line
+	5800 2600 5650 2600
+Wire Wire Line
+	5650 2700 5800 2700
+Wire Wire Line
+	5800 2800 5650 2800
+Wire Wire Line
+	5650 2900 5800 2900
+Wire Wire Line
+	5800 3000 5650 3000
+Wire Wire Line
+	5650 3100 5800 3100
+Wire Wire Line
+	5800 3200 5650 3200
+Wire Wire Line
+	5650 3300 5800 3300
+Wire Wire Line
+	5800 3400 5650 3400
+Wire Wire Line
+	5650 3500 5800 3500
+Wire Wire Line
+	5650 3600 5800 3600
+Wire Wire Line
+	5650 3700 5800 3700
+Wire Wire Line
+	5650 3800 5800 3800
+Wire Wire Line
+	5800 3900 5650 3900
+Wire Wire Line
+	5650 4000 5800 4000
+Wire Wire Line
+	5800 4100 5650 4100
+Wire Wire Line
+	5650 4200 5800 4200
+Wire Wire Line
+	5800 4300 5650 4300
+Text Label 7550 4200 0    50   ~ 0
+MISO
+Text Label 7550 4300 0    50   ~ 0
+MOSI
+Text Label 7550 4400 0    50   ~ 0
+SCK
+Wire Wire Line
+	7400 4200 7550 4200
+Wire Wire Line
+	7550 4300 7400 4300
+Wire Wire Line
+	7400 4400 7550 4400
 $EndSCHEMATC

Commit message: Added DIP switch to temperature board for BPS
Parts:
- added SW?: SW_DIP_x06, symbol Switch:SW_DIP_x06
Connections:
- net labels added: CS1_OUT, CS2_OUT, CS3_OUT, CS4_OUT, CS5_OUT, CS6_OUT
- wire segments 208 -> 235
Changed lines of the file:
@@
 Wire Wire Line
 	7400 4400 7550 4400
+Wire Wire Line
+	7850 4250 8400 4250
+Wire Wire Line
+	7950 4350 8400 4350
+Wire Wire Line
+	8050 4450 8400 4450
+Wire Wire Line
+	8050 4550 8400 4550
+Wire Wire Line
+	8050 4450 8050 4500
+Wire Wire Line
+	7950 4650 8400 4650
+Wire Wire Line
+	7950 4350 7950 4500
+Wire Wire Line
+	7850 4750 8400 4750
+Wire Wire Line
+	7850 4250 7850 4500
+Wire Wire Line
+	8050 4500 7950 4500
+Connection ~ 8050 4500
+Wire Wire Line
+	8050 4500 8050 4550
+Connection ~ 7950 4500
+Wire Wire Line
+	7950 4500 7950 4650
+Wire Wire Line
+	7850 4500 7950 4500
+Connection ~ 7850 4500
+Wire Wire Line
+	7850 4500 7850 4750
+Wire Wire Line
+	7850 4500 7400 4500
+$Comp
+L Switch:SW_DIP_x06 SW?
+U 1 1 5C72A387
+P 8200 5600
+F 0 "SW?" H 8200 6167 50  0000 C CNN
+F 1 "SW_DIP_x06" H 8200 6076 50  0000 C CNN
+F 2 "" H 8200 5600 50  0001 C CNN
+F 3 "" H 8200 5600 50  0001 C CNN
+	1    8200 5600
+	1    0    0    -1
+$EndComp
+Text Label 7750 5300 2    50   ~ 0
+CS1
+Text Label 7750 5400 2    50   ~ 0
+CS2
+Text Label 7750 5500 2    50   ~ 0
+CS3
+Text Label 7750 5600 2    50   ~ 0
+CS4
+Text Label 7750 5700 2    50   ~ 0
+CS5
+Text Label 7750 5800 2    50   ~ 0
+CS6
+Text Label 8650 5300 0    50   ~ 0
+CS1_OUT
+Text Label 8650 5400 0    50   ~ 0
+CS2_OUT
+Text Label 8650 5500 0    50   ~ 0
+CS3_OUT
+Text Label 8650 5600 0    50   ~ 0
+CS4_OUT
+Text Label 8650 5700 0    50   ~ 0
+CS5_OUT
+Text Label 8650 5800 0    50   ~ 0
+CS6_OUT
+Wire Wire Line
+	8500 5300 8650 5300
+Wire Wire Line
+	8650 5400 8500 5400
+Wire Wire Line
+	8500 5500 8650 5500
+Wire Wire Line
+	8650 5600 8500 5600
+Wire Wire Line
+	8500 5700 8650 5700
+Wire Wire Line
+	8650 5800 8500 5800
+Wire Wire Line
+	7900 5800 7750 5800
+Wire Wire Line
+	7750 5700 7900 5700
+Wire Wire Line
+	7900 5600 7750 5600
+Wire Wire Line
+	7750 5500 7900 5500
+Wire Wire Line
+	7900 5400 7750 5400
+Wire Wire Line
+	7750 5300 7900 5300
+Text Label 8400 4250 0    50   ~ 0
+CS1_OUT
+Text Label 8400 4350 0    50   ~ 0
+CS2_OUT
+Text Label 8400 4450 0    50   ~ 0
+CS3_OUT
+Text Label 8400 4550 0    50   ~ 0
+CS4_OUT
+Text Label 8400 4650 0    50   ~ 0
+CS5_OUT
+Text Label 8400 4750 0    50   ~ 0
+CS6_OUT
 $EndSCHEMATC

Commit message: Cleaned up schematic of temperature board for BPS
Parts:
- removed C?: C, symbol Device:C
- removed C?: 1uF, symbol Device:C
- removed R?: 1k, symbol Device:R
Connections:
- net labels removed: +5V
- wire segments 235 -> 230
Changed lines of the file:
@@
-	1    0    0    -1
-$EndComp
-$Comp
-L power:+5V #PWR?
-U 1 1 5C4CC3F1
-P 6600 1750
-F 0 "#PWR?" H 6600 1600 50  0001 C CNN
-F 1 "+5V" H 6615 1923 50  0000 C CNN
-F 2 "" H 6600 1750 50  0001 C CNN
-F 3 "" H 6600 1750 50  0001 C CNN
-	1    6600 1750
 	1    0    0    -1
 $EndComp
@@
 $Comp
 L Device:C C?
-U 1 1 5C4CC859
-P 9550 1850
-F 0 "C?" H 9665 1896 50  0000 L CNN
-F 1 "C" H 9665 1805 50  0000 L CNN
-F 2 "" H 9588 1700 50  0001 C CNN
-F 3 "~" H 9550 1850 50  0001 C CNN
-	1    9550 1850
-	1    0    0    -1
-$EndComp
-$Comp
-L Device:C C?
 U 1 1 5C4CC88B
 P 7500 2550
@@
 $Comp
 L power:GND #PWR?
-U 1 1 5C4CCB2D
-P 9850 1750
-F 0 "#PWR?" H 9850 1500 50  0001 C CNN
-F 1 "GND" H 9855 1577 50  0000 C CNN
-F 2 "" H 9850 1750 50  0001 C CNN
-F 3 "" H 9850 1750 50  0001 C CNN
-	1    9850 1750
-	1    0    0    -1
-$EndComp
-$Comp
-L power:GND #PWR?
 U 1 1 5C4CCEAB
 P 8150 2800
@@
 Wire Wire Line
 	7750 2800 7400 2800
-$Comp
-L Device:R R?
-U 1 1 5C4D96FF
-P 9100 1000
-F 0 "R?" H 9170 1046 50  0000 L CNN
-F 1 "1k" H 9170 955 50  0000 L CNN
-F 2 "" V 9030 1000 50  0001 C CNN
-F 3 "~" H 9100 1000 50  0001 C CNN
-	1    9100 1000
-	1    0    0    -1
-$EndComp
-$Comp
-L Device:C C?
-U 1 1 5C4D97A0
-P 9100 1450
-F 0 "C?" H 9215 1496 50  0000 L CNN
-F 1 "1uF" H 9215 1405 50  0000 L CNN
-F 2 "" H 9138 1300 50  0001 C CNN
-F 3 "~" H 9100 1450 50  0001 C CNN
-	1    9100 1450
-	1    0    0    -1
-$EndComp
-$Comp
-L power:GND #PWR?
-U 1 1 5C4D9F5A
-P 9100 1700
-F 0 "#PWR?" H 9100 1450 50  0001 C CNN
-F 1 "GND" H 9105 1527 50  0000 C CNN
-F 2 "" H 9100 1700 50  0001 C CNN
-F 3 "" H 9100 1700 50  0001 C CNN
-	1    9100 1700
-	1    0    0    -1
-$EndComp
-Wire Wire Line
-	9100 850  8900 850
-Wire Wire Line
-	9100 1700 9100 1600
-Wire Wire Line
-	9100 1150 9100 1200
-Wire Wire Line
-	9100 1200 9200 1200
-Connection ~ 9100 1200
-Wire Wire Line
-	9100 1200 9100 1300
 $Comp
 L Device:R R?
@@
 Text Label 8400 4750 0    50   ~ 0
 CS6_OUT
+Text Label 6600 1750 1    50   ~ 0
+5V
 $EndSCHEMATC

Commit message: Final schematic of Temperature board for BPS
Parts:
- removed J?: Conn_01x02, symbol Connector_Generic:Conn_01x02
- added D1: LED, symbol Device:LED
- added J2: Logic Analyzer, symbol Connector_Generic:Conn_01x05
- added J4: Conn_02x06_Counter_Clockwise, symbol Connector_Generic:Conn_02x06_Counter_Clockwise
- added MH1, MH2, MH3, MH4: MountingHole, MountingHole:MountingHole_3mm, symbol Mechanical:MountingHole
- added TP1, TP2: TestPoint, symbol Connector:TestPoint
- gave numbers to parts that had none: 50
Connections:
- net labels added: +5V, CS_FINAL
- net labels removed: +5VL, 5V, CH1, CH10, CH11, CH12, CH13, CH14, CH15, CH16, CH17, CH18, CH19, CH2, CH20, CH3, CH4, CH5, CH6, CH7, CH8, CH9
- wire segments 230 -> 307
- no-connect marks 0 -> 2

Commit message: Created PCB of Temperture Board for BPS
Parts:
- C1, C10, C11, C12, C13, C14, C15, C16, C17, C18, C19, C2, C20, C21, C22, C23, C24, C25, C26, C3, C4, C5, C6, C7, C8, C9: footprint (none) -> Capacitor_SMD:C_0805_2012Metric
- D1: footprint (none) -> LED_SMD:LED_0805_2012Metric
- J1: footprint (none) -> Connector_Molex:Molex_Micro-Fit_3.0_43045-2012_2x10_P3.00mm_Vertical
- J2: footprint (none) -> Connector_PinHeader_2.54mm:PinHeader_1x05_P2.54mm_Vertical
- J3, J4: footprint (none) -> UTSVT_Connectors:Molex_MicroFit3.0_2x6xP3.00mm_PolarizingPeg_Vertical
- R1, R10, R11, R12, R13, R14, R15, R16, R17, R18, R19, R2, R20, R3, R4, R5, R6, R7, R8, R9: footprint (none) -> Resistor_SMD:R_0805_2012Metric
- SW1: footprint (none) -> Button_Switch_SMD:SW_DIP_SPSTx06_Slide_Omron_A6S-610x_W8.9mm_P2.54mm
- TP1, TP2: footprint (none) -> TestPoint:TestPoint_Keystone_5005-5009_Compact
Other:
- note added: "6 position dip switch : Omron A6s-610x"
- note removed: "CT2196MST-ND : 6 position dip switch"

Commit message: Made edits to temperature board. Finalized boards.
Parts:
- added J5: Conn_01x02, UTSVT_Connectors:43650-0202_01x02_Microfit 3.0_horizontal, symbol Connector_Generic:Conn_01x02
- added L1, L10, L11, L12, L13, L14, L15, L16, L17, L18, L19, L2, L20, L3, L4, L5, L6, L7, L8, L9: Ferrite_Bead, Inductor_SMD:L_0805_2012Metric, symbol Device:Ferrite_Bead
- added R21: 1.55k, Resistor_SMD:R_0805_2012Metric, symbol Device:R
- J1: footprint Connector_Molex:Molex_Micro-Fit_3.0_43045-2012_2x10_P3.00mm_Vertical -> UTSVT_Connectors:Molex_Micro-Fit_3.0_43045-2010_2x10-1MP_P3.00mm_Horizontal
Connections:
- wire segments 307 -> 373
